Commit message: Refactor Allie URDF xacro, add ros2_control setup, update RViz launch with LC_ALL, and clean parent-child frame structure

File: cororos2_allie_description/urdf/allie/allie_macro.ros2_control.xacro (robot description, xacro)
@@ -8,6 +8,5 @@
                sim_gazebo_classic:=false
                sim_gazebo:=false
-               simulation_controllers"
-               >
+               simulation_controllers">
     <ros2_control name="${name}" type="system">
       <hardware>
@@ -26,96 +25,34 @@
         </xacro:unless>
       </hardware>
-      <joint name="${prefix}joint1">
-        <command_interface name="position">     <!-- Add/Remove interfaces as needed -->
-          <param name="min">-1</param>
-          <param name="max">1</param>
-        </command_interface>
+      <joint name="${prefix}front_left_wheel_joint">
+        <command_interface name="velocity" />
         <state_interface name="position">
           <param name="initial_value">0.0</param>
         </state_interface>
-        <state_interface name="velocity"/>
-        <state_interface name="acceleration"/>
+        <state_interface name="velocity" />
       </joint>
-      <joint name="${prefix}joint2">
-        <command_interface name="position">     <!-- Add/Remove interfaces as needed -->
-          <param name="min">-1</param>
-          <param name="max">1</param>
-        </command_interface>
+      <joint name="${prefix}front_right_wheel_joint">
+        <command_interface name="velocity" />
         <state_interface name="position">
           <param name="initial_value">0.0</param>
         </state_interface>
-        <state_interface name="velocity"/>
-        <state_interface name="acceleration"/>
+        <state_interface name="velocity" />
       </joint>
-      <joint name="${prefix}joint3">
-        <command_interface name="position">     <!-- Add/Remove interfaces as needed -->
-          <param name="min">-1</param>
-          <param name="max">1</param>
-        </command_interface>
+      <joint name="${prefix}rear_left_wheel_joint">
+        <command_interface name="velocity" />
         <state_interface name="position">
           <param name="initial_value">0.0</param>
         </state_interface>
-        <state_interface name="velocity"/>
-        <state_interface name="acceleration"/>
+        <state_interface name="velocity" />
       </joint>
-      <joint name="${prefix}joint4">
-        <command_interface name="position">     <!-- Add/Remove interfaces as needed -->
-          <param name="min">-1</param>
-          <param name="max">1</param>
-        </command_interface>
+      <joint name="${prefix}rear_right_wheel_joint">
+        <command_interface name="velocity" />
         <state_interface name="position">
           <param name="initial_value">0.0</param>
         </state_interface>
-        <state_interface name="velocity"/>
-        <state_interface name="acceleration"/>
+        <state_interface name="velocity" />
       </joint>
-      <joint name="${prefix}joint5">
-        <command_interface name="position">     <!-- Add/Remove interfaces as needed -->
-          <param name="min">-1</param>
-          <param name="max">1</param>
-        </command_interface>
-        <state_interface name="position">
-          <param name="initial_value">0.0</param>
-        </state_interface>
-        <state_interface name="velocity"/>
-        <state_interface name="acceleration"/>
-      </joint>
-      <joint name="${prefix}joint6">
-        <command_interface name="position">     <!-- Add/Remove interfaces as needed -->
-          <param name="min">-1</param>
-          <param name="max">1</param>
-        </command_interface>
-        <state_interface name="position">
-          <param name="initial_value">0.0</param>
-        </state_interface>
-        <state_interface name="velocity"/>
-        <state_interface name="acceleration"/>
-      </joint>
-      <sensor name="tcp_fts_sensor">            <!-- Remove/change sensors as needed -->
-        <state_interface name="fx"/>
-        <state_interface name="fy"/>
-        <state_interface name="fz"/>
-        <state_interface name="tx"/>
-        <state_interface name="ty"/>
-        <state_interface name="tz"/>
-        <param name="frame_id">tool0</param>    <!-- Change sensors as needed -->
-        <param name="min_fx">-100</param>
-        <param name="max_fx">100</param>
-        <param name="min_fy">-100</param>
-        <param name="max_fy">100</param>
-        <param name="min_fz">-200</param>
-        <param name="max_fz">200</param>
-        <param name="min_tx">-10</param>
-        <param name="max_tx">10</param>
-        <param name="min_ty">-10</param>
-        <param name="max_ty">10</param>
-        <param name="min_tz">-15</param>
-        <param name="max_tz">15</param>
-      </sensor>
     </ros2_control>
-    <xacro:if value="$(arg sim_gazebo_classic)">
-      <!-- Gazebo plugins -->
-      <gazebo reference="world">
-      </gazebo>
+    <xacro:if value="${sim_gazebo_classic}">
       <gazebo>
         <plugin filename="libgazebo_ros2_control.so" name="gazebo_ros2_control">
@@ -124,8 +61,5 @@
       </gazebo>
     </xacro:if>
-    <xacro:if value="$(arg sim_gazebo)">
-      <!-- Gazebo plugins -->
-      <gazebo reference="world">
-      </gazebo>
+    <xacro:if value="${sim_gazebo}">
       <gazebo>
         <plugin filename="gz_ros2_control-system" name="gz_ros2_control::GazeboSimROS2ControlPlugin">

File: cororos2_allie_description/urdf/allie/allie_macro.xacro (robot description, xacro)
@@ -1,244 +1,1015 @@
-<?xml version="1.0" encoding="UTF-8"?>
+<?xml version='1.0' encoding='utf-8'?>
 <robot xmlns:xacro="http://wiki.ros.org/xacro">
-  <xacro:include filename="$(find cororos2_allie_description)/urdf/common/inertials.xacro"/>
-  <xacro:include filename="$(find cororos2_allie_description)/urdf/common/materials.xacro"/>
   <xacro:macro name="allie" params="prefix parent *origin">
     <!-- LINKS -->
+    <!-- base footprint -->
+    <link name="${prefix}base_footprint">
+    </link>
     <!-- base link -->
     <link name="${prefix}base_link">
-      <!-- Default inertial for Gazebo - copy and edit block from 'common.xacro'
-           to get more realistic behavior -->
-      <xacro:default_inertial/>
-      <visual>
-        <origin xyz="0 0 0" rpy="0 0 0"/>
-        <geometry>
-          <cylinder length="0.3" radius="0.3"/>
-          <!--           <mesh filename="package://cororos2_allie_description/meshes/allie/visual/base_link.dae" /> -->
-        </geometry>
-        <material name="black"/>
-      </visual>
-      <collision>
-        <origin xyz="0 0 0" rpy="0 0 0"/>
-        <geometry>
-          <cylinder length="0.3" radius="0.3"/>
-          <!--           <mesh filename="package://cororos2_allie_description/meshes/allie/collision/base_link.stl" /> -->
+      <inertial>
+        <origin xyz="0 0 0.09" rpy="0 0 0" />
+        <mass value="26.6" />
+        <inertia ixx="0.387" ixy="0" ixz="0" iyy="0.790" iyz="0" izz="0.962" />
+      </inertial>
+      <collision name="chassis_collision">
+        <origin xyz="0 0 0.05" rpy="0 0 0" />
+        <geometry>
+          <box size="0.555 0.355 0.13" />
         </geometry>
       </collision>
-    </link>
-    <!-- link 1 -->
-    <link name="${prefix}link1">
-      <!-- Default inertial for Gazebo - copy and edit block from 'common.xacro'
-           to get more realistic behavior -->
-      <xacro:default_inertial/>
-      <visual>
-        <origin xyz="0 0 0" rpy="0 0 0"/>
-        <geometry>
-          <cylinder length="0.3" radius="0.15"/>
-          <!--           <mesh filename="package://cororos2_allie_description/meshes/allie/visual/link1.dae" /> -->
-        </geometry>
-        <material name="blue"/>
-      </visual>
-      <collision>
-        <origin xyz="0 0 0" rpy="0 0 0"/>
-        <geometry>
-          <cylinder length="0.3" radius="0.15"/>
-          <!--           <mesh filename="package://cororos2_allie_description/meshes/allie/collision/link1.stl" /> -->
-        </geometry>
-        <material name="green"/>
+      <collision name="tower_collision">
+        <origin xyz="0.13 0 0.27" rpy="0 0 0" />
+        <geometry>
+          <box size="0.2 0.2 0.34" />
+        </geometry>
       </collision>
-    </link>
-    <!-- link 2 -->
-    <link name="${prefix}link2">
-      <!-- Default inertial for Gazebo - copy and edit block from 'common.xacro'
-           to get more realistic behavior-->
-      <xacro:default_inertial/>
-      <visual>
-        <origin xyz="0 0 0" rpy="0 0 0"/>
-        <geometry>
-          <cylinder length="0.3" radius="0.15"/>
-          <!--           <mesh filename="package://cororos2_allie_description/meshes/allie/visual/link2.dae" /> -->
-        </geometry>
-        <material name="grey"/>
-      </visual>
-      <collision>
-        <origin xyz="0 0 0" rpy="0 0 0"/>
-        <geometry>
-          <cylinder length="0.3" radius="0.15"/>
-          <!--           <mesh filename="package://cororos2_allie_description/meshes/allie/collision/link2.stl"  /> -->
+      <visual name="chassis_main_visual">
+        <origin xyz="0 0 0.05" rpy="0 0 0" />
+        <geometry>
+          <box size="0.555 0.355 0.13" />
+        </geometry>
+        <material name="chassis_main_visual_mat">
+          <color rgba="0.6 0.6 0.6 1.0" />
+        </material>
+      </visual>
+      <visual name="emergency_stop_bottom_visual">
+        <origin xyz="0.2 0.15 0.125" rpy="0 0 0" />
+        <geometry>
+          <cylinder radius="0.015" length="0.015" />
+        </geometry>
+        <material name="emergency_stop_bottom_visual_mat">
+          <color rgba="0.7059 0.7059 0.7059 1.0" />
+        </material>
+      </visual>
+      <visual name="emergency_stop_top_visual">
+        <origin xyz="0.2 0.15 0.135" rpy="0 0 0" />
+        <geometry>
+          <cylinder radius="0.02" length="0.005" />
+        </geometry>
+        <material name="emergency_stop_top_visual_mat">
+          <color rgba="1.0 0.0 0.0 1.0" />
+        </material>
+      </visual>
+      <visual name="wheel_mount_front_visual">
+        <origin xyz="0.249 0 0.011" rpy="0 0 0" />
+        <geometry>
+          <box size="0.05 0.5 0.05" />
+        </geometry>
+        <material name="wheel_mount_front_visual_mat">
+          <color rgba="0.6 0.6 0.6 1.0" />
+        </material>
+      </visual>
+      <visual name="wheel_mount_rear_visual">
+        <origin xyz="-0.249 0 0.011" rpy="0 0 0" />
+        <geometry>
+          <box size="0.05 0.5 0.05" />
+        </geometry>
+        <material name="wheel_mount_rear_visual_mat">
+          <color rgba="0.6 0.6 0.6 1.0" />
+        </material>
+      </visual>
+      <visual name="plate1_visual">
+        <origin xyz="0.13 0 0.42" rpy="0 0 0" />
+        <geometry>
+          <box size="0.2 0.2 0.005" />
+        </geometry>
+        <material name="plate1_visual_mat">
+          <color rgba="0.7843 0.7843 0.7843 1.0" />
+        </material>
+      </visual>
+      <visual name="plate2_visual">
+        <origin xyz="0.13 0 0.31" rpy="0 0 0" />
+        <geometry>
+          <box size="0.2 0.2 0.005" />
+        </geometry>
+        <material name="plate2_visual_mat">
+          <color rgba="0.7843 0.7843 0.7843 1.0" />
+        </material>
+      </visual>
+      <visual name="plate3_visual">
+        <origin xyz="0.13 0 0.12" rpy="0 0 0" />
+        <geometry>
+          <box size="0.2 0.2 0.005" />
+        </geometry>
+        <material name="plate3_visual_mat">
+          <color rgba="0.9412 0.9412 0.9412 1.0" />
+        </material>
+      </visual>
+      <visual name="beam1_visual">
+        <origin xyz="0.221 0.091 0.27" rpy="0 0 0" />
+        <geometry>
+          <box size="0.02 0.02 0.3" />
+        </geometry>
+        <material name="beam1_visual_mat">
+          <color rgba="0.7843 0.7843 0.7843 1.0" />
+        </material>
+      </visual>
+      <visual name="beam2_visual">
+        <origin xyz="0.221 -0.091 0.27" rpy="0 0 0" />
+        <geometry>
+          <box size="0.02 0.02 0.3" />
+        </geometry>
+        <material name="beam2_visual_mat">
+          <color rgba="0.7843 0.7843 0.7843 1.0" />
+        </material>
+      </visual>
+      <visual name="beam3_visual">
+        <origin xyz="0.039 0.091 0.27" rpy="0 0 0" />
+        <geometry>
+          <box size="0.02 0.02 0.3" />
+        </geometry>
+        <material name="beam3_visual_mat">
+          <color rgba="0.7843 0.7843 0.7843 1.0" />
+        </material>
+      </visual>
+      <visual name="beam4_visual">
+        <origin xyz="0.039 -0.091 0.27" rpy="0 0 0" />
+        <geometry>
+          <box size="0.02 0.02 0.3" />
+        </geometry>
+        <material name="beam4_visual_mat">
+          <color rgba="0.7843 0.7843 0.7843 1.0" />
+        </material>
+      </visual>
+    </link>
+    <!-- drive wheels -->
+    <!-- front left wheel -->
+    <link name="${prefix}front_left_wheel">
+      <inertial>
+        <origin xyz="0 0 0" rpy="0 0 0" />
+        <mass value="5.124" />
+        <inertia ixx="0.0576" ixy="0" ixz="0" iyy="0.105" iyz="0" izz="0.0576" />
+      </inertial>
+      <collision name="front_left_wheel_collision">
+        <origin xyz="0 0 0" rpy="-1.5708 0 0" />
+        <geometry>
+          <cylinder radius="0.205" length="0.11" />
         </geometry>
       </collision>
-    </link>
-    <!-- link 3 -->
-    <link name="${prefix}link3">
-      <!-- Default inertial for Gazebo - copy and edit block from 'common.xacro'
-           to get more realistic behavior-->
-      <xacro:default_inertial/>
-      <visual>
-        <origin xyz="0 0 0" rpy="0 0 0"/>
-        <geometry>
-          <cylinder length="0.2" radius="0.1"/>
-          <!--           <mesh filename="package://cororos2_allie_description/meshes/allie/visual/link3.dae" /> -->
-        </geometry>
-        <material name="orange"/>
-      </visual>
-      <collision>
-        <origin xyz="0 0 0" rpy="0 0 0"/>
-        <geometry>
-          <cylinder length="0.2" radius="0.1"/>
-          <!--           <mesh filename="package://cororos2_allie_description/meshes/allie/collision/link3.stl"  /> -->
+      <visual name="front_left_wheel_tire_visual">
+        <origin xyz="0 0 0" rpy="0 0 0" />
+        <geometry>
+          <mesh filename="package://cororos2_allie_description/meshes/allie/visual/wheel.dae" scale="1.18 1.0 1.18" />
+        </geometry>
+      </visual>
+    </link>
+    <!-- front right wheel -->
+    <link name="${prefix}front_right_wheel">
+      <inertial>
+        <origin xyz="0 0 0" rpy="0 0 0" />
+        <mass value="5.124" />
+        <inertia ixx="0.0576" ixy="0" ixz="0" iyy="0.105" iyz="0" izz="0.0576" />
+      </inertial>
+      <collision name="front_right_wheel_collision">
+        <origin xyz="0 0 0" rpy="1.5708 0 0" />
+        <geometry>
+          <cylinder radius="0.205" length="0.11" />
         </geometry>
       </collision>
-    </link>
-    <!-- link 4 -->
-    <link name="${prefix}link4">
-      <!-- Default inertial for Gazebo - copy and edit block from 'common.xacro'
-           to get more realistic behavior-->
-      <xacro:default_inertial/>
-      <visual>
-        <origin xyz="0 0 0" rpy="0 0 0"/>
-        <geometry>
-          <cylinder length="0.1" radius="0.1"/>
-          <!--           <mesh filename="package://cororos2_allie_description/meshes/allie/visual/link4.dae" /> -->
-        </geometry>
-        <material name="brown"/>
-      </visual>
-      <collision>
-        <origin xyz="0 0 0" rpy="0 0 0"/>
-        <geometry>
-          <cylinder length="0.1" radius="0.1"/>
-          <!--           <mesh filename="package://cororos2_allie_description/meshes/allie/collision/link4.stl"  /> -->
+      <visual name="front_right_wheel_tire_visual">
+        <origin xyz="0 0 0" rpy="0 0 0" />
+        <geometry>
+          <mesh filename="package://cororos2_allie_description/meshes/allie/visual/wheel.dae" scale="1.18 1.0 1.18" />
+        </geometry>
+      </visual>
+    </link>
+    <!-- rear left wheel -->
+    <link name="${prefix}rear_left_wheel">
+      <inertial>
+        <origin xyz="0 0 0" rpy="0 0 0" />
+        <mass value="5.124" />
+        <inertia ixx="0.0576" ixy="0" ixz="0" iyy="0.105" iyz="0" izz="0.0576" />
+      </inertial>
+      <collision name="rear_left_wheel_collision">
+        <origin xyz="0 0 0" rpy="-1.5708 0 0" />
+        <geometry>
+          <cylinder radius="0.205" length="0.11" />
         </geometry>
       </collision>
-    </link>
-    <!-- link 5 -->
-    <link name="${prefix}link5">
-      <!-- Default inertial for Gazebo - copy and edit block from 'common.xacro'
-           to get more realistic behavior-->
-      <xacro:default_inertial/>
-      <visual>
-        <origin xyz="0 0 0" rpy="0 0 0"/>
-        <geometry>
-          <cylinder length="0.15" radius="0.1"/>
-          <!--           <mesh filename="package://cororos2_allie_description/meshes/allie/visual/link5.dae" /> -->
-        </geometry>
-        <material name="red"/>
-      </visual>
-      <collision>
-        <origin xyz="0 0 0" rpy="0 0 0"/>
-        <geometry>
-          <cylinder length="0.15" radius="0.1"/>
-          <!--           <mesh filename="package://cororos2_allie_description/meshes/allie/collision/link5.stl" /> -->
+      <visual name="rear_left_wheel_tire_visual">
+        <origin xyz="0 0 0" rpy="0 0 0" />
+        <geometry>
+          <mesh filename="package://cororos2_allie_description/meshes/allie/visual/wheel.dae" scale="1.18 1.0 1.18" />
+        </geometry>
+      </visual>
+    </link>
+    <!-- rear right wheel -->
+    <link name="${prefix}rear_right_wheel">
+      <inertial>
+        <origin xyz="0 0 0" rpy="0 0 0" />
+        <mass value="5.124" />
+        <inertia ixx="0.0576" ixy="0" ixz="0" iyy="0.105" iyz="0" izz="0.0576" />
+      </inertial>
+      <collision name="rear_right_wheel_collision">
+        <origin xyz="0 0 0" rpy="1.5708 0 0" />
+        <geometry>
+          <cylinder radius="0.205" length="0.11" />
         </geometry>
       </collision>
-    </link>
-    <!-- link 6 -->
-    <link name="${prefix}link6">
-      <!-- Default inertial for Gazebo - copy and edit block from 'common.xacro'
-           to get more realistic behavior-->
-      <xacro:default_inertial/>
-      <visual>
-        <origin xyz="0 0 0" rpy="0 0 0"/>
-        <geometry>
-          <cylinder length="0.05" radius="0.075"/>
-          <!--           <mesh filename="package://cororos2_allie_description/meshes/allie/visual/link6.dae" /> -->
-        </geometry>
-        <material name="white"/>
-      </visual>
-      <collision>
-        <origin xyz="0 0 0" rpy="0 0 0"/>
-        <geometry>
-          <cylinder length="0.05" radius="0.075"/>
-          <!--           <mesh filename="package://cororos2_allie_description/meshes/allie/collision/link6.stl" /> -->
-        </geometry>
-      </collision>
-    </link>
-    <!-- All-zero tool frame. This frame should correspond to the TOOL frame of the robot's controller.) -->
-    <link name="${prefix}tool0"/>
-    <!-- tool link -->
-    <!-- START Delete if not needed -->
-    <!-- Standard frames for industrial robots. Also useful for manipulators.
-         (ROS-I specs - https://wiki.ros.org/Industrial/Tutorials/WorkingWithRosIndustrialRobotSupportPackages#Standardised_links_.2F_frames)-->
-    <!-- This frame should correspond to the BASE coordinate system of robot's controller.) -->
-    <link name="${prefix}base"/>
-    <!-- Frame for mounting EEF models to a manipulator. x+ axis points forward (REP 103). -->
-    <link name="${prefix}flange"/>
-    <!-- END Delete if not needed  -->
-    <!-- END LINKS -->
+      <visual name="rear_right_wheel_tire_visual">
+        <origin xyz="0 0 0" rpy="0 0 0" />
+        <geometry>
+          <mesh filename="package://cororos2_allie_description/meshes/allie/visual/wheel.dae" scale="1.18 1.0 1.18" />
+        </geometry>
+      </visual>
+    </link>
+    <!-- sensor and light frames -->
+    <!-- IMU frame -->
+    <link name="${prefix}imu_sensor_link">
+      <inertial>
+        <origin xyz="0 0 0" rpy="0 0 0" />
+        <mass value="1e-6" />
+        <inertia ixx="1e-9" ixy="0" ixz="0" iyy="1e-9" iyz="0" izz="1e-9" />
+      </inertial>
+    </link>
+    <!-- air pressure frame -->
+    <link name="${prefix}air_pressure_link">
+      <inertial>
+        <origin xyz="0 0 0" rpy="0 0 0" />
+        <mass value="1e-6" />
+        <inertia ixx="1e-9" ixy="0" ixz="0" iyy="1e-9" iyz="0" izz="1e-9" />
+      </inertial>
+    </link>
+    <!-- magnetometer frame -->
+    <link name="${prefix}magnetometer_link">
+      <inertial>
+        <origin xyz="0 0 0" rpy="0 0 0" />
+        <mass value="1e-6" />
+        <inertia ixx="1e-9" ixy="0" ixz="0" iyy="1e-9" iyz="0" izz="1e-9" />
+      </inertial>
+    </link>
+    <!-- front RGB-D camera frame -->
+    <link name="${prefix}rgbd_front_link">
+      <inertial>
+        <origin xyz="0 0 0" rpy="0 0 0" />
+        <mass value="1e-6" />
+        <inertia ixx="1e-9" ixy="0" ixz="0" iyy="1e-9" iyz="0" izz="1e-9" />
+      </inertial>
+      <visual name="d435i_realsense_camera_visual">
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