Commit message: Add ouster lidar driver, dependency and frames

File: cororos2_allie_description/urdf/allie/allie_macro.xacro (robot description, xacro)
@@ -358,29 +358,37 @@
       </visual>
     </link>
-    <!-- front lidar frame -->
-    <link name="${prefix}front_laser_link">
-      <inertial>
-        <origin xyz="0 0 0" rpy="0 0 0" />
-        <mass value="1e-6" />
-        <inertia ixx="1e-9" ixy="0" ixz="0" iyy="1e-9" iyz="0" izz="1e-9" />
-      </inertial>
-      <visual name="vlp16_visual1">
-        <origin xyz="0 0 -0.038" rpy="0 0 0" />
-        <geometry>
-          <mesh filename="package://cororos2_allie_description/meshes/allie/visual/VLP16_base_1.dae" scale="1 1 1" />
-        </geometry>
-      </visual>
-      <visual name="vlp_visual2">
-        <origin xyz="0 0 -0.038" rpy="0 0 0" />
-        <geometry>
-          <mesh filename="package://cororos2_allie_description/meshes/allie/visual/VLP16_base_2.dae" scale="1 1 1" />
-        </geometry>
-      </visual>
-      <visual name="vlp_visual3">
-        <origin xyz="0 0 -0.038" rpy="0 0 0" />
-        <geometry>
-          <mesh filename="package://cororos2_allie_description/meshes/allie/visual/VLP16_scan.dae" scale="1 1 1" />
-        </geometry>
-      </visual>
+    <!-- Ouster sensor frame -->
+    <link name="${prefix}ouster_link">
+      <inertial>
+        <origin xyz="0 0 0" rpy="0 0 0" />
+        <mass value="1e-6" />
+        <inertia ixx="1e-9" ixy="0" ixz="0" iyy="1e-9" iyz="0" izz="1e-9" />
+      </inertial>
+      <visual name="ouster_body_visual">
+        <origin xyz="0 0 0" rpy="0 0 0" />
+        <geometry>
+          <cylinder radius="0.055" length="0.075" />
+        </geometry>
+        <material name="ouster_body_visual_mat">
+          <color rgba="0.1 0.1 0.1 1.0" />
+        </material>
+      </visual>
+      <visual name="ouster_window_visual">
+        <origin xyz="0.042 0 0" rpy="0 0 0" />
+        <geometry>
+          <box size="0.008 0.09 0.035" />
+        </geometry>
+        <material name="ouster_window_visual_mat">
+          <color rgba="0.2 0.25 0.3 1.0" />
+        </material>
+      </visual>
+    </link>
+    <!-- Ouster internal IMU frame -->
+    <link name="${prefix}ouster_imu_link">
+      <inertial>
+        <origin xyz="0 0 0" rpy="0 0 0" />
+        <mass value="1e-6" />
+        <inertia ixx="1e-9" ixy="0" ixz="0" iyy="1e-9" iyz="0" izz="1e-9" />
+      </inertial>
     </link>
     <!-- front light frame -->
@@ -548,9 +556,15 @@
       <origin xyz="0.13 -0.11 0.405" rpy="0 0 -1.5708" />
     </joint>
-    <!-- base link to front lidar frame -->
-    <joint name="${prefix}base_link_to_front_laser_link_joint" type="fixed">
-      <parent link="${prefix}base_link" />
-      <child link="${prefix}front_laser_link" />
+    <!-- base link to Ouster sensor frame -->
+    <joint name="${prefix}base_link_to_ouster_link_joint" type="fixed">
+      <parent link="${prefix}base_link" />
+      <child link="${prefix}ouster_link" />
       <origin xyz="0.13 0 0.35" rpy="0 -0 0" />
+    </joint>
+    <!-- Ouster sensor frame to Ouster IMU frame -->
+    <joint name="${prefix}ouster_link_to_ouster_imu_link_joint" type="fixed">
+      <parent link="${prefix}ouster_link" />
+      <child link="${prefix}ouster_imu_link" />
+      <origin xyz="0 0 0" rpy="0 0 0" />
     </joint>
     <!-- base link to front light frame -->
@@ -903,6 +917,6 @@
       </sensor>
     </gazebo>
-    <gazebo reference="${prefix}front_laser_link">
-      <sensor name="front_laser" type="gpu_lidar">
+    <gazebo reference="${prefix}ouster_link">
+      <sensor name="ouster_lidar" type="gpu_lidar">
         <visualize>0</visualize>
         <update_rate>10</update_rate>
@@ -916,8 +930,8 @@
             </horizontal>
             <vertical>
-              <samples>16</samples>
+              <samples>128</samples>
               <resolution>1</resolution>
-              <min_angle>-0.261799</min_angle>
-              <max_angle>0.261799</max_angle>
+              <min_angle>-0.785398</min_angle>
+              <max_angle>0.785398</max_angle>
             </vertical>
           </scan>

Commit message: Add realsense dependency, driver and fix mount position

File: cororos2_allie_description/urdf/allie/allie_macro.xacro (robot description, xacro)
@@ -530,5 +530,5 @@
       <parent link="${prefix}base_link" />
       <child link="${prefix}rgbd_front_link" />
-      <origin xyz="0.21 0 0.393" rpy="0 0.52 0" />
+      <origin xyz="0.21 0 1.5" rpy="0 -0.5236 0" />
     </joint>
     <!-- base link to front camera frame -->

Commit message: Add gps dependency, driver, yaml and frames

File: cororos2_allie_description/urdf/allie/allie_macro.xacro (robot description, xacro)
@@ -234,4 +234,12 @@
     <!-- magnetometer frame -->
     <link name="${prefix}magnetometer_link">
+      <inertial>
+        <origin xyz="0 0 0" rpy="0 0 0" />
+        <mass value="1e-6" />
+        <inertia ixx="1e-9" ixy="0" ixz="0" iyy="1e-9" iyz="0" izz="1e-9" />
+      </inertial>
+    </link>
+    <!-- GPS frame -->
+    <link name="${prefix}gps_link">
       <inertial>
         <origin xyz="0 0 0" rpy="0 0 0" />
@@ -525,4 +533,10 @@
       <child link="${prefix}magnetometer_link" />
       <origin xyz="0 0 0" rpy="0 0 0" />
+    </joint>
+    <!-- base link to GPS frame -->
+    <joint name="${prefix}base_link_to_gps_link_joint" type="fixed">
+      <parent link="${prefix}base_link" />
+      <child link="${prefix}gps_link" />
+      <origin xyz="0.13 0 1.58" rpy="0 0 0" />
     </joint>
     <!-- base link to front RGB-D camera frame -->

Commit message: Fix camera orientation

File: cororos2_allie_description/urdf/allie/allie_macro.xacro (robot description, xacro)
@@ -546,5 +546,5 @@
       <parent link="${prefix}base_link" />
       <child link="${prefix}rgbd_front_link" />
-      <origin xyz="0.21 0 1.5" rpy="0 -0.5236 0" />
+      <origin xyz="0.21 0 1.5" rpy="0 0.5236 0" />
     </joint>
     <!-- base link to front camera frame -->

Commit message: Remove unused Allie sensor references

File: cororos2_allie_description/urdf/allie/allie_macro.xacro (robot description, xacro)
@@ -224,20 +224,4 @@
       </inertial>
     </link>
-    <!-- air pressure frame -->
-    <link name="${prefix}air_pressure_link">
-      <inertial>
-        <origin xyz="0 0 0" rpy="0 0 0" />
-        <mass value="1e-6" />
-        <inertia ixx="1e-9" ixy="0" ixz="0" iyy="1e-9" iyz="0" izz="1e-9" />
-      </inertial>
-    </link>
-    <!-- magnetometer frame -->
-    <link name="${prefix}magnetometer_link">
-      <inertial>
-        <origin xyz="0 0 0" rpy="0 0 0" />
-        <mass value="1e-6" />
-        <inertia ixx="1e-9" ixy="0" ixz="0" iyy="1e-9" iyz="0" izz="1e-9" />
-      </inertial>
-    </link>
     <!-- GPS frame -->
     <link name="${prefix}gps_link">
@@ -260,108 +244,4 @@
           <mesh filename="package://cororos2_allie_description/meshes/allie/visual/realsense_d435.dae" scale="0.001 0.001 0.001" />
         </geometry>
-      </visual>
-    </link>
-    <!-- front camera frame -->
-    <link name="${prefix}camera_front_link">
-      <inertial>
-        <origin xyz="0 0 0" rpy="0 0 0" />
-        <mass value="1e-6" />
-        <inertia ixx="1e-9" ixy="0" ixz="0" iyy="1e-9" iyz="0" izz="1e-9" />
-      </inertial>
-      <visual name="camera_front_visual">
-        <origin xyz="-0.02 0 0" rpy="0 0 0" />
-        <geometry>
-          <box size="0.01 0.03 0.03" />
-        </geometry>
-        <material name="camera_front_visual_mat">
-          <color rgba="0.0 0.0 0.0 1.0" />
-        </material>
-      </visual>
-      <visual name="camera_lens_front_visual">
-        <origin xyz="-0.01 0 0" rpy="3.141593 1.570793 3.141593" />
-        <geometry>
-          <cylinder radius="0.005" length="0.011" />
-        </geometry>
-        <material name="camera_lens_front_visual_mat">
-          <color rgba="0.0 0.0 0.0 1.0" />
-        </material>
-      </visual>
-    </link>
-    <!-- rear camera frame -->
-    <link name="${prefix}camera_rear_link">
-      <inertial>
-        <origin xyz="0 0 0" rpy="0 0 0" />
-        <mass value="1e-6" />
-        <inertia ixx="1e-9" ixy="0" ixz="0" iyy="1e-9" iyz="0" izz="1e-9" />
-      </inertial>
-      <visual name="camera_rear_visual">
-        <origin xyz="-0.02 0 0" rpy="0 0 -3.14159" />
-        <geometry>
-          <box size="0.01 0.03 0.03" />
-        </geometry>
-        <material name="camera_rear_visual_mat">
-          <color rgba="0.0 0.0 0.0 1.0" />
-        </material>
-      </visual>
-      <visual name="camera_lens_rear_visual">
-        <origin xyz="-0.01 0 0" rpy="3.141593 1.570793 0.000003" />
-        <geometry>
-          <cylinder radius="0.005" length="0.011" />
-        </geometry>
-        <material name="camera_lens_rear_visual_mat">
-          <color rgba="0.0 0.0 0.0 1.0" />
-        </material>
-      </visual>
-    </link>
-    <!-- left camera frame -->
-    <link name="${prefix}camera_left_link">
-      <inertial>
-        <origin xyz="0 0 0" rpy="0 0 0" />
-        <mass value="1e-6" />
-        <inertia ixx="1e-9" ixy="0" ixz="0" iyy="1e-9" iyz="0" izz="1e-9" />
-      </inertial>
-      <visual name="camera_left_visual">
-        <origin xyz="-0.02 0 0" rpy="0 0 -1.5708" />
-        <geometry>
-          <box size="0.03 0.01 0.03" />
-        </geometry>
-        <material name="camera_left_visual_mat">
-          <color rgba="0.0 0.0 0.0 1.0" />
-        </material>
-      </visual>
-      <visual name="camera_lens_left_visual">
-        <origin xyz="-0.01 0 0" rpy="1.5708 0 -1.5708" />
-        <geometry>
-          <cylinder radius="0.005" length="0.011" />
-        </geometry>
-        <material name="camera_lens_left_visual_mat">
-          <color rgba="0.0 0.0 0.0 1.0" />
-        </material>
-      </visual>
-    </link>
-    <!-- right camera frame -->
-    <link name="${prefix}camera_right_link">
-      <inertial>
-        <origin xyz="0 0 0" rpy="0 0 0" />
-        <mass value="1e-6" />
-        <inertia ixx="1e-9" ixy="0" ixz="0" iyy="1e-9" iyz="0" izz="1e-9" />
-      </inertial>
-      <visual name="camera_right_visual">
-        <origin xyz="-0.02 0 0" rpy="0 0 1.5708" />
-        <geometry>
-          <box size="0.03 0.01 0.03" />
-        </geometry>
-        <material name="camera_right_visual_mat">
-          <color rgba="0.0 0.0 0.0 1.0" />
-        </material>
-      </visual>
-      <visual name="camera_lens_right_visual">
-        <origin xyz="-0.01 0 0" rpy="1.5708 0 1.5708" />
-        <geometry>
-          <cylinder radius="0.005" length="0.011" />
-        </geometry>
-        <material name="camera_lens_right_visual_mat">
-          <color rgba="0.0 0.0 0.0 1.0" />
-        </material>
       </visual>
     </link>
@@ -524,16 +404,4 @@
       <origin xyz="0 0 0" rpy="0 0 0" />
     </joint>
-    <!-- base link to air pressure frame -->
-    <joint name="${prefix}base_link_to_air_pressure_link_joint" type="fixed">
-      <parent link="${prefix}base_link" />
-      <child link="${prefix}air_pressure_link" />
-      <origin xyz="0 0 0" rpy="0 0 0" />
-    </joint>
-    <!-- base link to magnetometer frame -->
-    <joint name="${prefix}base_link_to_magnetometer_link_joint" type="fixed">
-      <parent link="${prefix}base_link" />
-      <child link="${prefix}magnetometer_link" />
-      <origin xyz="0 0 0" rpy="0 0 0" />
-    </joint>
     <!-- base link to GPS frame -->
     <joint name="${prefix}base_link_to_gps_link_joint" type="fixed">
@@ -547,28 +415,4 @@
       <child link="${prefix}rgbd_front_link" />
       <origin xyz="0.21 0 1.5" rpy="0 0.5236 0" />
-    </joint>
-    <!-- base link to front camera frame -->
-    <joint name="${prefix}base_link_to_camera_front_link_joint" type="fixed">
-      <parent link="${prefix}base_link" />
-      <child link="${prefix}camera_front_link" />
-      <origin xyz="0.24 0.06 0.405" rpy="0 0 0" />
-    </joint>
-    <!-- base link to rear camera frame -->
-    <joint name="${prefix}base_link_to_camera_rear_link_joint" type="fixed">
-      <parent link="${prefix}base_link" />
-      <child link="${prefix}camera_rear_link" />
-      <origin xyz="0.02 0 0.405" rpy="0 0 3.14159" />
-    </joint>
-    <!-- base link to left camera frame -->
-    <joint name="${prefix}base_link_to_camera_left_link_joint" type="fixed">
-      <parent link="${prefix}base_link" />
-      <child link="${prefix}camera_left_link" />
-      <origin xyz="0.13 0.11 0.405" rpy="0 0 1.5708" />
-    </joint>
-    <!-- base link to right camera frame -->
-    <joint name="${prefix}base_link_to_camera_right_link_joint" type="fixed">
-      <parent link="${prefix}base_link" />
-      <child link="${prefix}camera_right_link" />
-      <origin xyz="0.13 -0.11 0.405" rpy="0 0 -1.5708" />
     </joint>
     <!-- base link to Ouster sensor frame -->
@@ -697,42 +541,4 @@
       </sensor>
     </gazebo>
-    <gazebo reference="${prefix}air_pressure_link">
-      <sensor name="air_pressure" type="air_pressure">
-        <always_on>1</always_on>
-        <update_rate>20</update_rate>
-        <air_pressure>
-          <reference_altitude>0</reference_altitude>
-          <noise type="gaussian">
-            <mean>0.00000008</mean>
-          </noise>
-        </air_pressure>
-      </sensor>
-    </gazebo>
-    <gazebo reference="${prefix}magnetometer_link">
-      <sensor name="magnetometer" type="magnetometer">
-        <always_on>1</always_on>
-        <update_rate>50</update_rate>
-        <magnetometer>
-          <x>
-            <noise type="gaussian">
-              <mean>0.000000080</mean>
-              <bias_mean>0.000000400</bias_mean>
-            </noise>
-          </x>
-          <y>
-            <noise type="gaussian">
-              <mean>0.000000080</mean>
-              <bias_mean>0.000000400</bias_mean>
-            </noise>
-          </y>
-          <z>
-            <noise type="gaussian">
-              <mean>0.000000080</mean>
-              <bias_mean>0.000000400</bias_mean>
-            </noise>
-          </z>
-        </magnetometer>
-      </sensor>
-    </gazebo>
     <gazebo reference="${prefix}rgbd_front_link">
       <sensor name="rgbd_front" type="rgbd_camera">
@@ -781,164 +587,4 @@
       </sensor>
     </gazebo>
-    <gazebo reference="${prefix}camera_front_link">
-      <sensor name="camera_front" type="camera">
-        <always_on>1</always_on>
-        <update_rate>25</update_rate>
-        <camera name="camera_front">
-          <horizontal_fov>1.658</horizontal_fov>
-          <lens>
-            <intrinsics>
-              <fx>329.9</fx>
-              <fy>329.9</fy>
-              <cx>359.5</cx>
-              <cy>539.5</cy>
-              <s>0</s>
-            </intrinsics>
-          </lens>
-          <distortion>
-            <k1>0.0</k1>
-            <k2>0.0</k2>
-            <k3>0.0</k3>
-            <p1>0.0</p1>
-            <p2>0.0</p2>
-            <center>0.5 0.5</center>
-          </distortion>
-          <image>
-            <width>720</width>
-            <height>1080</height>
-            <format>R8G8B8</format>
-          </image>
-          <clip>
-            <near>0.01</near>
-            <far>300</far>
-          </clip>
-          <noise>
-            <type>gaussian</type>
-            <mean>0</mean>
-            <stddev>0.007</stddev>
-          </noise>
-        </camera>
-      </sensor>
-    </gazebo>
-    <gazebo reference="${prefix}camera_rear_link">
-      <sensor name="camera_rear" type="camera">
-        <always_on>1</always_on>
-        <update_rate>25</update_rate>
-        <camera name="camera_front">
-          <horizontal_fov>1.658</horizontal_fov>
-          <lens>
-            <intrinsics>
-              <fx>329.9</fx>
-              <fy>329.9</fy>
-              <cx>359.5</cx>
-              <cy>539.5</cy>
-              <s>0</s>
-            </intrinsics>
-          </lens>
-          <distortion>
-            <k1>0.0</k1>
-            <k2>0.0</k2>
-            <k3>0.0</k3>
-            <p1>0.0</p1>
-            <p2>0.0</p2>
-            <center>0.5 0.5</center>
-          </distortion>
-          <image>
-            <width>720</width>
-            <height>1080</height>
-            <format>R8G8B8</format>
-          </image>
-          <clip>
-            <near>0.01</near>
-            <far>300</far>
-          </clip>
-          <noise>
-            <type>gaussian</type>
-            <mean>0</mean>
-            <stddev>0.007</stddev>
-          </noise>
-        </camera>
-      </sensor>
-    </gazebo>
-    <gazebo reference="${prefix}camera_left_link">
-      <sensor name="camera_left" type="camera">
-        <always_on>1</always_on>
-        <update_rate>25</update_rate>
-        <camera name="camera_front">
-          <horizontal_fov>1.658</horizontal_fov>
-          <lens>
-            <intrinsics>
-              <fx>329.9</fx>
-              <fy>329.9</fy>
-              <cx>359.5</cx>
-              <cy>539.5</cy>
-              <s>0</s>
-            </intrinsics>
-          </lens>
-          <distortion>
-            <k1>0.0</k1>
-            <k2>0.0</k2>
-            <k3>0.0</k3>
-            <p1>0.0</p1>
-            <p2>0.0</p2>
-            <center>0.5 0.5</center>
-          </distortion>
-          <image>
-            <width>720</width>
-            <height>1080</height>
-            <format>R8G8B8</format>
-          </image>
-          <clip>
-            <near>0.01</near>
-            <far>300</far>
-          </clip>
-          <noise>
-            <type>gaussian</type>
-            <mean>0</mean>
-            <stddev>0.007</stddev>
-          </noise>
-        </camera>
-      </sensor>
-    </gazebo>
-    <gazebo reference="${prefix}camera_right_link">
-      <sensor name="camera_right" type="camera">
-        <always_on>1</always_on>
-        <update_rate>25</update_rate>
-        <camera name="camera_front">
-          <horizontal_fov>1.658</horizontal_fov>
-          <lens>
-            <intrinsics>
-              <fx>329.9</fx>
-              <fy>329.9</fy>
-              <cx>359.5</cx>
-              <cy>539.5</cy>
-              <s>0</s>
-            </intrinsics>
-          </lens>
-          <distortion>
-            <k1>0.0</k1>
-            <k2>0.0</k2>
-            <k3>0.0</k3>
-            <p1>0.0</p1>
-            <p2>0.0</p2>
-            <center>0.5 0.5</center>
-          </distortion>
-          <image>
-            <width>720</width>
-            <height>1080</height>
-            <format>R8G8B8</format>
-          </image>
-          <clip>
-            <near>0.01</near>
-            <far>300</far>
-          </clip>
-          <noise>
-            <type>gaussian</type>
-            <mean>0</mean>
-            <stddev>0.007</stddev>
-          </noise>
-        </camera>
-      </sensor>
-    </gazebo>
     <gazebo reference="${prefix}ouster_link">
       <sensor name="ouster_lidar" type="gpu_lidar">
