Commit message: Add gazebo dependencies, gz launch file, gz controllers, fix world attachment and controller manager name

File: cororos2_allie_description/urdf/allie.urdf.xacro (robot description, xacro)
@@ -8,13 +8,21 @@
   <xacro:arg name="sim_gazebo" default="false"/>
   <xacro:arg name="simulation_controllers" default=""/>
+  <xacro:arg name="attach_world" default="true"/>
   <xacro:include filename="$(find cororos2_allie_description)/urdf/allie/allie_macro.xacro"/>
   <xacro:include filename="$(find cororos2_allie_description)/urdf/allie/allie_macro.ros2_control.xacro"/>
-  <!-- create link fixed to the "world" -->
-  <link name="world"/>
-  <!-- Load robot's macro with parameters -->
-  <!-- set prefix if multiple robots are used -->
-  <xacro:allie prefix="$(arg prefix)" parent="world">
-    <origin xyz="0 0 0" rpy="0 0 0"/>          <!-- position robot in the world -->
-  </xacro:allie>
+  <xacro:if value="$(arg attach_world)">
+    <!-- create link fixed to the "world" -->
+    <link name="world"/>
+    <!-- Load robot's macro with parameters -->
+    <!-- set prefix if multiple robots are used -->
+    <xacro:allie prefix="$(arg prefix)" parent="world">
+      <origin xyz="0 0 0" rpy="0 0 0"/>          <!-- position robot in the world -->
+    </xacro:allie>
+  </xacro:if>
+  <xacro:unless value="$(arg attach_world)">
+    <xacro:allie prefix="$(arg prefix)" parent="">
+      <origin xyz="0 0 0" rpy="0 0 0"/>
+    </xacro:allie>
+  </xacro:unless>
   <xacro:allie_ros2_control
     name="allie"

File: cororos2_allie_description/urdf/allie/allie_macro.ros2_control.xacro (robot description, xacro)
@@ -65,5 +65,5 @@
         <plugin filename="gz_ros2_control-system" name="gz_ros2_control::GazeboSimROS2ControlPlugin">
           <parameters>${simulation_controllers}</parameters>
-          <controller_manager_node_name>b_controlled_box_cm</controller_manager_node_name>
+          <controller_manager_node_name>controller_manager</controller_manager_node_name>
         </plugin>
       </gazebo>

File: cororos2_allie_description/urdf/allie/allie_macro.xacro (robot description, xacro)
@@ -471,14 +471,16 @@
     <!-- base joints -->
     <!-- world to base footprint -->
-    <joint name="${prefix}base_joint" type="fixed">
-      <xacro:insert_block name="origin" />
-      <parent link="${parent}" />
-      <child link="${prefix}base_footprint" />
-    </joint>
+    <xacro:if value="${parent != ''}">
+      <joint name="${prefix}base_joint" type="fixed">
+        <xacro:insert_block name="origin" />
+        <parent link="${parent}" />
+        <child link="${prefix}base_footprint" />
+      </joint>
+    </xacro:if>
     <!-- base footprint to base link -->
     <joint name="${prefix}base_footprint_to_base_link" type="fixed">
       <parent link="${prefix}base_footprint" />
       <child link="${prefix}base_link" />
-      <origin xyz="0 0 0.1275" rpy="0 0 0" />
+      <origin xyz="0 0 0.205" rpy="0 0 0" />
     </joint>
     <!-- wheel joints -->
