Commit message: Convert Cornelius description package to URDF and package meshes

File: cororos2_cornelius_description/urdf/cornelius.urdf.xacro (robot description, xacro)
@@ -1,5 +1,4 @@
 <?xml version="1.0" encoding="UTF-8"?>
 <robot xmlns:xacro="http://wiki.ros.org/xacro" name="cornelius">
-  <!-- Use this if parameters are set from the launch file, otherwise delete -->
   <xacro:arg name="prefix" default=""/>
   <xacro:arg name="use_mock_hardware" default="false"/>
@@ -8,13 +7,18 @@
   <xacro:arg name="sim_gazebo" default="false"/>
   <xacro:arg name="simulation_controllers" default=""/>
+  <xacro:arg name="attach_world" default="true"/>
   <xacro:include filename="$(find cororos2_cornelius_description)/urdf/cornelius/cornelius_macro.xacro"/>
   <xacro:include filename="$(find cororos2_cornelius_description)/urdf/cornelius/cornelius_macro.ros2_control.xacro"/>
-  <!-- create link fixed to the "world" -->
-  <link name="world"/>
-  <!-- Load robot's macro with parameters -->
-  <!-- set prefix if multiple robots are used -->
-  <xacro:cornelius prefix="$(arg prefix)" parent="world">
-    <origin xyz="0 0 0" rpy="0 0 0"/>          <!-- position robot in the world -->
-  </xacro:cornelius>
+  <xacro:if value="$(arg attach_world)">
+    <link name="world"/>
+    <xacro:cornelius prefix="$(arg prefix)" parent="world">
+      <origin xyz="0 0 0" rpy="0 0 0"/>
+    </xacro:cornelius>
+  </xacro:if>
+  <xacro:unless value="$(arg attach_world)">
+    <xacro:cornelius prefix="$(arg prefix)" parent="">
+      <origin xyz="0 0 0" rpy="0 0 0"/>
+    </xacro:cornelius>
+  </xacro:unless>
   <xacro:cornelius_ros2_control
     name="cornelius"

File: cororos2_cornelius_description/urdf/cornelius/cornelius_macro.ros2_control.xacro (robot description, xacro)
@@ -8,131 +8,5 @@
                sim_gazebo_classic:=false
                sim_gazebo:=false
-               simulation_controllers"
-               >
-    <ros2_control name="${name}" type="system">
-      <hardware>
-        <xacro:if value="${use_mock_hardware}">
-          <plugin>mock_components/GenericSystem</plugin>
-          <param name="mock_sensor_commands">${mock_sensor_commands}</param>
-        </xacro:if>
-        <xacro:if value="${sim_gazebo_classic}">
-          <plugin>gazebo_ros2_control/GazeboSystem</plugin>
-        </xacro:if>
-        <xacro:if value="${sim_gazebo}">
-          <plugin>gz_ros2_control/GazeboSimSystem</plugin>
-        </xacro:if>
-        <xacro:unless value="${use_mock_hardware or sim_gazebo_classic or sim_gazebo}">
-          <plugin>robot_hardware_interface/RobotHardwareInterface</plugin>
-        </xacro:unless>
-      </hardware>
-      <joint name="${prefix}joint1">
-        <command_interface name="position">     <!-- Add/Remove interfaces as needed -->
-          <param name="min">-1</param>
-          <param name="max">1</param>
-        </command_interface>
-        <state_interface name="position">
-          <param name="initial_value">0.0</param>
-        </state_interface>
-        <state_interface name="velocity"/>
-        <state_interface name="acceleration"/>
-      </joint>
-      <joint name="${prefix}joint2">
-        <command_interface name="position">     <!-- Add/Remove interfaces as needed -->
-          <param name="min">-1</param>
-          <param name="max">1</param>
-        </command_interface>
-        <state_interface name="position">
-          <param name="initial_value">0.0</param>
-        </state_interface>
-        <state_interface name="velocity"/>
-        <state_interface name="acceleration"/>
-      </joint>
-      <joint name="${prefix}joint3">
-        <command_interface name="position">     <!-- Add/Remove interfaces as needed -->
-          <param name="min">-1</param>
-          <param name="max">1</param>
-        </command_interface>
-        <state_interface name="position">
-          <param name="initial_value">0.0</param>
-        </state_interface>
-        <state_interface name="velocity"/>
-        <state_interface name="acceleration"/>
-      </joint>
-      <joint name="${prefix}joint4">
-        <command_interface name="position">     <!-- Add/Remove interfaces as needed -->
-          <param name="min">-1</param>
-          <param name="max">1</param>
-        </command_interface>
-        <state_interface name="position">
-          <param name="initial_value">0.0</param>
-        </state_interface>
-        <state_interface name="velocity"/>
-        <state_interface name="acceleration"/>
-      </joint>
-      <joint name="${prefix}joint5">
-        <command_interface name="position">     <!-- Add/Remove interfaces as needed -->
-          <param name="min">-1</param>
-          <param name="max">1</param>
-        </command_interface>
-        <state_interface name="position">
-          <param name="initial_value">0.0</param>
-        </state_interface>
-        <state_interface name="velocity"/>
-        <state_interface name="acceleration"/>
-      </joint>
-      <joint name="${prefix}joint6">
-        <command_interface name="position">     <!-- Add/Remove interfaces as needed -->
-          <param name="min">-1</param>
-          <param name="max">1</param>
-        </command_interface>
-        <state_interface name="position">
-          <param name="initial_value">0.0</param>
-        </state_interface>
-        <state_interface name="velocity"/>
-        <state_interface name="acceleration"/>
-      </joint>
-      <sensor name="tcp_fts_sensor">            <!-- Remove/change sensors as needed -->
-        <state_interface name="fx"/>
-        <state_interface name="fy"/>
-        <state_interface name="fz"/>
-        <state_interface name="tx"/>
-        <state_interface name="ty"/>
-        <state_interface name="tz"/>
-        <param name="frame_id">tool0</param>    <!-- Change sensors as needed -->
-        <param name="min_fx">-100</param>
-        <param name="max_fx">100</param>
-        <param name="min_fy">-100</param>
-        <param name="max_fy">100</param>
-        <param name="min_fz">-200</param>
-        <param name="max_fz">200</param>
-        <param name="min_tx">-10</param>
-        <param name="max_tx">10</param>
-        <param name="min_ty">-10</param>
-        <param name="max_ty">10</param>
-        <param name="min_tz">-15</param>
-        <param name="max_tz">15</param>
-      </sensor>
-    </ros2_control>
-    <xacro:if value="$(arg sim_gazebo_classic)">
-      <!-- Gazebo plugins -->
-      <gazebo reference="world">
-      </gazebo>
-      <gazebo>
-        <plugin filename="libgazebo_ros2_control.so" name="gazebo_ros2_control">
-          <parameters>${simulation_controllers}</parameters>
-        </plugin>
-      </gazebo>
-    </xacro:if>
-    <xacro:if value="$(arg sim_gazebo)">
-      <!-- Gazebo plugins -->
-      <gazebo reference="world">
-      </gazebo>
-      <gazebo>
-        <plugin filename="gz_ros2_control-system" name="gz_ros2_control::GazeboSimROS2ControlPlugin">
-          <parameters>${simulation_controllers}</parameters>
-          <controller_manager_node_name>${prefix}controller_manager</controller_manager_node_name>
-        </plugin>
-      </gazebo>
-    </xacro:if>
+               simulation_controllers">
   </xacro:macro>
 </robot>

File: cororos2_cornelius_description/urdf/cornelius/cornelius_macro.xacro (robot description, xacro)
@@ -1,244 +1,1115 @@
-<?xml version="1.0" encoding="UTF-8"?>
+<?xml version='1.0' encoding='utf-8'?>
 <robot xmlns:xacro="http://wiki.ros.org/xacro">
-  <xacro:include filename="$(find cororos2_cornelius_description)/urdf/common/inertials.xacro"/>
-  <xacro:include filename="$(find cororos2_cornelius_description)/urdf/common/materials.xacro"/>
   <xacro:macro name="cornelius" params="prefix parent *origin">
     <!-- LINKS -->
+    <!-- base footprint -->
+    <link name="${prefix}base_footprint">
+    </link>
     <!-- base link -->
     <link name="${prefix}base_link">
-      <!-- Default inertial for Gazebo - copy and edit block from 'common.xacro'
-           to get more realistic behavior -->
-      <xacro:default_inertial/>
-      <visual>
-        <origin xyz="0 0 0" rpy="0 0 0"/>
-        <geometry>
-          <cylinder length="0.3" radius="0.3"/>
-          <!--           <mesh filename="package://cororos2_cornelius_description/meshes/cornelius/visual/base_link.dae" /> -->
-        </geometry>
-        <material name="black"/>
-      </visual>
-      <collision>
-        <origin xyz="0 0 0" rpy="0 0 0"/>
-        <geometry>
-          <cylinder length="0.3" radius="0.3"/>
-          <!--           <mesh filename="package://cororos2_cornelius_description/meshes/cornelius/collision/base_link.stl" /> -->
+      <inertial>
+        <origin xyz="-0.000649 -0.084945 0.062329" rpy="0 0 0" />
+        <mass value="21.8194" />
+        <inertia ixx="0.615397" ixy="-0.0240585" ixz="-0.120749" iyy="1.75388" iyz="-0.0028322" izz="2.03641" />
+      </inertial>
+      <collision name="base_link_collision_top">
+        <origin xyz="0 0 0.12" rpy="0 0 0" />
+        <geometry>
+          <box size="0.9874 0.5709 0.05" />
         </geometry>
       </collision>
-    </link>
-    <!-- link 1 -->
-    <link name="${prefix}link1">
-      <!-- Default inertial for Gazebo - copy and edit block from 'common.xacro'
-           to get more realistic behavior -->
-      <xacro:default_inertial/>
-      <visual>
-        <origin xyz="0 0 0" rpy="0 0 0"/>
-        <geometry>
-          <cylinder length="0.3" radius="0.15"/>
-          <!--           <mesh filename="package://cororos2_cornelius_description/meshes/cornelius/visual/link1.dae" /> -->
-        </geometry>
-        <material name="blue"/>
-      </visual>
-      <collision>
-        <origin xyz="0 0 0" rpy="0 0 0"/>
-        <geometry>
-          <cylinder length="0.3" radius="0.15"/>
-          <!--           <mesh filename="package://cororos2_cornelius_description/meshes/cornelius/collision/link1.stl" /> -->
-        </geometry>
-        <material name="green"/>
+      <collision name="base_link_collision_bottom">
+        <origin xyz="0 0 0.046" rpy="0 0 0" />
+        <geometry>
+          <box size="0.80 0.5709 0.2" />
+        </geometry>
       </collision>
-    </link>
-    <!-- link 2 -->
-    <link name="${prefix}link2">
-      <!-- Default inertial for Gazebo - copy and edit block from 'common.xacro'
-           to get more realistic behavior-->
-      <xacro:default_inertial/>
-      <visual>
-        <origin xyz="0 0 0" rpy="0 0 0"/>
-        <geometry>
-          <cylinder length="0.3" radius="0.15"/>
-          <!--           <mesh filename="package://cororos2_cornelius_description/meshes/cornelius/visual/link2.dae" /> -->
-        </geometry>
-        <material name="grey"/>
-      </visual>
-      <collision>
-        <origin xyz="0 0 0" rpy="0 0 0"/>
-        <geometry>
-          <cylinder length="0.3" radius="0.15"/>
-          <!--           <mesh filename="package://cororos2_cornelius_description/meshes/cornelius/collision/link2.stl"  /> -->
+      <collision name="base_link_collision_mid">
+        <origin xyz="0 0 0.185625" rpy="0 0 0" />
+        <geometry>
+          <box size="0.78992 0.5709 0.12375" />
         </geometry>
       </collision>
-    </link>
-    <!-- link 3 -->
-    <link name="${prefix}link3">
-      <!-- Default inertial for Gazebo - copy and edit block from 'common.xacro'
-           to get more realistic behavior-->
-      <xacro:default_inertial/>
-      <visual>
-        <origin xyz="0 0 0" rpy="0 0 0"/>
-        <geometry>
-          <cylinder length="0.2" radius="0.1"/>
-          <!--           <mesh filename="package://cororos2_cornelius_description/meshes/cornelius/visual/link3.dae" /> -->
-        </geometry>
-        <material name="orange"/>
-      </visual>
-      <collision>
-        <origin xyz="0 0 0" rpy="0 0 0"/>
-        <geometry>
-          <cylinder length="0.2" radius="0.1"/>
-          <!--           <mesh filename="package://cororos2_cornelius_description/meshes/cornelius/collision/link3.stl"  /> -->
+      <collision name="tower_collision_1">
+        <origin xyz="0.19 0 0.24" rpy="0 0 0" />
+        <geometry>
+          <box size="0.2 0.2 0.34" />
         </geometry>
       </collision>
-    </link>
-    <!-- link 4 -->
-    <link name="${prefix}link4">
-      <!-- Default inertial for Gazebo - copy and edit block from 'common.xacro'
-           to get more realistic behavior-->
-      <xacro:default_inertial/>
-      <visual>
-        <origin xyz="0 0 0" rpy="0 0 0"/>
-        <geometry>
-          <cylinder length="0.1" radius="0.1"/>
-          <!--           <mesh filename="package://cororos2_cornelius_description/meshes/cornelius/visual/link4.dae" /> -->
-        </geometry>
-        <material name="brown"/>
-      </visual>
-      <collision>
-        <origin xyz="0 0 0" rpy="0 0 0"/>
-        <geometry>
-          <cylinder length="0.1" radius="0.1"/>
-          <!--           <mesh filename="package://cororos2_cornelius_description/meshes/cornelius/collision/link4.stl"  /> -->
+      <visual name="body_visual">
+        <origin xyz="0 0 -0.135" rpy="0 0 1.57" />
+        <geometry>
+          <mesh filename="package://cororos2_cornelius_description/meshes/cornelius/visual/hd2_marble_base_body_metric.dae" />
+        </geometry>
+        <material name="body_visual_mat">
+          <color rgba="1.0 1.0 1.0 1.0" />
+        </material>
+      </visual>
+      <visual name="plate1_visual">
+        <origin xyz="0.19 0 0.38" rpy="0 0 0" />
+        <geometry>
+          <box size="0.2 0.2 0.005" />
+        </geometry>
+        <material name="plate1_visual_mat">
+          <color rgba="0.7843 0.7843 0.7843 1.0" />
+        </material>
+      </visual>
+      <visual name="plate2_visual">
+        <origin xyz="0.19 0 0.27" rpy="0 0 0" />
+        <geometry>
+          <box size="0.2 0.2 0.005" />
+        </geometry>
+        <material name="plate2_visual_mat">
+          <color rgba="0.7843 0.7843 0.7843 1.0" />
+        </material>
+      </visual>
+      <visual name="plate3_visual">
+        <origin xyz="0.19 0 0.08" rpy="0 0 0" />
+        <geometry>
+          <box size="0.2 0.2 0.005" />
+        </geometry>
+        <material name="plate3_visual_mat">
+          <color rgba="0.9412 0.9412 0.9412 1.0" />
+        </material>
+      </visual>
+      <visual name="beam1_visual">
+        <origin xyz="0.281 0.091 0.23" rpy="0 0 0" />
+        <geometry>
+          <box size="0.02 0.02 0.3" />
+        </geometry>
+        <material name="beam1_visual_mat">
+          <color rgba="0.7843 0.7843 0.7843 1.0" />
+        </material>
+      </visual>
+      <visual name="beam2_visual">
+        <origin xyz="0.281 -0.091 0.23" rpy="0 0 0" />
+        <geometry>
+          <box size="0.02 0.02 0.3" />
+        </geometry>
+        <material name="beam2_visual_mat">
+          <color rgba="0.7843 0.7843 0.7843 1.0" />
+        </material>
+      </visual>
+      <visual name="beam3_visual">
+        <origin xyz="0.099 0.091 0.23" rpy="0 0 0" />
+        <geometry>
+          <box size="0.02 0.02 0.3" />
+        </geometry>
+        <material name="beam3_visual_mat">
+          <color rgba="0.7843 0.7843 0.7843 1.0" />
+        </material>
+      </visual>
+      <visual name="beam4_visual">
+        <origin xyz="0.099 -0.091 0.23" rpy="0 0 0" />
+        <geometry>
+          <box size="0.02 0.02 0.3" />
+        </geometry>
+        <material name="beam4_visual_mat">
+          <color rgba="0.7843 0.7843 0.7843 1.0" />
+        </material>
+      </visual>
+    </link>
+    <!-- wheel links -->
+    <!-- left track body -->
+    <link name="${prefix}left_track">
+      <inertial>
+        <origin xyz="0 0 0" rpy="0 0 0" />
+        <mass value="4.0" />
+        <inertia ixx="0.02" ixy="0" ixz="0" iyy="0.18" iyz="0" izz="0.16" />
+      </inertial>
+      <collision name="left_track_box_collision">
+        <origin xyz="0 0 0" rpy="0 0 0" />
+        <geometry>
+          <box size="0.72 0.1 0.258" />
         </geometry>
       </collision>
-    </link>
-    <!-- link 5 -->
-    <link name="${prefix}link5">
-      <!-- Default inertial for Gazebo - copy and edit block from 'common.xacro'
-           to get more realistic behavior-->
-      <xacro:default_inertial/>
-      <visual>
-        <origin xyz="0 0 0" rpy="0 0 0"/>
-        <geometry>
-          <cylinder length="0.15" radius="0.1"/>
-          <!--           <mesh filename="package://cororos2_cornelius_description/meshes/cornelius/visual/link5.dae" /> -->
-        </geometry>
-        <material name="red"/>
-      </visual>
-      <collision>
-        <origin xyz="0 0 0" rpy="0 0 0"/>
-        <geometry>
-          <cylinder length="0.15" radius="0.1"/>
-          <!--           <mesh filename="package://cororos2_cornelius_description/meshes/cornelius/collision/link5.stl" /> -->
+      <visual name="left_track_body_visual">
+        <origin xyz="0 0 0" rpy="0 0 0" />
+        <geometry>
+          <box size="0.72 0.1 0.258" />
+        </geometry>
+        <material name="left_track_body_visual_mat">
+          <color rgba="0.08 0.08 0.08 1.0" />
+        </material>
+      </visual>
+    </link>
+    <!-- left rear drive roller -->
+    <link name="${prefix}left_rear_drive_roller">
+      <inertial>
+        <origin xyz="0 0 0" rpy="0 0 0" />
+        <mass value="1.0" />
+        <inertia ixx="0.01" ixy="0" ixz="0" iyy="0.01" iyz="0" izz="0.006" />
+      </inertial>
+      <collision name="left_rear_drive_roller_collision">
+        <origin xyz="0 0 0" rpy="1.5707963267948966 0 0" />
+        <geometry>
+          <cylinder radius="0.129" length="0.1" />
         </geometry>
       </collision>
-    </link>
-    <!-- link 6 -->
-    <link name="${prefix}link6">
-      <!-- Default inertial for Gazebo - copy and edit block from 'common.xacro'
-           to get more realistic behavior-->
-      <xacro:default_inertial/>
-      <visual>
-        <origin xyz="0 0 0" rpy="0 0 0"/>
-        <geometry>
-          <cylinder length="0.05" radius="0.075"/>
-          <!--           <mesh filename="package://cororos2_cornelius_description/meshes/cornelius/visual/link6.dae" /> -->
-        </geometry>
-        <material name="white"/>
-      </visual>
-      <collision>
-        <origin xyz="0 0 0" rpy="0 0 0"/>
-        <geometry>
-          <cylinder length="0.05" radius="0.075"/>
-          <!--           <mesh filename="package://cororos2_cornelius_description/meshes/cornelius/collision/link6.stl" /> -->
+      <visual name="left_rear_drive_roller_visual">
+        <origin xyz="0 0 0" rpy="1.5707963267948966 0 0" />
+        <geometry>
+          <cylinder radius="0.129" length="0.1" />
+        </geometry>
+        <material name="left_rear_drive_roller_visual_mat">
+          <color rgba="0.12 0.12 0.12 1.0" />
+        </material>
+      </visual>
+    </link>
+    <!-- left front idler roller -->
+    <link name="${prefix}left_front_idler">
+      <inertial>
+        <origin xyz="0 0 0" rpy="0 0 0" />
+        <mass value="1.0" />
+        <inertia ixx="0.01" ixy="0" ixz="0" iyy="0.01" iyz="0" izz="0.006" />
+      </inertial>
+      <collision name="left_front_idler_collision">
+        <origin xyz="0 0 0" rpy="1.5707963267948966 0 0" />
+        <geometry>
+          <cylinder radius="0.129" length="0.1" />
         </geometry>
       </collision>
-    </link>
-    <!-- All-zero tool frame. This frame should correspond to the TOOL frame of the robot's controller.) -->
-    <link name="${prefix}tool0"/>
-    <!-- tool link -->
-    <!-- START Delete if not needed -->
-    <!-- Standard frames for industrial robots. Also useful for manipulators.
-         (ROS-I specs - https://wiki.ros.org/Industrial/Tutorials/WorkingWithRosIndustrialRobotSupportPackages#Standardised_links_.2F_frames)-->
-    <!-- This frame should correspond to the BASE coordinate system of robot's controller.) -->
-    <link name="${prefix}base"/>
-    <!-- Frame for mounting EEF models to a manipulator. x+ axis points forward (REP 103). -->
-    <link name="${prefix}flange"/>
-    <!-- END Delete if not needed  -->
-    <!-- END LINKS -->
+      <visual name="left_front_idler_visual">
+        <origin xyz="0 0 0" rpy="1.5707963267948966 0 0" />
+        <geometry>
+          <cylinder radius="0.129" length="0.1" />
+        </geometry>
+        <material name="left_front_idler_visual_mat">
+          <color rgba="0.12 0.12 0.12 1.0" />
+        </material>
+      </visual>
+    </link>
+    <!-- right track body -->
+    <link name="${prefix}right_track">
+      <inertial>
+        <origin xyz="0 0 0" rpy="0 0 0" />
+        <mass value="4.0" />
+        <inertia ixx="0.02" ixy="0" ixz="0" iyy="0.18" iyz="0" izz="0.16" />
+      </inertial>
+      <collision name="right_track_box_collision">
+        <origin xyz="0 0 0" rpy="0 0 0" />
+        <geometry>
+          <box size="0.72 0.1 0.258" />
+        </geometry>
+      </collision>
+      <visual name="right_track_body_visual">
+        <origin xyz="0 0 0" rpy="0 0 0" />
+        <geometry>
+          <box size="0.72 0.1 0.258" />
+        </geometry>
+        <material name="right_track_body_visual_mat">
+          <color rgba="0.08 0.08 0.08 1.0" />
+        </material>
+      </visual>
+    </link>
+    <!-- right rear drive roller -->
+    <link name="${prefix}right_rear_drive_roller">
+      <inertial>
+        <origin xyz="0 0 0" rpy="0 0 0" />
+        <mass value="1.0" />
+        <inertia ixx="0.01" ixy="0" ixz="0" iyy="0.01" iyz="0" izz="0.006" />
+      </inertial>
+      <collision name="right_rear_drive_roller_collision">
+        <origin xyz="0 0 0" rpy="1.5707963267948966 0 0" />
+        <geometry>
+          <cylinder radius="0.129" length="0.1" />
+        </geometry>
+      </collision>
+      <visual name="right_rear_drive_roller_visual">
+        <origin xyz="0 0 0" rpy="1.5707963267948966 0 0" />
+        <geometry>
+          <cylinder radius="0.129" length="0.1" />
+        </geometry>
+        <material name="right_rear_drive_roller_visual_mat">
+          <color rgba="0.12 0.12 0.12 1.0" />
+        </material>
+      </visual>
+    </link>
+    <!-- right front idler roller -->
+    <link name="${prefix}right_front_idler">
+      <inertial>
+        <origin xyz="0 0 0" rpy="0 0 0" />
+        <mass value="1.0" />
+        <inertia ixx="0.01" ixy="0" ixz="0" iyy="0.01" iyz="0" izz="0.006" />
+      </inertial>
+      <collision name="right_front_idler_collision">
+        <origin xyz="0 0 0" rpy="1.5707963267948966 0 0" />
+        <geometry>
+          <cylinder radius="0.129" length="0.1" />
+        </geometry>
+      </collision>
+      <visual name="right_front_idler_visual">
+        <origin xyz="0 0 0" rpy="1.5707963267948966 0 0" />
+        <geometry>
+          <cylinder radius="0.129" length="0.1" />
+        </geometry>
+        <material name="right_front_idler_visual_mat">
+          <color rgba="0.12 0.12 0.12 1.0" />
+        </material>
+      </visual>
+    </link>
+    <!-- sensor and light frames -->
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