Commit message: Remove weird lighting and links, change lidar color in gazebo and add support skids

File: cororos2_cornelius_description/urdf/cornelius/cornelius_macro.xacro (robot description, xacro)
@@ -238,4 +238,31 @@
       </collision>
     </link>
+    <!-- hidden support contacts prevent the chassis from pitching onto the floor -->
+    <link name="${prefix}front_support_skid">
+      <inertial>
+        <origin xyz="0 0 0" rpy="0 0 0" />
+        <mass value="1e-6" />
+        <inertia ixx="1e-9" ixy="0" ixz="0" iyy="1e-9" iyz="0" izz="1e-9" />
+      </inertial>
+      <collision name="front_support_skid_collision">
+        <origin xyz="0 0 0" rpy="0 0 0" />
+        <geometry>
+          <sphere radius="0.03" />
+        </geometry>
+      </collision>
+    </link>
+    <link name="${prefix}rear_support_skid">
+      <inertial>
+        <origin xyz="0 0 0" rpy="0 0 0" />
+        <mass value="1e-6" />
+        <inertia ixx="1e-9" ixy="0" ixz="0" iyy="1e-9" iyz="0" izz="1e-9" />
+      </inertial>
+      <collision name="rear_support_skid_collision">
+        <origin xyz="0 0 0" rpy="0 0 0" />
+        <geometry>
+          <sphere radius="0.03" />
+        </geometry>
+      </collision>
+    </link>
     <!-- sensor and light frames -->
     <!-- IMU frame -->
@@ -282,5 +309,5 @@
         </geometry>
         <material name="vlp16_visual1_mat">
-          <color rgba="1.0 1.0 1.0 1.0" />
+          <color rgba="0.02 0.02 0.02 1.0" />
         </material>
       </visual>
@@ -291,5 +318,5 @@
         </geometry>
         <material name="vlp16_visual2_mat">
-          <color rgba="1.0 1.0 1.0 1.0" />
+          <color rgba="0.02 0.02 0.02 1.0" />
         </material>
       </visual>
@@ -300,5 +327,5 @@
         </geometry>
         <material name="vlp16_visual3_mat">
-          <color rgba="1.0 1.0 1.0 1.0" />
+          <color rgba="0.02 0.02 0.02 1.0" />
         </material>
       </visual>
@@ -311,72 +338,4 @@
         <inertia ixx="1e-9" ixy="0" ixz="0" iyy="1e-9" iyz="0" izz="1e-9" />
       </inertial>
-    </link>
-    <!-- front light frame -->
-    <link name="${prefix}light_front_link">
-      <inertial>
-        <origin xyz="0 0 0" rpy="0 0 0" />
-        <mass value="1e-6" />
-        <inertia ixx="1e-9" ixy="0" ixz="0" iyy="1e-9" iyz="0" izz="1e-9" />
-      </inertial>
-      <visual name="light_front_visual">
-        <origin xyz="0 0 0" rpy="0 0 0" />
-        <geometry>
-          <box size="0.04 0.13 0.04" />
-        </geometry>
-        <material name="light_front_visual_mat">
-          <color rgba="0.0 0.0 0.0 1.0" />
-        </material>
-      </visual>
-    </link>
-    <!-- rear light frame -->
-    <link name="${prefix}light_rear_link">
-      <inertial>
-        <origin xyz="0 0 0" rpy="0 0 0" />
-        <mass value="1e-6" />
-        <inertia ixx="1e-9" ixy="0" ixz="0" iyy="1e-9" iyz="0" izz="1e-9" />
-      </inertial>
-      <visual name="light_rear_visual">
-        <origin xyz="0 0 0" rpy="0 0 0" />
-        <geometry>
-          <box size="0.04 0.12 0.04" />
-        </geometry>
-        <material name="light_rear_visual_mat">
-          <color rgba="0.0 0.0 0.0 1.0" />
-        </material>
-      </visual>
-    </link>
-    <!-- left light frame -->
-    <link name="${prefix}light_left_link">
-      <inertial>
-        <origin xyz="0 0 0" rpy="0 0 0" />
-        <mass value="1e-6" />
-        <inertia ixx="1e-9" ixy="0" ixz="0" iyy="1e-9" iyz="0" izz="1e-9" />
-      </inertial>
-      <visual name="light_left_visual">
-        <origin xyz="0 0 0" rpy="0 0 0" />
-        <geometry>
-          <box size="0.12 0.04 0.04" />
-        </geometry>
-        <material name="light_left_visual_mat">
-          <color rgba="0.0 0.0 0.0 1.0" />
-        </material>
-      </visual>
-    </link>
-    <!-- right light frame -->
-    <link name="${prefix}light_right_link">
-      <inertial>
-        <origin xyz="0 0 0" rpy="0 0 0" />
-        <mass value="1e-6" />
-        <inertia ixx="1e-9" ixy="0" ixz="0" iyy="1e-9" iyz="0" izz="1e-9" />
-      </inertial>
-      <visual name="light_right_visual">
-        <origin xyz="0 0 0" rpy="0 0 0" />
-        <geometry>
-          <box size="0.12 0.04 0.04" />
-        </geometry>
-        <material name="light_right_visual_mat">
-          <color rgba="0.0 0.0 0.0 1.0" />
-        </material>
-      </visual>
     </link>
     <!-- JOINTS -->
@@ -417,4 +376,14 @@
       <axis xyz="0 1 0" />
     </joint>
+    <joint name="${prefix}base_link_to_front_support_skid_joint" type="fixed">
+      <parent link="${prefix}base_link" />
+      <child link="${prefix}front_support_skid" />
+      <origin xyz="0.30 0 -0.099" rpy="0 0 0" />
+    </joint>
+    <joint name="${prefix}base_link_to_rear_support_skid_joint" type="fixed">
+      <parent link="${prefix}base_link" />
+      <child link="${prefix}rear_support_skid" />
+      <origin xyz="-0.30 0 -0.099" rpy="0 0 0" />
+    </joint>
     <!-- sensor and light frame joints -->
     <joint name="${prefix}base_link_to_imu_sensor_link_joint" type="fixed">
@@ -442,24 +411,4 @@
       <child link="${prefix}ouster_imu_link" />
       <origin xyz="0 0 0" rpy="0 0 0" />
-    </joint>
-    <joint name="${prefix}base_link_to_light_front_link_joint" type="fixed">
-      <parent link="${prefix}base_link" />
-      <child link="${prefix}light_front_link" />
-      <origin xyz="0.28 0 0.402" rpy="0 0 0" />
-    </joint>
-    <joint name="${prefix}base_link_to_light_rear_link_joint" type="fixed">
-      <parent link="${prefix}base_link" />
-      <child link="${prefix}light_rear_link" />
-      <origin xyz="0.10 0 0.402" rpy="0 0 0" />
-    </joint>
-    <joint name="${prefix}base_link_to_light_left_link_joint" type="fixed">
-      <parent link="${prefix}base_link" />
-      <child link="${prefix}light_left_link" />
-      <origin xyz="0.19 0.09 0.402" rpy="0 0 0" />
-    </joint>
-    <joint name="${prefix}base_link_to_light_right_link_joint" type="fixed">
-      <parent link="${prefix}base_link" />
-      <child link="${prefix}light_right_link" />
-      <origin xyz="0.19 -0.09 0.402" rpy="0 0 0" />
     </joint>
     <!-- GAZEBO EXTENSIONS -->
@@ -643,84 +592,15 @@
       <kd>100.0</kd>
     </gazebo>
-    <!-- light definitions -->
-    <gazebo reference="${prefix}light_front_link">
-      <light name="light_front" type="spot">
-        <pose>0.03 0 0 0 -1.5707963267948966 0</pose>
-        <attenuation>
-          <range>25</range>
-          <linear>0</linear>
-          <constant>0.1</constant>
-          <quadratic>0.005</quadratic>
-        </attenuation>
-        <diffuse>0.8 0.8 0.5 1.0</diffuse>
-        <specular>0.8 0.8 0.5 1</specular>
-        <spot>
-          <inner_angle>1.571</inner_angle>
-          <outer_angle>2.1</outer_angle>
-          <falloff>1</falloff>
-        </spot>
-        <direction>1 0 0</direction>
-        <cast_shadows>1</cast_shadows>
-      </light>
-    </gazebo>
-    <gazebo reference="${prefix}light_rear_link">
-      <light name="light_rear" type="spot">
-        <pose>-0.03 0 0 0 1.5707963267948966 0</pose>
-        <attenuation>
-          <range>25</range>
-          <linear>0</linear>
-          <constant>0.1</constant>
-          <quadratic>0.005</quadratic>
-        </attenuation>
-        <diffuse>0.8 0.8 0.5 1.0</diffuse>
-        <specular>0.8 0.8 0.5 1</specular>
-        <spot>
-          <inner_angle>1.571</inner_angle>
-          <outer_angle>2.1</outer_angle>
-          <falloff>1</falloff>
-        </spot>
-        <direction>1 0 0</direction>
-        <cast_shadows>1</cast_shadows>
-      </light>
-    </gazebo>
-    <gazebo reference="${prefix}light_left_link">
-      <light name="light_left" type="spot">
-        <pose>0 0.03 0 1.5707963267948966 0 0</pose>
-        <attenuation>
-          <range>25</range>
-          <linear>0</linear>
-          <constant>0.1</constant>
-          <quadratic>0.005</quadratic>
-        </attenuation>
-        <diffuse>0.8 0.8 0.5 1.0</diffuse>
-        <specular>0.8 0.8 0.5 1</specular>
-        <spot>
-          <inner_angle>1.571</inner_angle>
-          <outer_angle>2.1</outer_angle>
-          <falloff>1</falloff>
-        </spot>
-        <direction>1 0 0</direction>
-        <cast_shadows>1</cast_shadows>
-      </light>
-    </gazebo>
-    <gazebo reference="${prefix}light_right_link">
-      <light name="light_right" type="spot">
-        <pose>0 -0.03 0 -1.5707963267948966 0 0</pose>
-        <attenuation>
-          <range>25</range>
-          <linear>0</linear>
-          <constant>0.1</constant>
-          <quadratic>0.005</quadratic>
-        </attenuation>
-        <diffuse>0.8 0.8 0.5 1.0</diffuse>
-        <specular>0.8 0.8 0.5 1</specular>
-        <spot>
-          <inner_angle>1.571</inner_angle>
-          <outer_angle>2.1</outer_angle>
-          <falloff>1</falloff>
-        </spot>
-        <direction>1 0 0</direction>
-        <cast_shadows>1</cast_shadows>
-      </light>
+    <gazebo reference="${prefix}front_support_skid">
+      <mu1>0.05</mu1>
+      <mu2>0.05</mu2>
+      <kp>1000000.0</kp>
+      <kd>100.0</kd>
+    </gazebo>
+    <gazebo reference="${prefix}rear_support_skid">
+      <mu1>0.05</mu1>
+      <mu2>0.05</mu2>
+      <kp>1000000.0</kp>
+      <kd>100.0</kd>
     </gazebo>
   </xacro:macro>
