Commit message: Add joe meshes, view launch file and the URDF in the same style as Allie and Cornelius

File: cororos2_joe_description/urdf/joe.urdf.xacro (robot description, xacro)
@@ -1,5 +1,4 @@
 <?xml version="1.0" encoding="UTF-8"?>
 <robot xmlns:xacro="http://wiki.ros.org/xacro" name="joe">
-  <!-- Use this if parameters are set from the launch file, otherwise delete -->
   <xacro:arg name="prefix" default=""/>
   <xacro:arg name="use_mock_hardware" default="false"/>
@@ -8,13 +7,18 @@
   <xacro:arg name="sim_gazebo" default="false"/>
   <xacro:arg name="simulation_controllers" default=""/>
+  <xacro:arg name="attach_world" default="true"/>
   <xacro:include filename="$(find cororos2_joe_description)/urdf/joe/joe_macro.xacro"/>
   <xacro:include filename="$(find cororos2_joe_description)/urdf/joe/joe_macro.ros2_control.xacro"/>
-  <!-- create link fixed to the "world" -->
-  <link name="world"/>
-  <!-- Load robot's macro with parameters -->
-  <!-- set prefix if multiple robots are used -->
-  <xacro:joe prefix="$(arg prefix)" parent="world">
-    <origin xyz="0 0 0" rpy="0 0 0"/>          <!-- position robot in the world -->
-  </xacro:joe>
+  <xacro:if value="$(arg attach_world)">
+    <link name="world"/>
+    <xacro:joe prefix="$(arg prefix)" parent="world">
+      <origin xyz="0 0 0" rpy="0 0 0"/>
+    </xacro:joe>
+  </xacro:if>
+  <xacro:unless value="$(arg attach_world)">
+    <xacro:joe prefix="$(arg prefix)" parent="">
+      <origin xyz="0 0 0" rpy="0 0 0"/>
+    </xacro:joe>
+  </xacro:unless>
   <xacro:joe_ros2_control
     name="joe"

File: cororos2_joe_description/urdf/joe/joe_macro.ros2_control.xacro (robot description, xacro)
@@ -8,6 +8,5 @@
                sim_gazebo_classic:=false
                sim_gazebo:=false
-               simulation_controllers"
-               >
+               simulation_controllers">
     <ros2_control name="${name}" type="system">
       <hardware>
@@ -26,96 +25,34 @@
         </xacro:unless>
       </hardware>
-      <joint name="${prefix}joint1">
-        <command_interface name="position">     <!-- Add/Remove interfaces as needed -->
-          <param name="min">-1</param>
-          <param name="max">1</param>
-        </command_interface>
+      <joint name="${prefix}front_left_wheel_joint">
+        <command_interface name="velocity"/>
         <state_interface name="position">
           <param name="initial_value">0.0</param>
         </state_interface>
         <state_interface name="velocity"/>
-        <state_interface name="acceleration"/>
       </joint>
-      <joint name="${prefix}joint2">
-        <command_interface name="position">     <!-- Add/Remove interfaces as needed -->
-          <param name="min">-1</param>
-          <param name="max">1</param>
-        </command_interface>
+      <joint name="${prefix}front_right_wheel_joint">
+        <command_interface name="velocity"/>
         <state_interface name="position">
           <param name="initial_value">0.0</param>
         </state_interface>
         <state_interface name="velocity"/>
-        <state_interface name="acceleration"/>
       </joint>
-      <joint name="${prefix}joint3">
-        <command_interface name="position">     <!-- Add/Remove interfaces as needed -->
-          <param name="min">-1</param>
-          <param name="max">1</param>
-        </command_interface>
+      <joint name="${prefix}rear_left_wheel_joint">
+        <command_interface name="velocity"/>
         <state_interface name="position">
           <param name="initial_value">0.0</param>
         </state_interface>
         <state_interface name="velocity"/>
-        <state_interface name="acceleration"/>
       </joint>
-      <joint name="${prefix}joint4">
-        <command_interface name="position">     <!-- Add/Remove interfaces as needed -->
-          <param name="min">-1</param>
-          <param name="max">1</param>
-        </command_interface>
+      <joint name="${prefix}rear_right_wheel_joint">
+        <command_interface name="velocity"/>
         <state_interface name="position">
           <param name="initial_value">0.0</param>
         </state_interface>
         <state_interface name="velocity"/>
-        <state_interface name="acceleration"/>
       </joint>
-      <joint name="${prefix}joint5">
-        <command_interface name="position">     <!-- Add/Remove interfaces as needed -->
-          <param name="min">-1</param>
-          <param name="max">1</param>
-        </command_interface>
-        <state_interface name="position">
-          <param name="initial_value">0.0</param>
-        </state_interface>
-        <state_interface name="velocity"/>
-        <state_interface name="acceleration"/>
-      </joint>
-      <joint name="${prefix}joint6">
-        <command_interface name="position">     <!-- Add/Remove interfaces as needed -->
-          <param name="min">-1</param>
-          <param name="max">1</param>
-        </command_interface>
-        <state_interface name="position">
-          <param name="initial_value">0.0</param>
-        </state_interface>
-        <state_interface name="velocity"/>
-        <state_interface name="acceleration"/>
-      </joint>
-      <sensor name="tcp_fts_sensor">            <!-- Remove/change sensors as needed -->
-        <state_interface name="fx"/>
-        <state_interface name="fy"/>
-        <state_interface name="fz"/>
-        <state_interface name="tx"/>
-        <state_interface name="ty"/>
-        <state_interface name="tz"/>
-        <param name="frame_id">tool0</param>    <!-- Change sensors as needed -->
-        <param name="min_fx">-100</param>
-        <param name="max_fx">100</param>
-        <param name="min_fy">-100</param>
-        <param name="max_fy">100</param>
-        <param name="min_fz">-200</param>
-        <param name="max_fz">200</param>
-        <param name="min_tx">-10</param>
-        <param name="max_tx">10</param>
-        <param name="min_ty">-10</param>
-        <param name="max_ty">10</param>
-        <param name="min_tz">-15</param>
-        <param name="max_tz">15</param>
-      </sensor>
     </ros2_control>
-    <xacro:if value="$(arg sim_gazebo_classic)">
-      <!-- Gazebo plugins -->
-      <gazebo reference="world">
-      </gazebo>
+    <xacro:if value="${sim_gazebo_classic}">
       <gazebo>
         <plugin filename="libgazebo_ros2_control.so" name="gazebo_ros2_control">
@@ -124,12 +61,9 @@
       </gazebo>
     </xacro:if>
-    <xacro:if value="$(arg sim_gazebo)">
-      <!-- Gazebo plugins -->
-      <gazebo reference="world">
-      </gazebo>
+    <xacro:if value="${sim_gazebo}">
       <gazebo>
         <plugin filename="gz_ros2_control-system" name="gz_ros2_control::GazeboSimROS2ControlPlugin">
           <parameters>${simulation_controllers}</parameters>
-          <controller_manager_node_name>${prefix}controller_manager</controller_manager_node_name>
+          <controller_manager_node_name>controller_manager</controller_manager_node_name>
         </plugin>
       </gazebo>

File: cororos2_joe_description/urdf/joe/joe_macro.xacro (robot description, xacro)
@@ -1,244 +1,399 @@
 <?xml version="1.0" encoding="UTF-8"?>
 <robot xmlns:xacro="http://wiki.ros.org/xacro">
-  <xacro:include filename="$(find cororos2_joe_description)/urdf/common/inertials.xacro"/>
-  <xacro:include filename="$(find cororos2_joe_description)/urdf/common/materials.xacro"/>
   <xacro:macro name="joe" params="prefix parent *origin">
-    <!-- LINKS -->
-    <!-- base link -->
+    <link name="${prefix}base_footprint"/>
     <link name="${prefix}base_link">
-      <!-- Default inertial for Gazebo - copy and edit block from 'common.xacro'
-           to get more realistic behavior -->
-      <xacro:default_inertial/>
-      <visual>
-        <origin xyz="0 0 0" rpy="0 0 0"/>
-        <geometry>
-          <cylinder length="0.3" radius="0.3"/>
-          <!--           <mesh filename="package://cororos2_joe_description/meshes/joe/visual/base_link.dae" /> -->
-        </geometry>
-        <material name="black"/>
-      </visual>
-      <collision>
-        <origin xyz="0 0 0" rpy="0 0 0"/>
-        <geometry>
-          <cylinder length="0.3" radius="0.3"/>
-          <!--           <mesh filename="package://cororos2_joe_description/meshes/joe/collision/base_link.stl" /> -->
-        </geometry>
-      </collision>
-    </link>
-    <!-- link 1 -->
-    <link name="${prefix}link1">
-      <!-- Default inertial for Gazebo - copy and edit block from 'common.xacro'
-           to get more realistic behavior -->
-      <xacro:default_inertial/>
-      <visual>
-        <origin xyz="0 0 0" rpy="0 0 0"/>
-        <geometry>
-          <cylinder length="0.3" radius="0.15"/>
-          <!--           <mesh filename="package://cororos2_joe_description/meshes/joe/visual/link1.dae" /> -->
-        </geometry>
-        <material name="blue"/>
-      </visual>
-      <collision>
-        <origin xyz="0 0 0" rpy="0 0 0"/>
-        <geometry>
-          <cylinder length="0.3" radius="0.15"/>
-          <!--           <mesh filename="package://cororos2_joe_description/meshes/joe/collision/link1.stl" /> -->
-        </geometry>
-        <material name="green"/>
-      </collision>
-    </link>
-    <!-- link 2 -->
-    <link name="${prefix}link2">
-      <!-- Default inertial for Gazebo - copy and edit block from 'common.xacro'
-           to get more realistic behavior-->
-      <xacro:default_inertial/>
-      <visual>
-        <origin xyz="0 0 0" rpy="0 0 0"/>
-        <geometry>
-          <cylinder length="0.3" radius="0.15"/>
-          <!--           <mesh filename="package://cororos2_joe_description/meshes/joe/visual/link2.dae" /> -->
-        </geometry>
-        <material name="grey"/>
-      </visual>
-      <collision>
-        <origin xyz="0 0 0" rpy="0 0 0"/>
-        <geometry>
-          <cylinder length="0.3" radius="0.15"/>
-          <!--           <mesh filename="package://cororos2_joe_description/meshes/joe/collision/link2.stl"  /> -->
-        </geometry>
-      </collision>
-    </link>
-    <!-- link 3 -->
-    <link name="${prefix}link3">
-      <!-- Default inertial for Gazebo - copy and edit block from 'common.xacro'
-           to get more realistic behavior-->
-      <xacro:default_inertial/>
-      <visual>
-        <origin xyz="0 0 0" rpy="0 0 0"/>
-        <geometry>
-          <cylinder length="0.2" radius="0.1"/>
-          <!--           <mesh filename="package://cororos2_joe_description/meshes/joe/visual/link3.dae" /> -->
-        </geometry>
-        <material name="orange"/>
-      </visual>
-      <collision>
-        <origin xyz="0 0 0" rpy="0 0 0"/>
-        <geometry>
-          <cylinder length="0.2" radius="0.1"/>
-          <!--           <mesh filename="package://cororos2_joe_description/meshes/joe/collision/link3.stl"  /> -->
-        </geometry>
-      </collision>
-    </link>
-    <!-- link 4 -->
-    <link name="${prefix}link4">
-      <!-- Default inertial for Gazebo - copy and edit block from 'common.xacro'
-           to get more realistic behavior-->
-      <xacro:default_inertial/>
-      <visual>
-        <origin xyz="0 0 0" rpy="0 0 0"/>
-        <geometry>
-          <cylinder length="0.1" radius="0.1"/>
-          <!--           <mesh filename="package://cororos2_joe_description/meshes/joe/visual/link4.dae" /> -->
-        </geometry>
-        <material name="brown"/>
-      </visual>
-      <collision>
-        <origin xyz="0 0 0" rpy="0 0 0"/>
-        <geometry>
-          <cylinder length="0.1" radius="0.1"/>
-          <!--           <mesh filename="package://cororos2_joe_description/meshes/joe/collision/link4.stl"  /> -->
-        </geometry>
-      </collision>
-    </link>
-    <!-- link 5 -->
-    <link name="${prefix}link5">
-      <!-- Default inertial for Gazebo - copy and edit block from 'common.xacro'
-           to get more realistic behavior-->
-      <xacro:default_inertial/>
-      <visual>
-        <origin xyz="0 0 0" rpy="0 0 0"/>
-        <geometry>
-          <cylinder length="0.15" radius="0.1"/>
-          <!--           <mesh filename="package://cororos2_joe_description/meshes/joe/visual/link5.dae" /> -->
-        </geometry>
-        <material name="red"/>
-      </visual>
-      <collision>
-        <origin xyz="0 0 0" rpy="0 0 0"/>
-        <geometry>
-          <cylinder length="0.15" radius="0.1"/>
-          <!--           <mesh filename="package://cororos2_joe_description/meshes/joe/collision/link5.stl" /> -->
-        </geometry>
-      </collision>
-    </link>
-    <!-- link 6 -->
-    <link name="${prefix}link6">
-      <!-- Default inertial for Gazebo - copy and edit block from 'common.xacro'
-           to get more realistic behavior-->
-      <xacro:default_inertial/>
-      <visual>
-        <origin xyz="0 0 0" rpy="0 0 0"/>
-        <geometry>
-          <cylinder length="0.05" radius="0.075"/>
-          <!--           <mesh filename="package://cororos2_joe_description/meshes/joe/visual/link6.dae" /> -->
-        </geometry>
-        <material name="white"/>
-      </visual>
-      <collision>
-        <origin xyz="0 0 0" rpy="0 0 0"/>
-        <geometry>
-          <cylinder length="0.05" radius="0.075"/>
-          <!--           <mesh filename="package://cororos2_joe_description/meshes/joe/collision/link6.stl" /> -->
-        </geometry>
-      </collision>
-    </link>
-    <!-- All-zero tool frame. This frame should correspond to the TOOL frame of the robot's controller.) -->
-    <link name="${prefix}tool0"/>
-    <!-- tool link -->
-    <!-- START Delete if not needed -->
-    <!-- Standard frames for industrial robots. Also useful for manipulators.
-         (ROS-I specs - https://wiki.ros.org/Industrial/Tutorials/WorkingWithRosIndustrialRobotSupportPackages#Standardised_links_.2F_frames)-->
-    <!-- This frame should correspond to the BASE coordinate system of robot's controller.) -->
-    <link name="${prefix}base"/>
-    <!-- Frame for mounting EEF models to a manipulator. x+ axis points forward (REP 103). -->
-    <link name="${prefix}flange"/>
-    <!-- END Delete if not needed  -->
-    <!-- END LINKS -->
-    <!-- JOINTS -->
-    <!-- base_joint fixes base_link to the environment -->
-    <joint name="${prefix}base_joint" type="fixed">
-      <xacro:insert_block name="origin"/>
-      <parent link="${parent}"/>
+      <inertial>
+        <origin xyz="0 0 0.09" rpy="0 0 0"/>
+        <mass value="26.6"/>
+        <inertia ixx="0.387" ixy="0" ixz="0" iyy="0.790" iyz="0" izz="0.962"/>
+      </inertial>
+      <collision name="chassis_collision">
+        <origin xyz="0 0 0.05" rpy="0 0 0"/>
+        <geometry>
+          <box size="0.555 0.355 0.13"/>
+        </geometry>
+      </collision>
+      <collision name="tower_collision">
+        <origin xyz="0.13 0 0.27" rpy="0 0 0"/>
+        <geometry>
+          <box size="0.2 0.2 0.34"/>
+        </geometry>
+      </collision>
+      <visual name="chassis_main_visual">
+        <origin xyz="0 0 0.07" rpy="0 0 0"/>
+        <geometry>
+          <box size="0.38 0.3 0.13"/>
+        </geometry>
+        <material name="chassis_main_visual_mat">
+          <color rgba="0.6 0.6 0.6 1.0"/>
+        </material>
+      </visual>
+      <visual name="wheel_mount_visual_front_left">
+        <origin xyz="0.17 0.12 0" rpy="0 0 0"/>
+        <geometry>
+          <box size="0.03 0.06 0.02"/>
+        </geometry>
+        <material name="wheel_mount_visual_front_left_mat">
+          <color rgba="0.6 0.6 0.6 1.0"/>
+        </material>
+      </visual>
+      <visual name="wheel_mount_visual_front_right">
+        <origin xyz="0.17 -0.12 0" rpy="0 0 0"/>
+        <geometry>
+          <box size="0.03 0.06 0.02"/>
+        </geometry>
+        <material name="wheel_mount_visual_front_right_mat">
+          <color rgba="0.6 0.6 0.6 1.0"/>
+        </material>
+      </visual>
+      <visual name="wheel_mount_visual_rear_left">
+        <origin xyz="-0.17 0.12 0" rpy="0 0 0"/>
+        <geometry>
+          <box size="0.03 0.06 0.02"/>
+        </geometry>
+        <material name="wheel_mount_visual_rear_left_mat">
+          <color rgba="0.6 0.6 0.6 1.0"/>
+        </material>
+      </visual>
+      <visual name="wheel_mount_visual_rear_right">
+        <origin xyz="-0.17 -0.12 0" rpy="0 0 0"/>
+        <geometry>
+          <box size="0.03 0.06 0.02"/>
+        </geometry>
+        <material name="wheel_mount_visual_rear_right_mat">
+          <color rgba="0.6 0.6 0.6 1.0"/>
+        </material>
+      </visual>
+      <visual name="emergency_stop_bottom_visual">
+        <origin xyz="0.11 0.125 0.145" rpy="0 0 0"/>
+        <geometry>
+          <cylinder radius="0.015" length="0.015"/>
+        </geometry>
+        <material name="emergency_stop_bottom_visual_mat">
+          <color rgba="0.7059 0.7059 0.7059 1.0"/>
+        </material>
+      </visual>
+      <visual name="emergency_stop_top_visual">
+        <origin xyz="0.11 0.125 0.155" rpy="0 0 0"/>
+        <geometry>
+          <cylinder radius="0.02" length="0.005"/>
+        </geometry>
+        <material name="emergency_stop_top_visual_mat">
+          <color rgba="1.0 0.0 0.0 1.0"/>
+        </material>
+      </visual>
+      <visual name="plate1_visual">
+        <origin xyz="0 0 0.435" rpy="0 0 0"/>
+        <geometry>
+          <box size="0.2 0.2 0.005"/>
+        </geometry>
+        <material name="plate1_visual_mat">
+          <color rgba="0.7843 0.7843 0.7843 1.0"/>
+        </material>
+      </visual>
+      <visual name="plate2_visual">
+        <origin xyz="0 0 0.325" rpy="0 0 0"/>
+        <geometry>
+          <box size="0.2 0.2 0.005"/>
+        </geometry>
+        <material name="plate2_visual_mat">
+          <color rgba="0.7843 0.7843 0.7843 1.0"/>
+        </material>
+      </visual>
+      <visual name="plate3_visual">
+        <origin xyz="0 0 0.135" rpy="0 0 0"/>
+        <geometry>
+          <box size="0.2 0.2 0.005"/>
+        </geometry>
+        <material name="plate3_visual_mat">
+          <color rgba="0.9412 0.9412 0.9412 1.0"/>
+        </material>
+      </visual>
+      <visual name="beam1_visual">
+        <origin xyz="0.091 0.091 0.285" rpy="0 0 0"/>
+        <geometry>
+          <box size="0.02 0.02 0.3"/>
+        </geometry>
+        <material name="beam1_visual_mat">
+          <color rgba="0.7843 0.7843 0.7843 1.0"/>
+        </material>
+      </visual>
+      <visual name="beam2_visual">
+        <origin xyz="0.091 -0.091 0.285" rpy="0 0 0"/>
+        <geometry>
+          <box size="0.02 0.02 0.3"/>
+        </geometry>
+        <material name="beam2_visual_mat">
+          <color rgba="0.7843 0.7843 0.7843 1.0"/>
+        </material>
+      </visual>
+      <visual name="beam3_visual">
+        <origin xyz="-0.091 0.091 0.285" rpy="0 0 0"/>
+        <geometry>
+          <box size="0.02 0.02 0.3"/>
+        </geometry>
+        <material name="beam3_visual_mat">
+          <color rgba="0.7843 0.7843 0.7843 1.0"/>
+        </material>
+      </visual>
+      <visual name="beam4_visual">
+        <origin xyz="-0.091 -0.091 0.285" rpy="0 0 0"/>
+        <geometry>
+          <box size="0.02 0.02 0.3"/>
+        </geometry>
+        <material name="beam4_visual_mat">
+          <color rgba="0.7843 0.7843 0.7843 1.0"/>
+        </material>
+      </visual>
+    </link>
+    <link name="${prefix}front_left_wheel">
+      <inertial>
+        <origin xyz="0 0 0" rpy="0 0 0"/>
+        <mass value="5.0"/>
+        <inertia ixx="0.0153" ixy="0" ixz="0" iyy="0.025" iyz="0" izz="0.0153"/>
+      </inertial>
+      <collision name="front_left_wheel_collision">
+        <origin xyz="0 0 0" rpy="-1.5707963267948966 0 0"/>
+        <geometry>
+          <cylinder radius="0.1275" length="0.075"/>
+        </geometry>
+      </collision>
+      <visual name="front_left_wheel_tire_visual">
+        <origin xyz="0 0 0" rpy="1.5708 0 0"/>
+        <geometry>
+          <mesh filename="package://cororos2_joe_description/meshes/joe/visual/wheel_left.dae" scale="1.22 1.22 1.71"/>
+        </geometry>
+      </visual>
+      <visual name="front_left_wheel_axle_visual">
+        <origin xyz="0 -0.055 0" rpy="1.5707963267948966 0 0"/>
+        <geometry>
+          <cylinder radius="0.007" length="0.05"/>
+        </geometry>
+        <material name="front_left_wheel_axle_visual_mat">
+          <color rgba="0.1 0.1 0.1 1.0"/>
+        </material>
+      </visual>
+    </link>
+    <link name="${prefix}front_right_wheel">
+      <inertial>
+        <origin xyz="0 0 0" rpy="0 0 0"/>
+        <mass value="5.0"/>
+        <inertia ixx="0.0153" ixy="0" ixz="0" iyy="0.025" iyz="0" izz="0.0153"/>
+      </inertial>
+      <collision name="front_right_wheel_collision">
+        <origin xyz="0 0 0" rpy="1.5707963267948966 0 0"/>
+        <geometry>
+          <cylinder radius="0.1275" length="0.075"/>
+        </geometry>
+      </collision>
+      <visual name="front_right_wheel_tire_visual">
+        <origin xyz="0 0 0" rpy="1.5708 0 0"/>
+        <geometry>
+          <mesh filename="package://cororos2_joe_description/meshes/joe/visual/wheel_right.dae" scale="1.22 1.22 1.71"/>
+        </geometry>
+      </visual>
+      <visual name="front_right_wheel_axle_visual">
+        <origin xyz="0 0.055 0" rpy="1.5707963267948966 0 0"/>
+        <geometry>
+          <cylinder radius="0.007" length="0.05"/>
+        </geometry>
+        <material name="front_right_wheel_axle_visual_mat">
+          <color rgba="0.1 0.1 0.1 1.0"/>
+        </material>
+      </visual>
+    </link>
+    <link name="${prefix}rear_left_wheel">
+      <inertial>
+        <origin xyz="0 0 0" rpy="0 0 0"/>
+        <mass value="5.0"/>
+        <inertia ixx="0.0153" ixy="0" ixz="0" iyy="0.025" iyz="0" izz="0.0153"/>
+      </inertial>
+      <collision name="rear_left_wheel_collision">
+        <origin xyz="0 0 0" rpy="-1.5707963267948966 0 0"/>
+        <geometry>
+          <cylinder radius="0.1275" length="0.075"/>
+        </geometry>
+      </collision>
+      <visual name="rear_left_wheel_tire_visual">
+        <origin xyz="0 0 0" rpy="1.5708 0 0"/>
+        <geometry>
+          <mesh filename="package://cororos2_joe_description/meshes/joe/visual/wheel_left.dae" scale="1.22 1.22 1.71"/>
+        </geometry>
+      </visual>
+      <visual name="rear_left_wheel_axle_visual">
+        <origin xyz="0 -0.055 0" rpy="1.5707963267948966 0 0"/>
+        <geometry>
+          <cylinder radius="0.007" length="0.05"/>
+        </geometry>
+        <material name="rear_left_wheel_axle_visual_mat">
+          <color rgba="0.1 0.1 0.1 1.0"/>
+        </material>
+      </visual>
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