Commit message: Add gps, imu, lidar and ralsense drivers. Add missing frames and clean uneeded frames

File: cororos2_joe_description/urdf/joe/joe_macro.xacro (robot description, xacro)
@@ -267,5 +267,5 @@
       </inertial>
     </link>
-    <link name="${prefix}rgbd_front_link">
+    <link name="${prefix}gps_link">
       <inertial>
         <origin xyz="0 0 0" rpy="0 0 0"/>
@@ -273,4 +273,11 @@
         <inertia ixx="1e-9" ixy="0" ixz="0" iyy="1e-9" iyz="0" izz="1e-9"/>
       </inertial>
+    </link>
+    <link name="${prefix}rgbd_front_link">
+      <inertial>
+        <origin xyz="0 0 0" rpy="0 0 0"/>
+        <mass value="1e-6"/>
+        <inertia ixx="1e-9" ixy="0" ixz="0" iyy="1e-9" iyz="0" izz="1e-9"/>
+      </inertial>
       <visual name="d435i_realsense_camera_visual">
         <origin xyz="-0.03 0 0" rpy="0 0 0"/>
@@ -280,5 +287,5 @@
       </visual>
     </link>
-    <link name="${prefix}front_laser_link">
+    <link name="${prefix}ouster_link">
       <inertial>
         <origin xyz="0 0 0" rpy="0 0 0"/>
@@ -304,4 +311,11 @@
         </geometry>
       </visual>
+    </link>
+    <link name="${prefix}ouster_imu_link">
+      <inertial>
+        <origin xyz="0 0 0" rpy="0 0 0"/>
+        <mass value="1e-6"/>
+        <inertia ixx="1e-9" ixy="0" ixz="0" iyy="1e-9" iyz="0" izz="1e-9"/>
+      </inertial>
     </link>
     <link name="${prefix}light_front_link">
@@ -366,4 +380,9 @@
       <origin xyz="0 0 0" rpy="0 0 0"/>
     </joint>
+    <joint name="${prefix}base_link_to_gps_link_joint" type="fixed">
+      <parent link="${prefix}base_link"/>
+      <child link="${prefix}gps_link"/>
+      <origin xyz="0 0 1.58" rpy="0 0 0"/>
+    </joint>
     <joint name="${prefix}base_link_to_rgbd_front_link_joint" type="fixed">
       <parent link="${prefix}base_link"/>
@@ -371,8 +390,13 @@
       <origin xyz="0.11 0 1.5" rpy="0 0.5236 0"/>
     </joint>
-    <joint name="${prefix}base_link_to_front_laser_link_joint" type="fixed">
-      <parent link="${prefix}base_link"/>
-      <child link="${prefix}front_laser_link"/>
+    <joint name="${prefix}base_link_to_ouster_link_joint" type="fixed">
+      <parent link="${prefix}base_link"/>
+      <child link="${prefix}ouster_link"/>
       <origin xyz="0 0 0.365" rpy="0 0 0"/>
+    </joint>
+    <joint name="${prefix}ouster_link_to_ouster_imu_link_joint" type="fixed">
+      <parent link="${prefix}ouster_link"/>
+      <child link="${prefix}ouster_imu_link"/>
+      <origin xyz="0 0 0" rpy="0 0 0"/>
     </joint>
     <joint name="${prefix}base_link_to_light_front_link_joint" type="fixed">

Commit message: Replace ouster lidar with velodyne

File: cororos2_joe_description/urdf/joe/joe_macro.xacro (robot description, xacro)
@@ -287,5 +287,5 @@
       </visual>
     </link>
-    <link name="${prefix}ouster_link">
+    <link name="${prefix}lidar_link">
       <inertial>
         <origin xyz="0 0 0" rpy="0 0 0"/>
@@ -311,11 +311,4 @@
         </geometry>
       </visual>
-    </link>
-    <link name="${prefix}ouster_imu_link">
-      <inertial>
-        <origin xyz="0 0 0" rpy="0 0 0"/>
-        <mass value="1e-6"/>
-        <inertia ixx="1e-9" ixy="0" ixz="0" iyy="1e-9" iyz="0" izz="1e-9"/>
-      </inertial>
     </link>
     <link name="${prefix}light_front_link">
@@ -390,13 +383,8 @@
       <origin xyz="0.11 0 1.5" rpy="0 0.5236 0"/>
     </joint>
-    <joint name="${prefix}base_link_to_ouster_link_joint" type="fixed">
-      <parent link="${prefix}base_link"/>
-      <child link="${prefix}ouster_link"/>
+    <joint name="${prefix}base_link_to_lidar_link_joint" type="fixed">
+      <parent link="${prefix}base_link"/>
+      <child link="${prefix}lidar_link"/>
       <origin xyz="0 0 0.365" rpy="0 0 0"/>
-    </joint>
-    <joint name="${prefix}ouster_link_to_ouster_imu_link_joint" type="fixed">
-      <parent link="${prefix}ouster_link"/>
-      <child link="${prefix}ouster_imu_link"/>
-      <origin xyz="0 0 0" rpy="0 0 0"/>
     </joint>
     <joint name="${prefix}base_link_to_light_front_link_joint" type="fixed">
@@ -555,6 +543,6 @@
       </sensor>
     </gazebo>
-    <gazebo reference="${prefix}ouster_link">
-      <sensor name="ouster_lidar" type="gpu_lidar">
+    <gazebo reference="${prefix}lidar_link">
+      <sensor name="lidar" type="gpu_lidar">
         <visualize>0</visualize>
         <update_rate>10</update_rate>
