Commit message: Add fixes derived from outdated MAHA navigation stack

File: cororos2_description/urdf/joe/joe_macro.xacro (robot description, xacro)
@@ -345,5 +345,5 @@
       <origin xyz="0.17 0.21 0" rpy="0 0 0"/>
       <axis xyz="0 1 0"/>
-      <limit effort="10" velocity="19.61"/>
+      <limit effort="50" velocity="19.61"/>
     </joint>
     <joint name="${prefix}rear_left_wheel_joint" type="continuous">
@@ -352,5 +352,5 @@
       <origin xyz="-0.17 0.21 0" rpy="0 0 0"/>
       <axis xyz="0 1 0"/>
-      <limit effort="10" velocity="19.61"/>
+      <limit effort="50" velocity="19.61"/>
     </joint>
     <joint name="${prefix}rear_right_wheel_joint" type="continuous">
@@ -359,5 +359,5 @@
       <origin xyz="-0.17 -0.21 0" rpy="0 0 0"/>
       <axis xyz="0 1 0"/>
-      <limit effort="10" velocity="19.61"/>
+      <limit effort="50" velocity="19.61"/>
     </joint>
     <joint name="${prefix}front_right_wheel_joint" type="continuous">
@@ -366,5 +366,5 @@
       <origin xyz="0.17 -0.21 0" rpy="0 0 0"/>
       <axis xyz="0 1 0"/>
-      <limit effort="10" velocity="19.61"/>
+      <limit effort="50" velocity="19.61"/>
     </joint>
     <joint name="${prefix}base_link_to_imu_sensor_link_joint" type="fixed">
@@ -386,5 +386,5 @@
       <parent link="${prefix}base_link"/>
       <child link="${prefix}lidar_link"/>
-      <origin xyz="0 0 0.365" rpy="0 0 0"/>
+      <origin xyz="0 0 0.48" rpy="0 0 0"/>
     </joint>
     <joint name="${prefix}base_link_to_light_front_link_joint" type="fixed">

Commit message: Fix joe effort for better simulation drive

File: cororos2_description/urdf/joe/joe_macro.xacro (robot description, xacro)
@@ -345,5 +345,5 @@
       <origin xyz="0.17 0.21 0" rpy="0 0 0"/>
       <axis xyz="0 1 0"/>
-      <limit effort="10" velocity="19.61"/>
+      <limit effort="50" velocity="19.61"/>
     </joint>
     <joint name="${prefix}rear_left_wheel_joint" type="continuous">
@@ -352,5 +352,5 @@
       <origin xyz="-0.17 0.21 0" rpy="0 0 0"/>
       <axis xyz="0 1 0"/>
-      <limit effort="10" velocity="19.61"/>
+      <limit effort="50" velocity="19.61"/>
     </joint>
     <joint name="${prefix}rear_right_wheel_joint" type="continuous">
@@ -359,5 +359,5 @@
       <origin xyz="-0.17 -0.21 0" rpy="0 0 0"/>
       <axis xyz="0 1 0"/>
-      <limit effort="10" velocity="19.61"/>
+      <limit effort="50" velocity="19.61"/>
     </joint>
     <joint name="${prefix}front_right_wheel_joint" type="continuous">
@@ -366,5 +366,5 @@
       <origin xyz="0.17 -0.21 0" rpy="0 0 0"/>
       <axis xyz="0 1 0"/>
-      <limit effort="10" velocity="19.61"/>
+      <limit effort="50" velocity="19.61"/>
     </joint>
     <joint name="${prefix}base_link_to_imu_sensor_link_joint" type="fixed">
