Commit message: Put parameters to yaml files

File: cororos2_description/urdf/allie.urdf.xacro (robot description, xacro)
@@ -9,16 +9,18 @@
   <xacro:arg name="simulation_controllers" default=""/>
   <xacro:arg name="attach_world" default="true"/>
-  <xacro:arg name="device_path" default="/dev/serial/by-id/usb-Pololu_Corporation_Pololu_Micro_Maestro_6-Servo_Controller_00467337-if00"/>
-  <xacro:arg name="channel_fl" default="0"/>
-  <xacro:arg name="channel_fr" default="1"/>
-  <xacro:arg name="channel_rl" default="2"/>
-  <xacro:arg name="channel_rr" default="3"/>
-  <xacro:arg name="pwm_min" default="1000"/>
-  <xacro:arg name="pwm_neutral" default="1500"/>
-  <xacro:arg name="pwm_max" default="2000"/>
-  <xacro:arg name="wheel_radius" default="0.205"/>
-  <xacro:arg name="max_wheel_speed_mps" default="2.8"/>
-  <xacro:arg name="invert_left" default="false"/>
-  <xacro:arg name="invert_right" default="false"/>
+  <xacro:arg name="pwm_config_file" default="$(find cororos2_bringup)/config/pwm.yaml"/>
+  <xacro:property name="pwm_config" value="${xacro.load_yaml('$(arg pwm_config_file)')}"/>
+  <xacro:arg name="device_path" default="${pwm_config['device_path']}"/>
+  <xacro:arg name="channel_fl" default="${pwm_config['channel_fl']}"/>
+  <xacro:arg name="channel_fr" default="${pwm_config['channel_fr']}"/>
+  <xacro:arg name="channel_rl" default="${pwm_config['channel_rl']}"/>
+  <xacro:arg name="channel_rr" default="${pwm_config['channel_rr']}"/>
+  <xacro:arg name="pwm_min" default="${pwm_config['pwm_min']}"/>
+  <xacro:arg name="pwm_neutral" default="${pwm_config['pwm_neutral']}"/>
+  <xacro:arg name="pwm_max" default="${pwm_config['pwm_max']}"/>
+  <xacro:arg name="wheel_radius" default="${pwm_config['wheel_radius']}"/>
+  <xacro:arg name="max_wheel_speed_mps" default="${pwm_config['max_wheel_speed_mps']}"/>
+  <xacro:arg name="invert_left" default="${pwm_config['invert_left']}"/>
+  <xacro:arg name="invert_right" default="${pwm_config['invert_right']}"/>
   <xacro:include filename="$(find cororos2_description)/urdf/allie/allie_macro.xacro"/>
   <xacro:include filename="$(find cororos2_description)/urdf/allie/allie_macro.ros2_control.xacro"/>

File: cororos2_description/urdf/cornelius.urdf.xacro (robot description, xacro)
@@ -8,18 +8,20 @@
   <xacro:arg name="simulation_controllers" default=""/>
   <xacro:arg name="attach_world" default="true"/>
-  <xacro:arg name="python_executable" default="python3"/>
-  <xacro:arg name="roboclaw_device" default="/dev/serial/by-id/usb-03eb_USB_Roboclaw_2x60A-if00"/>
-  <xacro:arg name="roboclaw_baud" default="115200"/>
-  <xacro:arg name="roboclaw_address" default="128"/>
-  <xacro:arg name="roboclaw_use_encoder" default="false"/>
-  <xacro:arg name="roboclaw_max_speed" default="1.2"/>
-  <xacro:arg name="roboclaw_ticks_at_max_speed" default="32760.0"/>
-  <xacro:arg name="roboclaw_acceleration" default="32000"/>
-  <xacro:arg name="roboclaw_ticks_per_meter" default="4342.2"/>
-  <xacro:arg name="roboclaw_m1_invert" default="false"/>
-  <xacro:arg name="roboclaw_m2_invert" default="false"/>
-  <xacro:arg name="roboclaw_m1_encoder_sign" default="1"/>
-  <xacro:arg name="roboclaw_m2_encoder_sign" default="1"/>
-  <xacro:arg name="roboclaw_wheel_radius" default="0.129"/>
+  <xacro:arg name="roboclaw_config_file" default="$(find cororos2_bringup)/config/roboclaw.yaml"/>
+  <xacro:property name="roboclaw_config" value="${xacro.load_yaml('$(arg roboclaw_config_file)')}"/>
+  <xacro:arg name="python_executable" default="${roboclaw_config['python_executable']}"/>
+  <xacro:arg name="roboclaw_device" default="${roboclaw_config['device']}"/>
+  <xacro:arg name="roboclaw_baud" default="${roboclaw_config['baud']}"/>
+  <xacro:arg name="roboclaw_address" default="${roboclaw_config['address']}"/>
+  <xacro:arg name="roboclaw_use_encoder" default="${roboclaw_config['use_encoder']}"/>
+  <xacro:arg name="roboclaw_max_speed" default="${roboclaw_config['max_speed']}"/>
+  <xacro:arg name="roboclaw_ticks_at_max_speed" default="${roboclaw_config['ticks_at_max_speed']}"/>
+  <xacro:arg name="roboclaw_acceleration" default="${roboclaw_config['acceleration']}"/>
+  <xacro:arg name="roboclaw_ticks_per_meter" default="${roboclaw_config['ticks_per_meter']}"/>
+  <xacro:arg name="roboclaw_m1_invert" default="${roboclaw_config['m1_invert']}"/>
+  <xacro:arg name="roboclaw_m2_invert" default="${roboclaw_config['m2_invert']}"/>
+  <xacro:arg name="roboclaw_m1_encoder_sign" default="${roboclaw_config['m1_encoder_sign']}"/>
+  <xacro:arg name="roboclaw_m2_encoder_sign" default="${roboclaw_config['m2_encoder_sign']}"/>
+  <xacro:arg name="roboclaw_wheel_radius" default="${roboclaw_config['wheel_radius']}"/>
   <xacro:include filename="$(find cororos2_description)/urdf/cornelius/cornelius_macro.xacro"/>
   <xacro:include filename="$(find cororos2_description)/urdf/cornelius/cornelius_macro.ros2_control.xacro"/>

File: cororos2_description/urdf/joe.urdf.xacro (robot description, xacro)
@@ -8,10 +8,12 @@
   <xacro:arg name="simulation_controllers" default=""/>
   <xacro:arg name="attach_world" default="true"/>
-  <xacro:arg name="python_executable" default="python3"/>
-  <xacro:arg name="front_serial_number" default=""/>
-  <xacro:arg name="rear_serial_number" default=""/>
-  <xacro:arg name="front_right_axis" default="0"/>
-  <xacro:arg name="rear_right_axis" default="1"/>
-  <xacro:arg name="connect_timeout" default="30.0"/>
+  <xacro:arg name="odrive_config_file" default="$(find cororos2_bringup)/config/odrive.yaml"/>
+  <xacro:property name="odrive_config" value="${xacro.load_yaml('$(arg odrive_config_file)')}"/>
+  <xacro:arg name="python_executable" default="${odrive_config['python_executable']}"/>
+  <xacro:arg name="front_serial_number" default="${odrive_config['front_serial_number']}"/>
+  <xacro:arg name="rear_serial_number" default="${odrive_config['rear_serial_number']}"/>
+  <xacro:arg name="front_right_axis" default="${odrive_config['front_right_axis']}"/>
+  <xacro:arg name="rear_right_axis" default="${odrive_config['rear_right_axis']}"/>
+  <xacro:arg name="connect_timeout" default="${odrive_config['connect_timeout']}"/>
   <xacro:include filename="$(find cororos2_description)/urdf/joe/joe_macro.xacro"/>
   <xacro:include filename="$(find cororos2_description)/urdf/joe/joe_macro.ros2_control.xacro"/>

Commit message: Edit physical properties for Allie and wheel radius. Add minimum active PWM offset for Allie. SHow  Ouster cloud in RViz.

File: cororos2_description/urdf/allie.urdf.xacro (robot description, xacro)
@@ -19,4 +19,5 @@
   <xacro:arg name="pwm_neutral" default="${pwm_config['pwm_neutral']}"/>
   <xacro:arg name="pwm_max" default="${pwm_config['pwm_max']}"/>
+  <xacro:arg name="min_active_pwm_delta" default="${pwm_config['min_active_pwm_delta']}"/>
   <xacro:arg name="wheel_radius" default="${pwm_config['wheel_radius']}"/>
   <xacro:arg name="max_wheel_speed_mps" default="${pwm_config['max_wheel_speed_mps']}"/>
@@ -55,4 +56,5 @@
     pwm_neutral="$(arg pwm_neutral)"
     pwm_max="$(arg pwm_max)"
+    min_active_pwm_delta="$(arg min_active_pwm_delta)"
     wheel_radius="$(arg wheel_radius)"
     max_wheel_speed_mps="$(arg max_wheel_speed_mps)"

File: cororos2_description/urdf/allie/allie_macro.ros2_control.xacro (robot description, xacro)
@@ -17,6 +17,7 @@
                pwm_neutral:=1500
                pwm_max:=2000
-               wheel_radius:=0.205
-               max_wheel_speed_mps:=2.8
+               min_active_pwm_delta:=100
+               wheel_radius:=0.2
+               max_wheel_speed_mps:=1.0
                invert_left:=false
                invert_right:=false">
@@ -43,4 +44,5 @@
           <param name="pwm_neutral">${pwm_neutral}</param>
           <param name="pwm_max">${pwm_max}</param>
+          <param name="min_active_pwm_delta">${min_active_pwm_delta}</param>
           <param name="wheel_radius">${wheel_radius}</param>
           <param name="max_wheel_speed_mps">${max_wheel_speed_mps}</param>

File: cororos2_description/urdf/allie/allie_macro.xacro (robot description, xacro)
@@ -145,5 +145,5 @@
         <origin xyz="0 0 0" rpy="-1.5708 0 0" />
         <geometry>
-          <cylinder radius="0.205" length="0.11" />
+          <cylinder radius="0.2" length="0.11" />
         </geometry>
       </collision>
@@ -151,5 +151,5 @@
         <origin xyz="0 0 0" rpy="0 0 0" />
         <geometry>
-          <mesh filename="package://cororos2_description/meshes/allie/visual/wheel.dae" scale="1.18 1.0 1.18" />
+          <mesh filename="package://cororos2_description/meshes/allie/visual/wheel.dae" scale="1.1512 1.0 1.1512" />
         </geometry>
       </visual>
@@ -165,5 +165,5 @@
         <origin xyz="0 0 0" rpy="1.5708 0 0" />
         <geometry>
-          <cylinder radius="0.205" length="0.11" />
+          <cylinder radius="0.2" length="0.11" />
         </geometry>
       </collision>
@@ -171,5 +171,5 @@
         <origin xyz="0 0 0" rpy="0 0 0" />
         <geometry>
-          <mesh filename="package://cororos2_description/meshes/allie/visual/wheel.dae" scale="1.18 1.0 1.18" />
+          <mesh filename="package://cororos2_description/meshes/allie/visual/wheel.dae" scale="1.1512 1.0 1.1512" />
         </geometry>
       </visual>
@@ -185,5 +185,5 @@
         <origin xyz="0 0 0" rpy="-1.5708 0 0" />
         <geometry>
-          <cylinder radius="0.205" length="0.11" />
+          <cylinder radius="0.2" length="0.11" />
         </geometry>
       </collision>
@@ -191,5 +191,5 @@
         <origin xyz="0 0 0" rpy="0 0 0" />
         <geometry>
-          <mesh filename="package://cororos2_description/meshes/allie/visual/wheel.dae" scale="1.18 1.0 1.18" />
+          <mesh filename="package://cororos2_description/meshes/allie/visual/wheel.dae" scale="1.1512 1.0 1.1512" />
         </geometry>
       </visual>
@@ -205,5 +205,5 @@
         <origin xyz="0 0 0" rpy="1.5708 0 0" />
         <geometry>
-          <cylinder radius="0.205" length="0.11" />
+          <cylinder radius="0.2" length="0.11" />
         </geometry>
       </collision>
@@ -211,5 +211,5 @@
         <origin xyz="0 0 0" rpy="0 0 0" />
         <geometry>
-          <mesh filename="package://cororos2_description/meshes/allie/visual/wheel.dae" scale="1.18 1.0 1.18" />
+          <mesh filename="package://cororos2_description/meshes/allie/visual/wheel.dae" scale="1.1512 1.0 1.1512" />
         </geometry>
       </visual>
@@ -294,5 +294,5 @@
       <parent link="${prefix}base_footprint" />
       <child link="${prefix}base_link" />
-      <origin xyz="0 0 0.205" rpy="0 0 0" />
+      <origin xyz="0 0 0.2" rpy="0 0 0" />
     </joint>
     <!-- wheel joints -->
