Commit message: Readjust physical parameters and wheel sizes

File: cororos2_description/urdf/cornelius/cornelius_macro.ros2_control.xacro (robot description, xacro)
@@ -13,9 +13,9 @@
                roboclaw_address:=128
                roboclaw_use_encoder:=false
-               roboclaw_max_speed:=1.2
+               roboclaw_max_speed:=1.0
                roboclaw_ticks_at_max_speed:=32760.0
                roboclaw_acceleration:=32000
                roboclaw_ticks_per_meter:=4342.2
-               roboclaw_wheel_radius:=0.129
+               roboclaw_wheel_radius:=0.13
                roboclaw_status_interval_sec:=2.0">
     <ros2_control name="${name}" type="system">

File: cororos2_description/urdf/cornelius/cornelius_macro.xacro (robot description, xacro)
@@ -160,5 +160,5 @@
         <origin xyz="0.36 0 0" rpy="1.5707963267948966 0 0" />
         <geometry>
-          <cylinder radius="0.129" length="0.1" />
+          <cylinder radius="0.13" length="0.1" />
         </geometry>
         <material name="left_track_front_wheel_visual_mat">
@@ -169,5 +169,5 @@
         <origin xyz="-0.36 0 0" rpy="1.5707963267948966 0 0" />
         <geometry>
-          <cylinder radius="0.129" length="0.1" />
+          <cylinder radius="0.13" length="0.1" />
         </geometry>
         <material name="left_track_rear_wheel_visual_mat">
@@ -195,5 +195,5 @@
         <origin xyz="0.36 0 0" rpy="1.5707963267948966 0 0" />
         <geometry>
-          <cylinder radius="0.129" length="0.1" />
+          <cylinder radius="0.13" length="0.1" />
         </geometry>
         <material name="right_track_front_wheel_visual_mat">
@@ -204,5 +204,5 @@
         <origin xyz="-0.36 0 0" rpy="1.5707963267948966 0 0" />
         <geometry>
-          <cylinder radius="0.129" length="0.1" />
+          <cylinder radius="0.13" length="0.1" />
         </geometry>
         <material name="right_track_rear_wheel_visual_mat">
@@ -221,5 +221,5 @@
         <origin xyz="0 0 0" rpy="-1.5707963267948966 0 0" />
         <geometry>
-          <cylinder radius="0.129" length="0.1" />
+          <cylinder radius="0.13" length="0.1" />
         </geometry>
       </collision>
@@ -234,5 +234,5 @@
         <origin xyz="0 0 0" rpy="1.5707963267948966 0 0" />
         <geometry>
-          <cylinder radius="0.129" length="0.1" />
+          <cylinder radius="0.13" length="0.1" />
         </geometry>
       </collision>
@@ -351,5 +351,5 @@
       <parent link="${prefix}base_footprint" />
       <child link="${prefix}base_link" />
-      <origin xyz="0 0 0.129" rpy="0 0 0" />
+      <origin xyz="0 0 0.13" rpy="0 0 0" />
     </joint>
     <!-- tracked side joints -->
@@ -357,15 +357,15 @@
       <parent link="${prefix}base_link" />
       <child link="${prefix}left_track" />
-      <origin xyz="0 0.26 0" rpy="0 0 0" />
+      <origin xyz="0 0.1825 0" rpy="0 0 0" />
     </joint>
     <joint name="${prefix}right_track_mount_joint" type="fixed">
       <parent link="${prefix}base_link" />
       <child link="${prefix}right_track" />
-      <origin xyz="0 -0.26 0" rpy="0 0 0" />
+      <origin xyz="0 -0.1825 0" rpy="0 0 0" />
     </joint>
     <joint name="${prefix}left_track_joint" type="continuous">
       <parent link="${prefix}base_link" />
       <child link="${prefix}left_drive_wheel" />
-      <origin xyz="0 0.26 0" rpy="0 0 0" />
+      <origin xyz="0 0.1825 0" rpy="0 0 0" />
       <axis xyz="0 1 0" />
     </joint>
@@ -373,5 +373,5 @@
       <parent link="${prefix}base_link" />
       <child link="${prefix}right_drive_wheel" />
-      <origin xyz="0 -0.26 0" rpy="0 0 0" />
+      <origin xyz="0 -0.1825 0" rpy="0 0 0" />
       <axis xyz="0 1 0" />
     </joint>

File: cororos2_description/urdf/joe/joe_macro.xacro (robot description, xacro)
@@ -157,5 +157,5 @@
         <origin xyz="0 0 0" rpy="-1.5707963267948966 0 0"/>
         <geometry>
-          <cylinder radius="0.1275" length="0.075"/>
+          <cylinder radius="0.15" length="0.075"/>
         </geometry>
       </collision>
@@ -163,5 +163,5 @@
         <origin xyz="0 0 0" rpy="1.5708 0 0"/>
         <geometry>
-          <mesh filename="package://cororos2_description/meshes/joe/visual/wheel_left.dae" scale="1.22 1.22 1.71"/>
+          <mesh filename="package://cororos2_description/meshes/joe/visual/wheel_left.dae" scale="1.4353 1.4353 1.71"/>
         </geometry>
       </visual>
@@ -185,5 +185,5 @@
         <origin xyz="0 0 0" rpy="1.5707963267948966 0 0"/>
         <geometry>
-          <cylinder radius="0.1275" length="0.075"/>
+          <cylinder radius="0.15" length="0.075"/>
         </geometry>
       </collision>
@@ -191,5 +191,5 @@
         <origin xyz="0 0 0" rpy="1.5708 0 0"/>
         <geometry>
-          <mesh filename="package://cororos2_description/meshes/joe/visual/wheel_right.dae" scale="1.22 1.22 1.71"/>
+          <mesh filename="package://cororos2_description/meshes/joe/visual/wheel_right.dae" scale="1.4353 1.4353 1.71"/>
         </geometry>
       </visual>
@@ -213,5 +213,5 @@
         <origin xyz="0 0 0" rpy="-1.5707963267948966 0 0"/>
         <geometry>
-          <cylinder radius="0.1275" length="0.075"/>
+          <cylinder radius="0.15" length="0.075"/>
         </geometry>
       </collision>
@@ -219,5 +219,5 @@
         <origin xyz="0 0 0" rpy="1.5708 0 0"/>
         <geometry>
-          <mesh filename="package://cororos2_description/meshes/joe/visual/wheel_left.dae" scale="1.22 1.22 1.71"/>
+          <mesh filename="package://cororos2_description/meshes/joe/visual/wheel_left.dae" scale="1.4353 1.4353 1.71"/>
         </geometry>
       </visual>
@@ -241,5 +241,5 @@
         <origin xyz="0 0 0" rpy="1.5707963267948966 0 0"/>
         <geometry>
-          <cylinder radius="0.1275" length="0.075"/>
+          <cylinder radius="0.15" length="0.075"/>
         </geometry>
       </collision>
@@ -247,5 +247,5 @@
         <origin xyz="0 0 0" rpy="1.5708 0 0"/>
         <geometry>
-          <mesh filename="package://cororos2_description/meshes/joe/visual/wheel_right.dae" scale="1.22 1.22 1.71"/>
+          <mesh filename="package://cororos2_description/meshes/joe/visual/wheel_right.dae" scale="1.4353 1.4353 1.71"/>
         </geometry>
       </visual>
@@ -338,10 +338,10 @@
       <parent link="${prefix}base_footprint"/>
       <child link="${prefix}base_link"/>
-      <origin xyz="0 0 0.1275" rpy="0 0 0"/>
+      <origin xyz="0 0 0.15" rpy="0 0 0"/>
     </joint>
     <joint name="${prefix}front_left_wheel_joint" type="continuous">
       <parent link="${prefix}base_link"/>
       <child link="${prefix}front_left_wheel"/>
-      <origin xyz="0.17 0.21 0" rpy="0 0 0"/>
+      <origin xyz="0.17 0.212 0" rpy="0 0 0"/>
       <axis xyz="0 1 0"/>
       <limit effort="50" velocity="19.61"/>
@@ -350,5 +350,5 @@
       <parent link="${prefix}base_link"/>
       <child link="${prefix}rear_left_wheel"/>
-      <origin xyz="-0.17 0.21 0" rpy="0 0 0"/>
+      <origin xyz="-0.17 0.212 0" rpy="0 0 0"/>
       <axis xyz="0 1 0"/>
       <limit effort="50" velocity="19.61"/>
@@ -357,5 +357,5 @@
       <parent link="${prefix}base_link"/>
       <child link="${prefix}rear_right_wheel"/>
-      <origin xyz="-0.17 -0.21 0" rpy="0 0 0"/>
+      <origin xyz="-0.17 -0.212 0" rpy="0 0 0"/>
       <axis xyz="0 1 0"/>
       <limit effort="50" velocity="19.61"/>
@@ -364,5 +364,5 @@
       <parent link="${prefix}base_link"/>
       <child link="${prefix}front_right_wheel"/>
-      <origin xyz="0.17 -0.21 0" rpy="0 0 0"/>
+      <origin xyz="0.17 -0.212 0" rpy="0 0 0"/>
       <axis xyz="0 1 0"/>
       <limit effort="50" velocity="19.61"/>
