Commit message: Readjust base footprints sizes

File: cororos2_description/urdf/cornelius/cornelius_macro.xacro (robot description, xacro)
@@ -132,17 +132,17 @@
         <origin xyz="0 0 0" rpy="0 0 0" />
         <geometry>
-          <box size="0.72 0.1 0.258" />
+          <box size="0.72 0.14 0.258" />
         </geometry>
       </collision>
       <collision name="left_track_front_wheel_collision">
-        <origin xyz="0.36 0 0" rpy="1.5707963267948966 0 0" />
-        <geometry>
-          <cylinder radius="0.129" length="0.1" />
+        <origin xyz="0.355 0 0" rpy="1.5707963267948966 0 0" />
+        <geometry>
+          <cylinder radius="0.13" length="0.14" />
         </geometry>
       </collision>
       <collision name="left_track_rear_wheel_collision">
-        <origin xyz="-0.36 0 0" rpy="1.5707963267948966 0 0" />
-        <geometry>
-          <cylinder radius="0.129" length="0.1" />
+        <origin xyz="-0.355 0 0" rpy="1.5707963267948966 0 0" />
+        <geometry>
+          <cylinder radius="0.13" length="0.14" />
         </geometry>
       </collision>
@@ -150,5 +150,5 @@
         <origin xyz="0 0 0" rpy="0 0 0" />
         <geometry>
-          <box size="0.72 0.1 0.258" />
+          <box size="0.72 0.14 0.258" />
         </geometry>
         <material name="left_track_body_visual_mat">
@@ -157,7 +157,7 @@
       </visual>
       <visual name="left_track_front_wheel_visual">
-        <origin xyz="0.36 0 0" rpy="1.5707963267948966 0 0" />
-        <geometry>
-          <cylinder radius="0.13" length="0.1" />
+        <origin xyz="0.355 0 0" rpy="1.5707963267948966 0 0" />
+        <geometry>
+          <cylinder radius="0.13" length="0.14" />
         </geometry>
         <material name="left_track_front_wheel_visual_mat">
@@ -166,7 +166,7 @@
       </visual>
       <visual name="left_track_rear_wheel_visual">
-        <origin xyz="-0.36 0 0" rpy="1.5707963267948966 0 0" />
-        <geometry>
-          <cylinder radius="0.13" length="0.1" />
+        <origin xyz="-0.355 0 0" rpy="1.5707963267948966 0 0" />
+        <geometry>
+          <cylinder radius="0.13" length="0.14" />
         </geometry>
         <material name="left_track_rear_wheel_visual_mat">
@@ -185,17 +185,17 @@
         <origin xyz="0 0 0" rpy="0 0 0" />
         <geometry>
-          <box size="0.72 0.1 0.258" />
+          <box size="0.72 0.14 0.258" />
         </geometry>
       </collision>
       <collision name="right_track_front_wheel_collision">
-        <origin xyz="0.36 0 0" rpy="1.5707963267948966 0 0" />
-        <geometry>
-          <cylinder radius="0.129" length="0.1" />
+        <origin xyz="0.355 0 0" rpy="1.5707963267948966 0 0" />
+        <geometry>
+          <cylinder radius="0.13" length="0.14" />
         </geometry>
       </collision>
       <collision name="right_track_rear_wheel_collision">
-        <origin xyz="-0.36 0 0" rpy="1.5707963267948966 0 0" />
-        <geometry>
-          <cylinder radius="0.129" length="0.1" />
+        <origin xyz="-0.355 0 0" rpy="1.5707963267948966 0 0" />
+        <geometry>
+          <cylinder radius="0.13" length="0.14" />
         </geometry>
       </collision>
@@ -203,5 +203,5 @@
         <origin xyz="0 0 0" rpy="0 0 0" />
         <geometry>
-          <box size="0.72 0.1 0.258" />
+          <box size="0.72 0.14 0.258" />
         </geometry>
         <material name="right_track_body_visual_mat">
@@ -210,7 +210,7 @@
       </visual>
       <visual name="right_track_front_wheel_visual">
-        <origin xyz="0.36 0 0" rpy="1.5707963267948966 0 0" />
-        <geometry>
-          <cylinder radius="0.13" length="0.1" />
+        <origin xyz="0.355 0 0" rpy="1.5707963267948966 0 0" />
+        <geometry>
+          <cylinder radius="0.13" length="0.14" />
         </geometry>
         <material name="right_track_front_wheel_visual_mat">
@@ -219,7 +219,7 @@
       </visual>
       <visual name="right_track_rear_wheel_visual">
-        <origin xyz="-0.36 0 0" rpy="1.5707963267948966 0 0" />
-        <geometry>
-          <cylinder radius="0.13" length="0.1" />
+        <origin xyz="-0.355 0 0" rpy="1.5707963267948966 0 0" />
+        <geometry>
+          <cylinder radius="0.13" length="0.14" />
         </geometry>
         <material name="right_track_rear_wheel_visual_mat">
@@ -238,5 +238,5 @@
         <origin xyz="0 0 0" rpy="-1.5707963267948966 0 0" />
         <geometry>
-          <cylinder radius="0.13" length="0.1" />
+          <cylinder radius="0.13" length="0.14" />
         </geometry>
       </collision>
@@ -251,5 +251,5 @@
         <origin xyz="0 0 0" rpy="1.5707963267948966 0 0" />
         <geometry>
-          <cylinder radius="0.13" length="0.1" />
+          <cylinder radius="0.13" length="0.14" />
         </geometry>
       </collision>

File: cororos2_description/urdf/joe/joe_macro.xacro (robot description, xacro)
@@ -19,5 +19,5 @@
       </collision>
       <collision name="front_left_wheel_mount_collision">
-        <origin xyz="0.17 0.12 0" rpy="0 0 0"/>
+        <origin xyz="0.17 0.22 0" rpy="0 0 0"/>
         <geometry>
           <box size="0.03 0.06 0.02"/>
@@ -25,5 +25,5 @@
       </collision>
       <collision name="front_right_wheel_mount_collision">
-        <origin xyz="0.17 -0.12 0" rpy="0 0 0"/>
+        <origin xyz="0.17 -0.22 0" rpy="0 0 0"/>
         <geometry>
           <box size="0.03 0.06 0.02"/>
@@ -31,5 +31,5 @@
       </collision>
       <collision name="rear_left_wheel_mount_collision">
-        <origin xyz="-0.17 0.12 0" rpy="0 0 0"/>
+        <origin xyz="-0.17 0.22 0" rpy="0 0 0"/>
         <geometry>
           <box size="0.03 0.06 0.02"/>
@@ -37,5 +37,5 @@
       </collision>
       <collision name="rear_right_wheel_mount_collision">
-        <origin xyz="-0.17 -0.12 0" rpy="0 0 0"/>
+        <origin xyz="-0.17 -0.22 0" rpy="0 0 0"/>
         <geometry>
           <box size="0.03 0.06 0.02"/>
@@ -65,5 +65,5 @@
       </visual>
       <visual name="front_left_wheel_mount_visual">
-        <origin xyz="0.17 0.12 0" rpy="0 0 0"/>
+        <origin xyz="0.17 0.22 0" rpy="0 0 0"/>
         <geometry>
           <box size="0.03 0.06 0.02"/>
@@ -74,5 +74,5 @@
       </visual>
       <visual name="front_right_wheel_mount_visual">
-        <origin xyz="0.17 -0.12 0" rpy="0 0 0"/>
+        <origin xyz="0.17 -0.22 0" rpy="0 0 0"/>
         <geometry>
           <box size="0.03 0.06 0.02"/>
@@ -83,5 +83,5 @@
       </visual>
       <visual name="rear_left_wheel_mount_visual">
-        <origin xyz="-0.17 0.12 0" rpy="0 0 0"/>
+        <origin xyz="-0.17 0.22 0" rpy="0 0 0"/>
         <geometry>
           <box size="0.03 0.06 0.02"/>
@@ -92,5 +92,5 @@
       </visual>
       <visual name="rear_right_wheel_mount_visual">
-        <origin xyz="-0.17 -0.12 0" rpy="0 0 0"/>
+        <origin xyz="-0.17 -0.22 0" rpy="0 0 0"/>
         <geometry>
           <box size="0.03 0.06 0.02"/>

Commit message: Fix dae and collisions for Cornelius

File: cororos2_description/urdf/cornelius/cornelius_macro.xacro (robot description, xacro)
@@ -17,5 +17,5 @@
         <origin xyz="0 0 -0.135" rpy="0 0 1.57" />
         <geometry>
-          <mesh filename="package://cororos2_description/meshes/cornelius/visual/hd2_marble_base_body_metric.dae" />
+          <mesh filename="package://cororos2_description/meshes/cornelius/collision/hd2_marble_base_body_collision.stl" />
         </geometry>
       </collision>

Commit message: Fix sensor positions

File: cororos2_description/urdf/cornelius/cornelius_macro.xacro (robot description, xacro)
@@ -105,5 +105,5 @@
       </visual>
       <visual name="camera_plate_visual">
-        <origin xyz="0.2425 0.01 1.521" rpy="0 0 0" />
+        <origin xyz="0.2525 0.04 1.423" rpy="0 0 0" />
         <geometry>
           <box size="0.085 0.22 0.012" />
@@ -114,5 +114,5 @@
       </visual>
       <visual name="gps_board_visual">
-        <origin xyz="0.27 0.09 1.675" rpy="0 0 0" />
+        <origin xyz="0.25 0.12 1.536" rpy="0 0 0" />
         <geometry>
           <box size="0.12 0.08 0.012" />
@@ -482,15 +482,15 @@
       <parent link="${prefix}base_link" />
       <child link="${prefix}imu_sensor_link" />
-      <origin xyz="0 0 0" rpy="0 0 0" />
+      <origin xyz="0 0 -0.048" rpy="0 0 0" />
     </joint>
     <joint name="${prefix}base_link_to_gps_link_joint" type="fixed">
       <parent link="${prefix}base_link" />
       <child link="${prefix}gps_link" />
-      <origin xyz="0.27 0.09 1.681" rpy="0 0 0" />
+      <origin xyz="0.25 0.12 1.542" rpy="0 0 0" />
     </joint>
     <joint name="${prefix}base_link_to_rgbd_front_link_joint" type="fixed">
       <parent link="${prefix}base_link" />
       <child link="${prefix}rgbd_front_link" />
-      <origin xyz="0.28 0 1.5" rpy="0 0.5236 0" />
+      <origin xyz="0.29 0.03 1.402" rpy="0 0.5236 0" />
     </joint>
     <joint name="${prefix}base_link_to_ouster_link_joint" type="fixed">

File: cororos2_description/urdf/joe/joe_macro.xacro (robot description, xacro)
@@ -182,7 +182,7 @@
       </visual>
       <visual name="sensor_mast_visual">
-        <origin xyz="0 0 1.0125" rpy="0 0 0"/>
-        <geometry>
-          <box size="0.025 0.025 1.125"/>
+        <origin xyz="0.075 0.075 0.86" rpy="0 0 0"/>
+        <geometry>
+          <box size="0.025 0.025 0.85"/>
         </geometry>
         <material name="sensor_mast_visual_mat">
@@ -191,5 +191,5 @@
       </visual>
       <visual name="camera_plate_visual">
-        <origin xyz="0.035 0 1.521" rpy="0 0 0"/>
+        <origin xyz="0.045 0.02 1.181" rpy="0 0 0"/>
         <geometry>
           <box size="0.11 0.12 0.012"/>
@@ -200,5 +200,5 @@
       </visual>
       <visual name="gps_board_visual">
-        <origin xyz="0 0 1.57" rpy="0 0 0"/>
+        <origin xyz="0.10 0.12 1.294" rpy="0 0 0"/>
         <geometry>
           <box size="0.14 0.10 0.012"/>
@@ -491,15 +491,15 @@
       <parent link="${prefix}base_link"/>
       <child link="${prefix}imu_sensor_link"/>
-      <origin xyz="0 0 0" rpy="0 0 0"/>
+      <origin xyz="-0.02 0 0.17" rpy="0 0 0"/>
     </joint>
     <joint name="${prefix}base_link_to_gps_link_joint" type="fixed">
       <parent link="${prefix}base_link"/>
       <child link="${prefix}gps_link"/>
-      <origin xyz="0 0 1.576" rpy="0 0 0"/>
+      <origin xyz="0.10 0.12 1.30" rpy="0 0 0"/>
     </joint>
     <joint name="${prefix}base_link_to_rgbd_front_link_joint" type="fixed">
       <parent link="${prefix}base_link"/>
       <child link="${prefix}rgbd_front_link"/>
-      <origin xyz="0.11 0 1.5" rpy="0 0.5236 0"/>
+      <origin xyz="0.12 0.02 1.16" rpy="0 0.5236 0"/>
     </joint>
     <joint name="${prefix}base_link_to_lidar_link_joint" type="fixed">

Commit message: change cornelius ouster rotation

File: cororos2_description/urdf/cornelius/cornelius_macro.xacro (robot description, xacro)
@@ -501,5 +501,5 @@
       </xacro:if>
       <xacro:unless value="${sim_gazebo or sim_gazebo_classic}">
-        <origin xyz="0.19 0 0.272" rpy="0 0 0" />
+        <origin xyz="0.19 0 0.272" rpy="0 0 3.141592653589793" />
       </xacro:unless>
     </joint>

Commit message: Add pointcloud_to_laserscan node instead of Ouster native scan. Restore Cornelius Ouster frame

File: cororos2_description/urdf/cornelius/cornelius_macro.xacro (robot description, xacro)
@@ -501,5 +501,5 @@
       </xacro:if>
       <xacro:unless value="${sim_gazebo or sim_gazebo_classic}">
-        <origin xyz="0.19 0 0.272" rpy="0 0 3.141592653589793" />
+        <origin xyz="0.19 0 0.272" rpy="0 0 0" />
       </xacro:unless>
     </joint>
