Commit message: Fix sensors positions and add mast and sensor boards

File: cororos2_description/urdf/allie/allie_macro.xacro (robot description, xacro)
@@ -13,5 +13,6 @@
         <inertia ixx="0.387" ixy="0" ixz="0" iyy="0.790" iyz="0" izz="0.962" />
       </inertial>
-      <collision name="chassis_collision">
+      <!-- collisions -->
+      <collision name="chassis_main_collision">
         <origin xyz="0 0 0.05" rpy="0 0 0" />
         <geometry>
@@ -19,10 +20,53 @@
         </geometry>
       </collision>
-      <collision name="tower_collision">
-        <origin xyz="0.13 0 0.27" rpy="0 0 0" />
-        <geometry>
-          <box size="0.2 0.2 0.34" />
-        </geometry>
-      </collision>
+      <collision name="ouster_deck_collision">
+        <origin xyz="0.175 0.01 0.3625" rpy="0 0 0" />
+        <geometry>
+          <box size="0.24 0.18 0.02" />
+        </geometry>
+      </collision>
+      <collision name="beam1_collision">
+        <origin xyz="0.255 0.07 0.24375" rpy="0 0 0" />
+        <geometry>
+          <box size="0.02 0.02 0.2375" />
+        </geometry>
+      </collision>
+      <collision name="beam2_collision">
+        <origin xyz="0.255 -0.05 0.24375" rpy="0 0 0" />
+        <geometry>
+          <box size="0.02 0.02 0.2375" />
+        </geometry>
+      </collision>
+      <collision name="beam3_collision">
+        <origin xyz="0.095 0.07 0.24375" rpy="0 0 0" />
+        <geometry>
+          <box size="0.02 0.02 0.2375" />
+        </geometry>
+      </collision>
+      <collision name="beam4_collision">
+        <origin xyz="0.095 -0.05 0.24375" rpy="0 0 0" />
+        <geometry>
+          <box size="0.02 0.02 0.2375" />
+        </geometry>
+      </collision>
+      <collision name="sensor_mast_collision">
+        <origin xyz="0.255 0.07 1.01625" rpy="0 0 0" />
+        <geometry>
+          <box size="0.03 0.03 1.3175" />
+        </geometry>
+      </collision>
+      <collision name="camera_plate_collision">
+        <origin xyz="0.2745 0.01 1.552" rpy="0 0 0" />
+        <geometry>
+          <box size="0.095 0.16 0.02" />
+        </geometry>
+      </collision>
+      <collision name="gps_board_collision">
+        <origin xyz="0.27 0.09 1.675" rpy="0 0 0" />
+        <geometry>
+          <box size="0.12 0.08 0.02" />
+        </geometry>
+      </collision>
+      <!-- visuals -->
       <visual name="chassis_main_visual">
         <origin xyz="0 0 0.05" rpy="0 0 0" />
@@ -55,5 +99,5 @@
         <origin xyz="0.249 0 0.011" rpy="0 0 0" />
         <geometry>
-          <box size="0.05 0.5 0.05" />
+          <box size="0.05 0.52 0.05" />
         </geometry>
         <material name="wheel_mount_front_visual_mat">
@@ -64,5 +108,5 @@
         <origin xyz="-0.249 0 0.011" rpy="0 0 0" />
         <geometry>
-          <box size="0.05 0.5 0.05" />
+          <box size="0.05 0.52 0.05" />
         </geometry>
         <material name="wheel_mount_rear_visual_mat">
@@ -70,64 +114,67 @@
         </material>
       </visual>
-      <visual name="plate1_visual">
-        <origin xyz="0.13 0 0.42" rpy="0 0 0" />
-        <geometry>
-          <box size="0.2 0.2 0.005" />
-        </geometry>
-        <material name="plate1_visual_mat">
+      <visual name="ouster_deck_visual">
+        <origin xyz="0.175 0.01 0.3625" rpy="0 0 0" />
+        <geometry>
+          <box size="0.24 0.18 0.012" />
+        </geometry>
+        <material name="ouster_deck_visual_mat">
           <color rgba="0.7843 0.7843 0.7843 1.0" />
         </material>
       </visual>
-      <visual name="plate2_visual">
-        <origin xyz="0.13 0 0.31" rpy="0 0 0" />
-        <geometry>
-          <box size="0.2 0.2 0.005" />
-        </geometry>
-        <material name="plate2_visual_mat">
+      <visual name="beam1_visual">
+        <origin xyz="0.255 0.07 0.24375" rpy="0 0 0" />
+        <geometry>
+          <box size="0.018 0.018 0.2375" />
+        </geometry>
+        <material name="beam_visual_mat">
           <color rgba="0.7843 0.7843 0.7843 1.0" />
         </material>
       </visual>
-      <visual name="plate3_visual">
-        <origin xyz="0.13 0 0.12" rpy="0 0 0" />
-        <geometry>
-          <box size="0.2 0.2 0.005" />
-        </geometry>
-        <material name="plate3_visual_mat">
-          <color rgba="0.9412 0.9412 0.9412 1.0" />
-        </material>
-      </visual>
-      <visual name="beam1_visual">
-        <origin xyz="0.221 0.091 0.27" rpy="0 0 0" />
-        <geometry>
-          <box size="0.02 0.02 0.3" />
-        </geometry>
-        <material name="beam1_visual_mat">
+      <visual name="beam2_visual">
+        <origin xyz="0.255 -0.05 0.24375" rpy="0 0 0" />
+        <geometry>
+          <box size="0.018 0.018 0.2375" />
+        </geometry>
+        <material name="beam_visual_mat" />
+      </visual>
+      <visual name="beam3_visual">
+        <origin xyz="0.095 0.07 0.24375" rpy="0 0 0" />
+        <geometry>
+          <box size="0.018 0.018 0.2375" />
+        </geometry>
+        <material name="beam_visual_mat" />
+      </visual>
+      <visual name="beam4_visual">
+        <origin xyz="0.095 -0.05 0.24375" rpy="0 0 0" />
+        <geometry>
+          <box size="0.018 0.018 0.2375" />
+        </geometry>
+        <material name="beam_visual_mat" />
+      </visual>
+      <visual name="sensor_mast_visual">
+        <origin xyz="0.255 0.07 1.01625" rpy="0 0 0" />
+        <geometry>
+          <box size="0.025 0.025 1.3175" />
+        </geometry>
+        <material name="sensor_mast_visual_mat">
           <color rgba="0.7843 0.7843 0.7843 1.0" />
         </material>
       </visual>
-      <visual name="beam2_visual">
-        <origin xyz="0.221 -0.091 0.27" rpy="0 0 0" />
-        <geometry>
-          <box size="0.02 0.02 0.3" />
-        </geometry>
-        <material name="beam2_visual_mat">
+      <visual name="camera_plate_visual">
+        <origin xyz="0.2745 0.01 1.548" rpy="0 0 0" />
+        <geometry>
+          <box size="0.095 0.16 0.012" />
+        </geometry>
+        <material name="camera_plate_visual_mat">
           <color rgba="0.7843 0.7843 0.7843 1.0" />
         </material>
       </visual>
-      <visual name="beam3_visual">
-        <origin xyz="0.039 0.091 0.27" rpy="0 0 0" />
-        <geometry>
-          <box size="0.02 0.02 0.3" />
-        </geometry>
-        <material name="beam3_visual_mat">
-          <color rgba="0.7843 0.7843 0.7843 1.0" />
-        </material>
-      </visual>
-      <visual name="beam4_visual">
-        <origin xyz="0.039 -0.091 0.27" rpy="0 0 0" />
-        <geometry>
-          <box size="0.02 0.02 0.3" />
-        </geometry>
-        <material name="beam4_visual_mat">
+      <visual name="gps_board_visual">
+        <origin xyz="0.27 0.09 1.675" rpy="0 0 0" />
+        <geometry>
+          <box size="0.12 0.08 0.012" />
+        </geometry>
+        <material name="gps_board_visual_mat">
           <color rgba="0.7843 0.7843 0.7843 1.0" />
         </material>
@@ -142,5 +189,5 @@
         <inertia ixx="0.0576" ixy="0" ixz="0" iyy="0.105" iyz="0" izz="0.0576" />
       </inertial>
-      <collision name="front_left_wheel_collision">
+      <collision name="front_left_wheel_tire_collision">
         <origin xyz="0 0 0" rpy="-1.5708 0 0" />
         <geometry>
@@ -162,5 +209,5 @@
         <inertia ixx="0.0576" ixy="0" ixz="0" iyy="0.105" iyz="0" izz="0.0576" />
       </inertial>
-      <collision name="front_right_wheel_collision">
+      <collision name="front_right_wheel_tire_collision">
         <origin xyz="0 0 0" rpy="1.5708 0 0" />
         <geometry>
@@ -182,5 +229,5 @@
         <inertia ixx="0.0576" ixy="0" ixz="0" iyy="0.105" iyz="0" izz="0.0576" />
       </inertial>
-      <collision name="rear_left_wheel_collision">
+      <collision name="rear_left_wheel_tire_collision">
         <origin xyz="0 0 0" rpy="-1.5708 0 0" />
         <geometry>
@@ -202,5 +249,5 @@
         <inertia ixx="0.0576" ixy="0" ixz="0" iyy="0.105" iyz="0" izz="0.0576" />
       </inertial>
-      <collision name="rear_right_wheel_collision">
+      <collision name="rear_right_wheel_tire_collision">
         <origin xyz="0 0 0" rpy="1.5708 0 0" />
         <geometry>
@@ -231,4 +278,31 @@
         <inertia ixx="1e-9" ixy="0" ixz="0" iyy="1e-9" iyz="0" izz="1e-9" />
       </inertial>
+      <visual name="gps_base_visual">
+        <origin xyz="0 0 0.012" rpy="0 0 0" />
+        <geometry>
+          <cylinder radius="0.028" length="0.024" />
+        </geometry>
+        <material name="gps_base_visual_mat">
+          <color rgba="0.92 0.92 0.92 1.0" />
+        </material>
+      </visual>
+      <visual name="gps_cap_visual">
+        <origin xyz="0 0 0.028" rpy="0 0 0" />
+        <geometry>
+          <sphere radius="0.016" />
+        </geometry>
+        <material name="gps_cap_visual_mat">
+          <color rgba="0.96 0.96 0.96 1.0" />
+        </material>
+      </visual>
+      <visual name="gps_antenna_tip_visual">
+        <origin xyz="0 0 0.060" rpy="0 0 0" />
+        <geometry>
+          <cylinder radius="0.0035" length="0.024" />
+        </geometry>
+        <material name="gps_antenna_tip_visual_mat">
+          <color rgba="0.2 0.2 0.2 1.0" />
+        </material>
+      </visual>
     </link>
     <!-- front RGB-D camera frame -->
@@ -334,5 +408,5 @@
       <parent link="${prefix}base_link" />
       <child link="${prefix}imu_sensor_link" />
-      <origin xyz="0 0 0" rpy="0 0 0" />
+      <origin xyz="0 0 -0.025" rpy="0 0 0" />
     </joint>
     <!-- base link to GPS frame -->
@@ -340,5 +414,5 @@
       <parent link="${prefix}base_link" />
       <child link="${prefix}gps_link" />
-      <origin xyz="0.13 0 1.58" rpy="0 0 0" />
+      <origin xyz="0.27 0.09 1.685" rpy="0 0 0" />
     </joint>
     <!-- base link to front RGB-D camera frame -->
@@ -346,5 +420,5 @@
       <parent link="${prefix}base_link" />
       <child link="${prefix}rgbd_front_link" />
-      <origin xyz="0.21 0 1.5" rpy="0 0.5236 0" />
+      <origin xyz="0.34 0.01 1.545" rpy="0 0.5236 0" />
     </joint>
     <!-- base link to Ouster sensor frame -->
@@ -352,5 +426,5 @@
       <parent link="${prefix}base_link" />
       <child link="${prefix}ouster_link" />
-      <origin xyz="0.13 0 0.35" rpy="0 -0 0" />
+      <origin xyz="0.16 0 0.405" rpy="0 0 0" />
     </joint>
     <!-- Ouster sensor frame to Ouster IMU frame -->
