Commit message: Fix sensor chassis and collisoin meshes for Joe

File: cororos2_description/urdf/allie/allie_macro.xacro (robot description, xacro)
@@ -18,4 +18,28 @@
         <geometry>
           <box size="0.555 0.355 0.13" />
+        </geometry>
+      </collision>
+      <collision name="emergency_stop_bottom_collision">
+        <origin xyz="0.2 0.15 0.125" rpy="0 0 0" />
+        <geometry>
+          <cylinder radius="0.015" length="0.015" />
+        </geometry>
+      </collision>
+      <collision name="emergency_stop_top_collision">
+        <origin xyz="0.2 0.15 0.135" rpy="0 0 0" />
+        <geometry>
+          <cylinder radius="0.02" length="0.005" />
+        </geometry>
+      </collision>
+      <collision name="wheel_mount_front_collision">
+        <origin xyz="0.249 0 0.011" rpy="0 0 0" />
+        <geometry>
+          <box size="0.05 0.52 0.05" />
+        </geometry>
+      </collision>
+      <collision name="wheel_mount_rear_collision">
+        <origin xyz="-0.249 0 0.011" rpy="0 0 0" />
+        <geometry>
+          <box size="0.05 0.52 0.05" />
         </geometry>
       </collision>

File: cororos2_description/urdf/joe/joe_macro.xacro (robot description, xacro)
@@ -2,5 +2,7 @@
 <robot xmlns:xacro="http://wiki.ros.org/xacro">
   <xacro:macro name="joe" params="prefix parent *origin">
+    <!-- LINKS -->
     <link name="${prefix}base_footprint"/>
+    <!-- base link -->
     <link name="${prefix}base_link">
       <inertial>
@@ -9,16 +11,108 @@
         <inertia ixx="0.387" ixy="0" ixz="0" iyy="0.790" iyz="0" izz="0.962"/>
       </inertial>
-      <collision name="chassis_collision">
-        <origin xyz="0 0 0.05" rpy="0 0 0"/>
-        <geometry>
-          <box size="0.555 0.355 0.13"/>
-        </geometry>
-      </collision>
-      <collision name="tower_collision">
-        <origin xyz="0.13 0 0.27" rpy="0 0 0"/>
-        <geometry>
-          <box size="0.2 0.2 0.34"/>
-        </geometry>
-      </collision>
+      <!-- collisions -->
+      <collision name="chassis_main_collision">
+        <origin xyz="0 0 0.07" rpy="0 0 0"/>
+        <geometry>
+          <box size="0.38 0.3 0.13"/>
+        </geometry>
+      </collision>
+      <collision name="front_left_wheel_mount_collision">
+        <origin xyz="0.17 0.12 0" rpy="0 0 0"/>
+        <geometry>
+          <box size="0.03 0.06 0.02"/>
+        </geometry>
+      </collision>
+      <collision name="front_right_wheel_mount_collision">
+        <origin xyz="0.17 -0.12 0" rpy="0 0 0"/>
+        <geometry>
+          <box size="0.03 0.06 0.02"/>
+        </geometry>
+      </collision>
+      <collision name="rear_left_wheel_mount_collision">
+        <origin xyz="-0.17 0.12 0" rpy="0 0 0"/>
+        <geometry>
+          <box size="0.03 0.06 0.02"/>
+        </geometry>
+      </collision>
+      <collision name="rear_right_wheel_mount_collision">
+        <origin xyz="-0.17 -0.12 0" rpy="0 0 0"/>
+        <geometry>
+          <box size="0.03 0.06 0.02"/>
+        </geometry>
+      </collision>
+      <collision name="emergency_stop_bottom_collision">
+        <origin xyz="0.11 0.125 0.145" rpy="0 0 0"/>
+        <geometry>
+          <cylinder radius="0.015" length="0.015"/>
+        </geometry>
+      </collision>
+      <collision name="emergency_stop_top_collision">
+        <origin xyz="0.11 0.125 0.155" rpy="0 0 0"/>
+        <geometry>
+          <cylinder radius="0.02" length="0.005"/>
+        </geometry>
+      </collision>
+      <collision name="sensor_upper_deck_collision">
+        <origin xyz="0 0 0.435" rpy="0 0 0"/>
+        <geometry>
+          <box size="0.2 0.2 0.01"/>
+        </geometry>
+      </collision>
+      <collision name="sensor_mid_deck_collision">
+        <origin xyz="0 0 0.325" rpy="0 0 0"/>
+        <geometry>
+          <box size="0.2 0.2 0.01"/>
+        </geometry>
+      </collision>
+      <collision name="sensor_lower_deck_collision">
+        <origin xyz="0 0 0.135" rpy="0 0 0"/>
+        <geometry>
+          <box size="0.2 0.2 0.01"/>
+        </geometry>
+      </collision>
+      <collision name="beam1_collision">
+        <origin xyz="0.091 0.091 0.285" rpy="0 0 0"/>
+        <geometry>
+          <box size="0.02 0.02 0.3"/>
+        </geometry>
+      </collision>
+      <collision name="beam2_collision">
+        <origin xyz="0.091 -0.091 0.285" rpy="0 0 0"/>
+        <geometry>
+          <box size="0.02 0.02 0.3"/>
+        </geometry>
+      </collision>
+      <collision name="beam3_collision">
+        <origin xyz="-0.091 0.091 0.285" rpy="0 0 0"/>
+        <geometry>
+          <box size="0.02 0.02 0.3"/>
+        </geometry>
+      </collision>
+      <collision name="beam4_collision">
+        <origin xyz="-0.091 -0.091 0.285" rpy="0 0 0"/>
+        <geometry>
+          <box size="0.02 0.02 0.3"/>
+        </geometry>
+      </collision>
+      <collision name="sensor_mast_collision">
+        <origin xyz="0 0 1.0125" rpy="0 0 0"/>
+        <geometry>
+          <box size="0.03 0.03 1.125"/>
+        </geometry>
+      </collision>
+      <collision name="camera_plate_collision">
+        <origin xyz="0.035 0 1.525" rpy="0 0 0"/>
+        <geometry>
+          <box size="0.11 0.12 0.02"/>
+        </geometry>
+      </collision>
+      <collision name="gps_board_collision">
+        <origin xyz="0 0 1.57" rpy="0 0 0"/>
+        <geometry>
+          <box size="0.14 0.10 0.02"/>
+        </geometry>
+      </collision>
+      <!-- visuals -->
       <visual name="chassis_main_visual">
         <origin xyz="0 0 0.07" rpy="0 0 0"/>
@@ -30,37 +124,37 @@
         </material>
       </visual>
-      <visual name="wheel_mount_visual_front_left">
+      <visual name="front_left_wheel_mount_visual">
         <origin xyz="0.17 0.12 0" rpy="0 0 0"/>
         <geometry>
           <box size="0.03 0.06 0.02"/>
         </geometry>
-        <material name="wheel_mount_visual_front_left_mat">
+        <material name="front_left_wheel_mount_visual_mat">
           <color rgba="0.6 0.6 0.6 1.0"/>
         </material>
       </visual>
-      <visual name="wheel_mount_visual_front_right">
+      <visual name="front_right_wheel_mount_visual">
         <origin xyz="0.17 -0.12 0" rpy="0 0 0"/>
         <geometry>
           <box size="0.03 0.06 0.02"/>
         </geometry>
-        <material name="wheel_mount_visual_front_right_mat">
+        <material name="front_right_wheel_mount_visual_mat">
           <color rgba="0.6 0.6 0.6 1.0"/>
         </material>
       </visual>
-      <visual name="wheel_mount_visual_rear_left">
+      <visual name="rear_left_wheel_mount_visual">
         <origin xyz="-0.17 0.12 0" rpy="0 0 0"/>
         <geometry>
           <box size="0.03 0.06 0.02"/>
         </geometry>
-        <material name="wheel_mount_visual_rear_left_mat">
+        <material name="rear_left_wheel_mount_visual_mat">
           <color rgba="0.6 0.6 0.6 1.0"/>
         </material>
       </visual>
-      <visual name="wheel_mount_visual_rear_right">
+      <visual name="rear_right_wheel_mount_visual">
         <origin xyz="-0.17 -0.12 0" rpy="0 0 0"/>
         <geometry>
           <box size="0.03 0.06 0.02"/>
         </geometry>
-        <material name="wheel_mount_visual_rear_right_mat">
+        <material name="rear_right_wheel_mount_visual_mat">
           <color rgba="0.6 0.6 0.6 1.0"/>
         </material>
@@ -84,28 +178,28 @@
         </material>
       </visual>
-      <visual name="plate1_visual">
+      <visual name="sensor_upper_deck_visual">
         <origin xyz="0 0 0.435" rpy="0 0 0"/>
         <geometry>
           <box size="0.2 0.2 0.005"/>
         </geometry>
-        <material name="plate1_visual_mat">
-          <color rgba="0.7843 0.7843 0.7843 1.0"/>
-        </material>
-      </visual>
-      <visual name="plate2_visual">
+        <material name="sensor_upper_deck_visual_mat">
+          <color rgba="0.7843 0.7843 0.7843 1.0"/>
+        </material>
+      </visual>
+      <visual name="sensor_mid_deck_visual">
         <origin xyz="0 0 0.325" rpy="0 0 0"/>
         <geometry>
           <box size="0.2 0.2 0.005"/>
         </geometry>
-        <material name="plate2_visual_mat">
-          <color rgba="0.7843 0.7843 0.7843 1.0"/>
-        </material>
-      </visual>
-      <visual name="plate3_visual">
+        <material name="sensor_mid_deck_visual_mat">
+          <color rgba="0.7843 0.7843 0.7843 1.0"/>
+        </material>
+      </visual>
+      <visual name="sensor_lower_deck_visual">
         <origin xyz="0 0 0.135" rpy="0 0 0"/>
         <geometry>
           <box size="0.2 0.2 0.005"/>
         </geometry>
-        <material name="plate3_visual_mat">
+        <material name="sensor_lower_deck_visual_mat">
           <color rgba="0.9412 0.9412 0.9412 1.0"/>
         </material>
@@ -147,5 +241,33 @@
         </material>
       </visual>
-    </link>
+      <visual name="sensor_mast_visual">
+        <origin xyz="0 0 1.0125" rpy="0 0 0"/>
+        <geometry>
+          <box size="0.025 0.025 1.125"/>
+        </geometry>
+        <material name="sensor_mast_visual_mat">
+          <color rgba="0.7843 0.7843 0.7843 1.0"/>
+        </material>
+      </visual>
+      <visual name="camera_plate_visual">
+        <origin xyz="0.035 0 1.521" rpy="0 0 0"/>
+        <geometry>
+          <box size="0.11 0.12 0.012"/>
+        </geometry>
+        <material name="camera_plate_visual_mat">
+          <color rgba="0.7843 0.7843 0.7843 1.0"/>
+        </material>
+      </visual>
+      <visual name="gps_board_visual">
+        <origin xyz="0 0 1.57" rpy="0 0 0"/>
+        <geometry>
+          <box size="0.14 0.10 0.012"/>
+        </geometry>
+        <material name="gps_board_visual_mat">
+          <color rgba="0.7843 0.7843 0.7843 1.0"/>
+        </material>
+      </visual>
+    </link>
+    <!-- drive wheels -->
     <link name="${prefix}front_left_wheel">
       <inertial>
@@ -154,5 +276,5 @@
         <inertia ixx="0.0153" ixy="0" ixz="0" iyy="0.025" iyz="0" izz="0.0153"/>
       </inertial>
-      <collision name="front_left_wheel_collision">
+      <collision name="front_left_wheel_tire_collision">
         <origin xyz="0 0 0" rpy="-1.5707963267948966 0 0"/>
         <geometry>
@@ -182,5 +304,5 @@
         <inertia ixx="0.0153" ixy="0" ixz="0" iyy="0.025" iyz="0" izz="0.0153"/>
       </inertial>
-      <collision name="front_right_wheel_collision">
+      <collision name="front_right_wheel_tire_collision">
         <origin xyz="0 0 0" rpy="1.5707963267948966 0 0"/>
         <geometry>
@@ -210,5 +332,5 @@
         <inertia ixx="0.0153" ixy="0" ixz="0" iyy="0.025" iyz="0" izz="0.0153"/>
       </inertial>
-      <collision name="rear_left_wheel_collision">
+      <collision name="rear_left_wheel_tire_collision">
         <origin xyz="0 0 0" rpy="-1.5707963267948966 0 0"/>
         <geometry>
@@ -238,5 +360,5 @@
         <inertia ixx="0.0153" ixy="0" ixz="0" iyy="0.025" iyz="0" izz="0.0153"/>
       </inertial>
-      <collision name="rear_right_wheel_collision">
+      <collision name="rear_right_wheel_tire_collision">
         <origin xyz="0 0 0" rpy="1.5707963267948966 0 0"/>
         <geometry>
@@ -260,4 +382,5 @@
       </visual>
     </link>
+    <!-- sensor and light frames -->
     <link name="${prefix}imu_sensor_link">
       <inertial>
@@ -273,4 +396,31 @@
         <inertia ixx="1e-9" ixy="0" ixz="0" iyy="1e-9" iyz="0" izz="1e-9"/>
       </inertial>
+      <visual name="gps_base_visual">
+        <origin xyz="0 0 0.012" rpy="0 0 0"/>
+        <geometry>
+          <cylinder radius="0.028" length="0.024"/>
+        </geometry>
+        <material name="gps_base_visual_mat">
+          <color rgba="0.92 0.92 0.92 1.0"/>
+        </material>
+      </visual>
+      <visual name="gps_cap_visual">
+        <origin xyz="0 0 0.028" rpy="0 0 0"/>
+        <geometry>
+          <sphere radius="0.016"/>
+        </geometry>
+        <material name="gps_cap_visual_mat">
+          <color rgba="0.96 0.96 0.96 1.0"/>
+        </material>
+      </visual>
+      <visual name="gps_antenna_tip_visual">
+        <origin xyz="0 0 0.060" rpy="0 0 0"/>
+        <geometry>
+          <cylinder radius="0.0035" length="0.024"/>
+        </geometry>
+        <material name="gps_antenna_tip_visual_mat">
+          <color rgba="0.2 0.2 0.2 1.0"/>
+        </material>
+      </visual>
     </link>
     <link name="${prefix}rgbd_front_link">
@@ -312,20 +462,6 @@
       </visual>
     </link>
-    <link name="${prefix}light_front_link">
-      <inertial><origin xyz="0 0 0" rpy="0 0 0"/><mass value="1e-6"/><inertia ixx="1e-9" ixy="0" ixz="0" iyy="1e-9" iyz="0" izz="1e-9"/></inertial>
-      <visual name="light_front_visual"><origin xyz="-0.03 0 0" rpy="0 0 0"/><geometry><box size="0.04 0.13 0.04"/></geometry><material name="light_front_visual_mat"><color rgba="0.0 0.0 0.0 1.0"/></material></visual>
-    </link>
-    <link name="${prefix}light_rear_link">
-      <inertial><origin xyz="0 0 0" rpy="0 0 0"/><mass value="1e-6"/><inertia ixx="1e-9" ixy="0" ixz="0" iyy="1e-9" iyz="0" izz="1e-9"/></inertial>
-      <visual name="light_rear_visual"><origin xyz="0.03 0 0" rpy="0 0 0"/><geometry><box size="0.04 0.12 0.04"/></geometry><material name="light_rear_visual_mat"><color rgba="0.0 0.0 0.0 1.0"/></material></visual>
-    </link>
-    <link name="${prefix}light_left_link">
-      <inertial><origin xyz="0 0 0" rpy="0 0 0"/><mass value="1e-6"/><inertia ixx="1e-9" ixy="0" ixz="0" iyy="1e-9" iyz="0" izz="1e-9"/></inertial>
-      <visual name="light_left_visual"><origin xyz="0 -0.03 0" rpy="0 0 0"/><geometry><box size="0.12 0.04 0.04"/></geometry><material name="light_left_visual_mat"><color rgba="0.0 0.0 0.0 1.0"/></material></visual>
-    </link>
-    <link name="${prefix}light_right_link">
-      <inertial><origin xyz="0 0 0" rpy="0 0 0"/><mass value="1e-6"/><inertia ixx="1e-9" ixy="0" ixz="0" iyy="1e-9" iyz="0" izz="1e-9"/></inertial>
-      <visual name="light_right_visual"><origin xyz="0 0.03 0" rpy="0 0 0"/><geometry><box size="0.12 0.04 0.04"/></geometry><material name="light_right_visual_mat"><color rgba="0.0 0.0 0.0 1.0"/></material></visual>
-    </link>
+    <!-- JOINTS -->
+    <!-- base joints -->
     <xacro:if value="${parent != ''}">
       <joint name="${prefix}base_joint" type="fixed">
@@ -340,4 +476,5 @@
       <origin xyz="0 0 0.1275" rpy="0 0 0"/>
     </joint>
+    <!-- wheel joints -->
     <joint name="${prefix}front_left_wheel_joint" type="continuous">
       <parent link="${prefix}base_link"/>
@@ -368,4 +505,5 @@
       <limit effort="50" velocity="19.61"/>
     </joint>
+    <!-- sensor and light frame joints -->
     <joint name="${prefix}base_link_to_imu_sensor_link_joint" type="fixed">
       <parent link="${prefix}base_link"/>
@@ -387,24 +525,4 @@
       <child link="${prefix}lidar_link"/>
       <origin xyz="0 0 0.365" rpy="0 0 0"/>
-    </joint>
-    <joint name="${prefix}base_link_to_light_front_link_joint" type="fixed">
-      <parent link="${prefix}base_link"/>
-      <child link="${prefix}light_front_link"/>
-      <origin xyz="0.12 0 0.457" rpy="0 -1.5707963267948966 0"/>
-    </joint>
-    <joint name="${prefix}base_link_to_light_rear_link_joint" type="fixed">
-      <parent link="${prefix}base_link"/>
-      <child link="${prefix}light_rear_link"/>
-      <origin xyz="-0.12 0 0.457" rpy="0 1.5707963267948966 0"/>
-    </joint>
-    <joint name="${prefix}base_link_to_light_left_link_joint" type="fixed">
-      <parent link="${prefix}base_link"/>
-      <child link="${prefix}light_left_link"/>
-      <origin xyz="0 0.12 0.457" rpy="1.5707963267948966 0 0"/>
-    </joint>
-    <joint name="${prefix}base_link_to_light_right_link_joint" type="fixed">
-      <parent link="${prefix}base_link"/>
-      <child link="${prefix}light_right_link"/>
-      <origin xyz="0 -0.12 0.457" rpy="-1.5707963267948966 0 0"/>
     </joint>
     <!-- GAZEBO EXTENSIONS -->
