Commit message: Add visual structure fo Cornelius for the sensors

File: cororos2_description/urdf/allie/allie_macro.xacro (robot description, xacro)
@@ -44,52 +44,4 @@
         </geometry>
       </collision>
-      <collision name="ouster_deck_collision">
-        <origin xyz="0.175 0.01 0.3625" rpy="0 0 0" />
-        <geometry>
-          <box size="0.24 0.18 0.02" />
-        </geometry>
-      </collision>
-      <collision name="beam1_collision">
-        <origin xyz="0.255 0.07 0.24375" rpy="0 0 0" />
-        <geometry>
-          <box size="0.02 0.02 0.2375" />
-        </geometry>
-      </collision>
-      <collision name="beam2_collision">
-        <origin xyz="0.255 -0.05 0.24375" rpy="0 0 0" />
-        <geometry>
-          <box size="0.02 0.02 0.2375" />
-        </geometry>
-      </collision>
-      <collision name="beam3_collision">
-        <origin xyz="0.095 0.07 0.24375" rpy="0 0 0" />
-        <geometry>
-          <box size="0.02 0.02 0.2375" />
-        </geometry>
-      </collision>
-      <collision name="beam4_collision">
-        <origin xyz="0.095 -0.05 0.24375" rpy="0 0 0" />
-        <geometry>
-          <box size="0.02 0.02 0.2375" />
-        </geometry>
-      </collision>
-      <collision name="sensor_mast_collision">
-        <origin xyz="0.255 0.07 1.01625" rpy="0 0 0" />
-        <geometry>
-          <box size="0.03 0.03 1.3175" />
-        </geometry>
-      </collision>
-      <collision name="camera_plate_collision">
-        <origin xyz="0.2745 0.01 1.552" rpy="0 0 0" />
-        <geometry>
-          <box size="0.095 0.16 0.02" />
-        </geometry>
-      </collision>
-      <collision name="gps_board_collision">
-        <origin xyz="0.27 0.09 1.675" rpy="0 0 0" />
-        <geometry>
-          <box size="0.12 0.08 0.02" />
-        </geometry>
-      </collision>
       <!-- visuals -->
       <visual name="chassis_main_visual">
@@ -302,4 +254,22 @@
         <inertia ixx="1e-9" ixy="0" ixz="0" iyy="1e-9" iyz="0" izz="1e-9" />
       </inertial>
+      <collision name="gps_base_collision">
+        <origin xyz="0 0 0.012" rpy="0 0 0" />
+        <geometry>
+          <cylinder radius="0.028" length="0.024" />
+        </geometry>
+      </collision>
+      <collision name="gps_cap_collision">
+        <origin xyz="0 0 0.028" rpy="0 0 0" />
+        <geometry>
+          <sphere radius="0.016" />
+        </geometry>
+      </collision>
+      <collision name="gps_antenna_tip_collision">
+        <origin xyz="0 0 0.060" rpy="0 0 0" />
+        <geometry>
+          <cylinder radius="0.0035" length="0.024" />
+        </geometry>
+      </collision>
       <visual name="gps_base_visual">
         <origin xyz="0 0 0.012" rpy="0 0 0" />
@@ -337,4 +307,10 @@
         <inertia ixx="1e-9" ixy="0" ixz="0" iyy="1e-9" iyz="0" izz="1e-9" />
       </inertial>
+      <collision name="d435i_realsense_camera_collision">
+        <origin xyz="-0.017356 0 -0.009938" rpy="0 0 0" />
+        <geometry>
+          <mesh filename="package://cororos2_description/meshes/allie/visual/realsense_d435.dae" scale="0.001 0.001 0.001" />
+        </geometry>
+      </collision>
       <visual name="d435i_realsense_camera_visual">
         <origin xyz="-0.017356 0 -0.009938" rpy="0 0 0" />
@@ -351,4 +327,16 @@
         <inertia ixx="1e-9" ixy="0" ixz="0" iyy="1e-9" iyz="0" izz="1e-9" />
       </inertial>
+      <collision name="ouster_body_collision">
+        <origin xyz="0 0 0" rpy="0 0 0" />
+        <geometry>
+          <cylinder radius="0.055" length="0.075" />
+        </geometry>
+      </collision>
+      <collision name="ouster_window_collision">
+        <origin xyz="0.042 0 0" rpy="0 0 0" />
+        <geometry>
+          <box size="0.008 0.09 0.035" />
+        </geometry>
+      </collision>
       <visual name="ouster_body_visual">
         <origin xyz="0 0 0" rpy="0 0 0" />
@@ -438,5 +426,5 @@
       <parent link="${prefix}base_link" />
       <child link="${prefix}gps_link" />
-      <origin xyz="0.27 0.09 1.685" rpy="0 0 0" />
+      <origin xyz="0.27 0.09 1.681" rpy="0 0 0" />
     </joint>
     <!-- base link to front RGB-D camera frame -->

File: cororos2_description/urdf/cornelius/cornelius_macro.xacro (robot description, xacro)
@@ -13,91 +13,45 @@
         <inertia ixx="0.615397" ixy="-0.0240585" ixz="-0.120749" iyy="1.75388" iyz="-0.0028322" izz="2.03641" />
       </inertial>
-      <collision name="base_link_collision_top">
-        <origin xyz="0 0 0.12" rpy="0 0 0" />
-        <geometry>
-          <box size="0.92 0.52 0.04" />
-        </geometry>
-      </collision>
-      <collision name="base_link_collision_bottom">
-        <origin xyz="0 0 0.046" rpy="0 0 0" />
-        <geometry>
-          <box size="0.80 0.5709 0.2" />
-        </geometry>
-      </collision>
-      <collision name="plate1_collision">
+      <!-- collisions -->
+      <collision name="chassis_main_collision">
+        <origin xyz="0 0 -0.135" rpy="0 0 1.57" />
+        <geometry>
+          <mesh filename="package://cororos2_description/meshes/cornelius/visual/hd2_marble_base_body_metric.dae" />
+        </geometry>
+      </collision>
+      <!-- visuals -->
+      <visual name="chassis_main_visual">
+        <origin xyz="0 0 -0.135" rpy="0 0 1.57" />
+        <geometry>
+          <mesh filename="package://cororos2_description/meshes/cornelius/visual/hd2_marble_base_body_metric.dae" />
+        </geometry>
+        <material name="chassis_main_visual_mat">
+          <color rgba="1.0 1.0 1.0 1.0" />
+        </material>
+      </visual>
+      <visual name="sensor_upper_deck_visual">
         <origin xyz="0.19 0 0.38" rpy="0 0 0" />
         <geometry>
-          <box size="0.2 0.2 0.01" />
-        </geometry>
-      </collision>
-      <collision name="plate2_collision">
+          <box size="0.2 0.22 0.005" />
+        </geometry>
+        <material name="sensor_upper_deck_visual_mat">
+          <color rgba="0.7843 0.7843 0.7843 1.0" />
+        </material>
+      </visual>
+      <visual name="sensor_mid_deck_visual">
         <origin xyz="0.19 0 0.27" rpy="0 0 0" />
         <geometry>
-          <box size="0.2 0.2 0.01" />
-        </geometry>
-      </collision>
-      <collision name="plate3_collision">
+          <box size="0.2 0.2 0.005" />
+        </geometry>
+        <material name="sensor_mid_deck_visual_mat">
+          <color rgba="0.7843 0.7843 0.7843 1.0" />
+        </material>
+      </visual>
+      <visual name="sensor_lower_deck_visual">
         <origin xyz="0.19 0 0.08" rpy="0 0 0" />
         <geometry>
-          <box size="0.2 0.2 0.01" />
-        </geometry>
-      </collision>
-      <collision name="beam1_collision">
-        <origin xyz="0.281 0.091 0.23" rpy="0 0 0" />
-        <geometry>
-          <box size="0.03 0.03 0.3" />
-        </geometry>
-      </collision>
-      <collision name="beam2_collision">
-        <origin xyz="0.281 -0.091 0.23" rpy="0 0 0" />
-        <geometry>
-          <box size="0.03 0.03 0.3" />
-        </geometry>
-      </collision>
-      <collision name="beam3_collision">
-        <origin xyz="0.099 0.091 0.23" rpy="0 0 0" />
-        <geometry>
-          <box size="0.03 0.03 0.3" />
-        </geometry>
-      </collision>
-      <collision name="beam4_collision">
-        <origin xyz="0.099 -0.091 0.23" rpy="0 0 0" />
-        <geometry>
-          <box size="0.03 0.03 0.3" />
-        </geometry>
-      </collision>
-      <visual name="body_visual">
-        <origin xyz="0 0 -0.135" rpy="0 0 1.57" />
-        <geometry>
-          <mesh filename="package://cororos2_description/meshes/cornelius/visual/hd2_marble_base_body_metric.dae" />
-        </geometry>
-        <material name="body_visual_mat">
-          <color rgba="1.0 1.0 1.0 1.0" />
-        </material>
-      </visual>
-      <visual name="plate1_visual">
-        <origin xyz="0.19 0 0.38" rpy="0 0 0" />
-        <geometry>
           <box size="0.2 0.2 0.005" />
         </geometry>
-        <material name="plate1_visual_mat">
-          <color rgba="0.7843 0.7843 0.7843 1.0" />
-        </material>
-      </visual>
-      <visual name="plate2_visual">
-        <origin xyz="0.19 0 0.27" rpy="0 0 0" />
-        <geometry>
-          <box size="0.2 0.2 0.005" />
-        </geometry>
-        <material name="plate2_visual_mat">
-          <color rgba="0.7843 0.7843 0.7843 1.0" />
-        </material>
-      </visual>
-      <visual name="plate3_visual">
-        <origin xyz="0.19 0 0.08" rpy="0 0 0" />
-        <geometry>
-          <box size="0.2 0.2 0.005" />
-        </geometry>
-        <material name="plate3_visual_mat">
+        <material name="sensor_lower_deck_visual_mat">
           <color rgba="0.9412 0.9412 0.9412 1.0" />
         </material>
@@ -136,4 +90,31 @@
         </geometry>
         <material name="beam4_visual_mat">
+          <color rgba="0.7843 0.7843 0.7843 1.0" />
+        </material>
+      </visual>
+      <visual name="sensor_mast_visual">
+        <origin xyz="0.27 0.09 1.03" rpy="0 0 0" />
+        <geometry>
+          <box size="0.025 0.025 1.30" />
+        </geometry>
+        <material name="sensor_mast_visual_mat">
+          <color rgba="0.7843 0.7843 0.7843 1.0" />
+        </material>
+      </visual>
+      <visual name="camera_plate_visual">
+        <origin xyz="0.2425 0.01 1.521" rpy="0 0 0" />
+        <geometry>
+          <box size="0.085 0.22 0.012" />
+        </geometry>
+        <material name="camera_plate_visual_mat">
+          <color rgba="0.7843 0.7843 0.7843 1.0" />
+        </material>
+      </visual>
+      <visual name="gps_board_visual">
+        <origin xyz="0.27 0.09 1.675" rpy="0 0 0" />
+        <geometry>
+          <box size="0.12 0.08 0.012" />
+        </geometry>
+        <material name="gps_board_visual_mat">
           <color rgba="0.7843 0.7843 0.7843 1.0" />
         </material>
@@ -148,4 +129,22 @@
         <inertia ixx="0.03828" ixy="0" ixz="0" iyy="0.2925" iyz="0" izz="0.2642" />
       </inertial>
+      <collision name="left_track_body_collision">
+        <origin xyz="0 0 0" rpy="0 0 0" />
+        <geometry>
+          <box size="0.72 0.1 0.258" />
+        </geometry>
+      </collision>
+      <collision name="left_track_front_wheel_collision">
+        <origin xyz="0.36 0 0" rpy="1.5707963267948966 0 0" />
+        <geometry>
+          <cylinder radius="0.129" length="0.1" />
+        </geometry>
+      </collision>
+      <collision name="left_track_rear_wheel_collision">
+        <origin xyz="-0.36 0 0" rpy="1.5707963267948966 0 0" />
+        <geometry>
+          <cylinder radius="0.129" length="0.1" />
+        </geometry>
+      </collision>
       <visual name="left_track_body_visual">
         <origin xyz="0 0 0" rpy="0 0 0" />
@@ -183,4 +182,22 @@
         <inertia ixx="0.03828" ixy="0" ixz="0" iyy="0.2925" iyz="0" izz="0.2642" />
       </inertial>
+      <collision name="right_track_body_collision">
+        <origin xyz="0 0 0" rpy="0 0 0" />
+        <geometry>
+          <box size="0.72 0.1 0.258" />
+        </geometry>
+      </collision>
+      <collision name="right_track_front_wheel_collision">
+        <origin xyz="0.36 0 0" rpy="1.5707963267948966 0 0" />
+        <geometry>
+          <cylinder radius="0.129" length="0.1" />
+        </geometry>
+      </collision>
+      <collision name="right_track_rear_wheel_collision">
+        <origin xyz="-0.36 0 0" rpy="1.5707963267948966 0 0" />
+        <geometry>
+          <cylinder radius="0.129" length="0.1" />
+        </geometry>
+      </collision>
       <visual name="right_track_body_visual">
         <origin xyz="0 0 0" rpy="0 0 0" />
@@ -281,4 +298,49 @@
         <inertia ixx="1e-9" ixy="0" ixz="0" iyy="1e-9" iyz="0" izz="1e-9" />
       </inertial>
+      <collision name="gps_base_collision">
+        <origin xyz="0 0 0.012" rpy="0 0 0" />
+        <geometry>
+          <cylinder radius="0.028" length="0.024" />
+        </geometry>
+      </collision>
+      <collision name="gps_cap_collision">
+        <origin xyz="0 0 0.028" rpy="0 0 0" />
+        <geometry>
+          <sphere radius="0.016" />
+        </geometry>
+      </collision>
+      <collision name="gps_antenna_tip_collision">
+        <origin xyz="0 0 0.060" rpy="0 0 0" />
+        <geometry>
+          <cylinder radius="0.0035" length="0.024" />
+        </geometry>
+      </collision>
+      <visual name="gps_base_visual">
+        <origin xyz="0 0 0.012" rpy="0 0 0" />
+        <geometry>
+          <cylinder radius="0.028" length="0.024" />
+        </geometry>
+        <material name="gps_base_visual_mat">
+          <color rgba="0.92 0.92 0.92 1.0" />
+        </material>
+      </visual>
+      <visual name="gps_cap_visual">
+        <origin xyz="0 0 0.028" rpy="0 0 0" />
+        <geometry>
+          <sphere radius="0.016" />
+        </geometry>
+        <material name="gps_cap_visual_mat">
+          <color rgba="0.96 0.96 0.96 1.0" />
+        </material>
+      </visual>
+      <visual name="gps_antenna_tip_visual">
+        <origin xyz="0 0 0.060" rpy="0 0 0" />
+        <geometry>
+          <cylinder radius="0.0035" length="0.024" />
+        </geometry>
+        <material name="gps_antenna_tip_visual_mat">
+          <color rgba="0.2 0.2 0.2 1.0" />
+        </material>
+      </visual>
     </link>
     <!-- front RGB-D camera frame -->
@@ -289,5 +351,11 @@
         <inertia ixx="1e-9" ixy="0" ixz="0" iyy="1e-9" iyz="0" izz="1e-9" />
       </inertial>
-      <visual name="rgbd_front_visual">
+      <collision name="d435i_realsense_camera_collision">
+        <origin xyz="0 0 0" rpy="0 0 0" />
+        <geometry>
+          <mesh filename="package://cororos2_description/meshes/cornelius/visual/realsense_d435.dae" scale="0.001 0.001 0.001" />
+        </geometry>
+      </collision>
+      <visual name="d435i_realsense_camera_visual">
         <origin xyz="0 0 0" rpy="0 0 0" />
         <geometry>
@@ -303,4 +371,22 @@
         <inertia ixx="1e-9" ixy="0" ixz="0" iyy="1e-9" iyz="0" izz="1e-9" />
       </inertial>
+      <collision name="vlp16_collision1">
+        <origin xyz="0 0 0" rpy="0 0 0" />
+        <geometry>
+          <mesh filename="package://cororos2_description/meshes/cornelius/visual/VLP16_base_1.dae" />
+        </geometry>
+      </collision>
+      <collision name="vlp16_collision2">
+        <origin xyz="0 0 0" rpy="0 0 0" />
+        <geometry>
+          <mesh filename="package://cororos2_description/meshes/cornelius/visual/VLP16_base_2.dae" />
+        </geometry>
+      </collision>
+      <collision name="vlp16_collision3">
+        <origin xyz="0 0 0" rpy="0 0 0" />
+        <geometry>
+          <mesh filename="package://cororos2_description/meshes/cornelius/visual/VLP16_scan.dae" />
+        </geometry>
+      </collision>
       <visual name="vlp16_visual1">
         <origin xyz="0 0 0" rpy="0 0 0" />
@@ -395,10 +481,10 @@
       <parent link="${prefix}base_link" />
       <child link="${prefix}gps_link" />
-      <origin xyz="0.19 0 0.402" rpy="0 0 0" />
+      <origin xyz="0.27 0.09 1.681" rpy="0 0 0" />
     </joint>
     <joint name="${prefix}base_link_to_rgbd_front_link_joint" type="fixed">
       <parent link="${prefix}base_link" />
       <child link="${prefix}rgbd_front_link" />
-      <origin xyz="0.28 0 1.5" rpy="0 -0.5236 0" />
+      <origin xyz="0.28 0 1.5" rpy="0 0.5236 0" />
     </joint>
     <joint name="${prefix}base_link_to_ouster_link_joint" type="fixed">

File: cororos2_description/urdf/joe/joe_macro.xacro (robot description, xacro)
@@ -54,64 +54,4 @@
         </geometry>
       </collision>
-      <collision name="sensor_upper_deck_collision">
-        <origin xyz="0 0 0.435" rpy="0 0 0"/>
-        <geometry>
-          <box size="0.2 0.2 0.01"/>
-        </geometry>
-      </collision>
-      <collision name="sensor_mid_deck_collision">
-        <origin xyz="0 0 0.325" rpy="0 0 0"/>
-        <geometry>
-          <box size="0.2 0.2 0.01"/>
-        </geometry>
-      </collision>
-      <collision name="sensor_lower_deck_collision">
-        <origin xyz="0 0 0.135" rpy="0 0 0"/>
-        <geometry>
-          <box size="0.2 0.2 0.01"/>
-        </geometry>
-      </collision>
-      <collision name="beam1_collision">
-        <origin xyz="0.091 0.091 0.285" rpy="0 0 0"/>
-        <geometry>
-          <box size="0.02 0.02 0.3"/>
-        </geometry>
-      </collision>
-      <collision name="beam2_collision">
-        <origin xyz="0.091 -0.091 0.285" rpy="0 0 0"/>
-        <geometry>
-          <box size="0.02 0.02 0.3"/>
-        </geometry>
-      </collision>
-      <collision name="beam3_collision">
-        <origin xyz="-0.091 0.091 0.285" rpy="0 0 0"/>
-        <geometry>
-          <box size="0.02 0.02 0.3"/>
-        </geometry>
-      </collision>
-      <collision name="beam4_collision">
-        <origin xyz="-0.091 -0.091 0.285" rpy="0 0 0"/>
-        <geometry>
-          <box size="0.02 0.02 0.3"/>
-        </geometry>
-      </collision>
-      <collision name="sensor_mast_collision">
-        <origin xyz="0 0 1.0125" rpy="0 0 0"/>
-        <geometry>
-          <box size="0.03 0.03 1.125"/>
-        </geometry>
-      </collision>
-      <collision name="camera_plate_collision">
-        <origin xyz="0.035 0 1.525" rpy="0 0 0"/>
-        <geometry>
-          <box size="0.11 0.12 0.02"/>
-        </geometry>
-      </collision>
-      <collision name="gps_board_collision">
-        <origin xyz="0 0 1.57" rpy="0 0 0"/>
-        <geometry>
-          <box size="0.14 0.10 0.02"/>
-        </geometry>
-      </collision>
       <!-- visuals -->
       <visual name="chassis_main_visual">
@@ -396,4 +336,22 @@
         <inertia ixx="1e-9" ixy="0" ixz="0" iyy="1e-9" iyz="0" izz="1e-9"/>
       </inertial>
+      <collision name="gps_base_collision">
+        <origin xyz="0 0 0.012" rpy="0 0 0"/>
+        <geometry>
+          <cylinder radius="0.028" length="0.024"/>
+        </geometry>
+      </collision>
+      <collision name="gps_cap_collision">
+        <origin xyz="0 0 0.028" rpy="0 0 0"/>
+        <geometry>
+          <sphere radius="0.016"/>
+        </geometry>
+      </collision>
+      <collision name="gps_antenna_tip_collision">
+        <origin xyz="0 0 0.060" rpy="0 0 0"/>
+        <geometry>
+          <cylinder radius="0.0035" length="0.024"/>
+        </geometry>
+      </collision>
       <visual name="gps_base_visual">
         <origin xyz="0 0 0.012" rpy="0 0 0"/>
@@ -430,4 +388,10 @@
         <inertia ixx="1e-9" ixy="0" ixz="0" iyy="1e-9" iyz="0" izz="1e-9"/>
       </inertial>
+      <collision name="d435i_realsense_camera_collision">
+        <origin xyz="-0.03 0 0" rpy="0 0 0"/>
+        <geometry>
+          <mesh filename="package://cororos2_description/meshes/joe/visual/realsense_d435.dae" scale="0.001 0.001 0.001"/>
+        </geometry>
+      </collision>
       <visual name="d435i_realsense_camera_visual">
         <origin xyz="-0.03 0 0" rpy="0 0 0"/>
@@ -443,4 +407,22 @@
         <inertia ixx="1e-9" ixy="0" ixz="0" iyy="1e-9" iyz="0" izz="1e-9"/>
       </inertial>
+      <collision name="vlp16_collision1">
+        <origin xyz="0 0 -0.038" rpy="0 0 0"/>
+        <geometry>
+          <mesh filename="package://cororos2_description/meshes/joe/visual/VLP16_base_1.dae" scale="1 1 1"/>
+        </geometry>
+      </collision>
+      <collision name="vlp16_collision2">
+        <origin xyz="0 0 -0.038" rpy="0 0 0"/>
+        <geometry>
+          <mesh filename="package://cororos2_description/meshes/joe/visual/VLP16_base_2.dae" scale="1 1 1"/>
+        </geometry>
+      </collision>
+      <collision name="vlp16_collision3">
+        <origin xyz="0 0 -0.038" rpy="0 0 0"/>
+        <geometry>
+          <mesh filename="package://cororos2_description/meshes/joe/visual/VLP16_scan.dae" scale="1 1 1"/>
+        </geometry>
+      </collision>
       <visual name="vlp16_visual1">
         <origin xyz="0 0 -0.038" rpy="0 0 0"/>
@@ -514,5 +496,5 @@
       <parent link="${prefix}base_link"/>
       <child link="${prefix}gps_link"/>
-      <origin xyz="0 0 1.58" rpy="0 0 0"/>
+      <origin xyz="0 0 1.576" rpy="0 0 0"/>
     </joint>
     <joint name="${prefix}base_link_to_rgbd_front_link_joint" type="fixed">

Commit message: Fix ouster sensor positions and ekf in gazebo. Update README. Make allie use open loop.

File: cororos2_description/urdf/allie/allie_macro.xacro (robot description, xacro)
@@ -438,5 +438,5 @@
       <parent link="${prefix}base_link" />
       <child link="${prefix}ouster_link" />
-      <origin xyz="0.16 0 0.405" rpy="0 0 0" />
+      <origin xyz="0.16 0 0.405" rpy="0 0 3.141592653589793" />
     </joint>
     <!-- Ouster sensor frame to Ouster IMU frame -->

File: cororos2_description/urdf/cornelius/cornelius_macro.xacro (robot description, xacro)
@@ -491,5 +491,5 @@
       <parent link="${prefix}base_link" />
       <child link="${prefix}ouster_link" />
-      <origin xyz="0.19 0 0.272" rpy="0 0 0" />
+      <origin xyz="0.19 0 0.272" rpy="0 0 3.141592653589793" />
     </joint>
     <joint name="${prefix}ouster_link_to_ouster_imu_link_joint" type="fixed">

Commit message: Adjust ouster orientation. Add an ekf hw config file

File: cororos2_description/urdf/allie/allie_macro.xacro (robot description, xacro)
@@ -1,5 +1,5 @@
 <?xml version='1.0' encoding='utf-8'?>
 <robot xmlns:xacro="http://wiki.ros.org/xacro">
-  <xacro:macro name="allie" params="prefix parent *origin">
+  <xacro:macro name="allie" params="prefix parent sim_gazebo:=false sim_gazebo_classic:=false *origin">
     <!-- LINKS -->
     <!-- base footprint -->
@@ -438,5 +438,10 @@
       <parent link="${prefix}base_link" />
       <child link="${prefix}ouster_link" />
-      <origin xyz="0.16 0 0.405" rpy="0 0 3.141592653589793" />
+      <xacro:if value="${sim_gazebo or sim_gazebo_classic}">
+        <origin xyz="0.16 0 0.405" rpy="0 0 3.141592653589793" />
+      </xacro:if>
+      <xacro:unless value="${sim_gazebo or sim_gazebo_classic}">
+        <origin xyz="0.16 0 0.405" rpy="0 0 0" />
+      </xacro:unless>
     </joint>
     <!-- Ouster sensor frame to Ouster IMU frame -->

File: cororos2_description/urdf/cornelius/cornelius_macro.xacro (robot description, xacro)
@@ -1,5 +1,5 @@
 <?xml version='1.0' encoding='utf-8'?>
 <robot xmlns:xacro="http://wiki.ros.org/xacro">
-  <xacro:macro name="cornelius" params="prefix parent *origin">
+  <xacro:macro name="cornelius" params="prefix parent sim_gazebo:=false sim_gazebo_classic:=false *origin">
     <!-- LINKS -->
     <!-- base footprint -->
@@ -491,5 +491,10 @@
       <parent link="${prefix}base_link" />
       <child link="${prefix}ouster_link" />
-      <origin xyz="0.19 0 0.272" rpy="0 0 3.141592653589793" />
+      <xacro:if value="${sim_gazebo or sim_gazebo_classic}">
+        <origin xyz="0.19 0 0.272" rpy="0 0 3.141592653589793" />
+      </xacro:if>
+      <xacro:unless value="${sim_gazebo or sim_gazebo_classic}">
+        <origin xyz="0.19 0 0.272" rpy="0 0 0" />
+      </xacro:unless>
     </joint>
     <joint name="${prefix}ouster_link_to_ouster_imu_link_joint" type="fixed">
