Commit message: Add fixes

File: cororos2_description/urdf/allie/allie_macro.xacro (robot description, xacro)
@@ -622,4 +622,28 @@
       </sensor>
     </gazebo>
+    <gazebo reference="${prefix}front_left_wheel">
+      <mu1>2.5</mu1>
+      <mu2>2.5</mu2>
+      <kp>1000000.0</kp>
+      <kd>100.0</kd>
+    </gazebo>
+    <gazebo reference="${prefix}front_right_wheel">
+      <mu1>2.5</mu1>
+      <mu2>2.5</mu2>
+      <kp>1000000.0</kp>
+      <kd>100.0</kd>
+    </gazebo>
+    <gazebo reference="${prefix}rear_left_wheel">
+      <mu1>2.5</mu1>
+      <mu2>2.5</mu2>
+      <kp>1000000.0</kp>
+      <kd>100.0</kd>
+    </gazebo>
+    <gazebo reference="${prefix}rear_right_wheel">
+      <mu1>2.5</mu1>
+      <mu2>2.5</mu2>
+      <kp>1000000.0</kp>
+      <kd>100.0</kd>
+    </gazebo>
   </xacro:macro>
 </robot>

File: cororos2_description/urdf/cornelius/cornelius_macro.xacro (robot description, xacro)
@@ -14,10 +14,12 @@
       </inertial>
       <!-- collisions -->
-      <collision name="chassis_main_collision">
-        <origin xyz="0 0 -0.135" rpy="0 0 1.57" />
-        <geometry>
-          <mesh filename="package://cororos2_description/meshes/cornelius/collision/hd2_marble_base_body_collision.stl" />
-        </geometry>
-      </collision>
+      <xacro:unless value="${sim_gazebo or sim_gazebo_classic}">
+        <collision name="chassis_main_collision">
+          <origin xyz="0 0 -0.135" rpy="0 0 1.57" />
+          <geometry>
+            <mesh filename="package://cororos2_description/meshes/cornelius/collision/hd2_marble_base_body_collision.stl" />
+          </geometry>
+        </collision>
+      </xacro:unless>
       <!-- visuals -->
       <visual name="chassis_main_visual">
@@ -129,22 +131,24 @@
         <inertia ixx="0.03828" ixy="0" ixz="0" iyy="0.2925" iyz="0" izz="0.2642" />
       </inertial>
-      <collision name="left_track_body_collision">
-        <origin xyz="0 0 0" rpy="0 0 0" />
-        <geometry>
-          <box size="0.72 0.14 0.258" />
-        </geometry>
-      </collision>
-      <collision name="left_track_front_wheel_collision">
-        <origin xyz="0.355 0 0" rpy="1.5707963267948966 0 0" />
-        <geometry>
-          <cylinder radius="0.13" length="0.14" />
-        </geometry>
-      </collision>
-      <collision name="left_track_rear_wheel_collision">
-        <origin xyz="-0.355 0 0" rpy="1.5707963267948966 0 0" />
-        <geometry>
-          <cylinder radius="0.13" length="0.14" />
-        </geometry>
-      </collision>
+      <xacro:unless value="${sim_gazebo or sim_gazebo_classic}">
+        <collision name="left_track_body_collision">
+          <origin xyz="0 0 0" rpy="0 0 0" />
+          <geometry>
+            <box size="0.72 0.14 0.258" />
+          </geometry>
+        </collision>
+        <collision name="left_track_front_wheel_collision">
+          <origin xyz="0.355 0 0" rpy="1.5707963267948966 0 0" />
+          <geometry>
+            <cylinder radius="0.13" length="0.14" />
+          </geometry>
+        </collision>
+        <collision name="left_track_rear_wheel_collision">
+          <origin xyz="-0.355 0 0" rpy="1.5707963267948966 0 0" />
+          <geometry>
+            <cylinder radius="0.13" length="0.14" />
+          </geometry>
+        </collision>
+      </xacro:unless>
       <visual name="left_track_body_visual">
         <origin xyz="0 0 0" rpy="0 0 0" />
@@ -182,22 +186,24 @@
         <inertia ixx="0.03828" ixy="0" ixz="0" iyy="0.2925" iyz="0" izz="0.2642" />
       </inertial>
-      <collision name="right_track_body_collision">
-        <origin xyz="0 0 0" rpy="0 0 0" />
-        <geometry>
-          <box size="0.72 0.14 0.258" />
-        </geometry>
-      </collision>
-      <collision name="right_track_front_wheel_collision">
-        <origin xyz="0.355 0 0" rpy="1.5707963267948966 0 0" />
-        <geometry>
-          <cylinder radius="0.13" length="0.14" />
-        </geometry>
-      </collision>
-      <collision name="right_track_rear_wheel_collision">
-        <origin xyz="-0.355 0 0" rpy="1.5707963267948966 0 0" />
-        <geometry>
-          <cylinder radius="0.13" length="0.14" />
-        </geometry>
-      </collision>
+      <xacro:unless value="${sim_gazebo or sim_gazebo_classic}">
+        <collision name="right_track_body_collision">
+          <origin xyz="0 0 0" rpy="0 0 0" />
+          <geometry>
+            <box size="0.72 0.14 0.258" />
+          </geometry>
+        </collision>
+        <collision name="right_track_front_wheel_collision">
+          <origin xyz="0.355 0 0" rpy="1.5707963267948966 0 0" />
+          <geometry>
+            <cylinder radius="0.13" length="0.14" />
+          </geometry>
+        </collision>
+        <collision name="right_track_rear_wheel_collision">
+          <origin xyz="-0.355 0 0" rpy="1.5707963267948966 0 0" />
+          <geometry>
+            <cylinder radius="0.13" length="0.14" />
+          </geometry>
+        </collision>
+      </xacro:unless>
       <visual name="right_track_body_visual">
         <origin xyz="0 0 0" rpy="0 0 0" />
